Commit message: create gazebo ros control packages

File: summit_mico_description/robots/summit_xl_hl_ext_mico.urdf.xacro (robot description, xacro)
@@ -12,5 +12,6 @@
 	<xacro:include filename="$(find robotnik_sensors)/urdf/all_sensors.urdf.xacro" />
 	<!-- Import Mico Arm -->
-	<xacro:include filename="$(find mico_description)/urdf/mico_arm.urdf.xacro" />
+<!--	<xacro:include filename="$(find mico_description)/urdf/mico_arm.urdf.xacro" />-->
+	<xacro:include filename="$(find kinova_description)/urdf/m1n6s200.xacro" />
 	<!-- ***************** -->
 	<!-- Global parameters -->
@@ -47,5 +48,13 @@
 	</xacro:rubber_wheel>
 <!-- ARM KINOVA MICO2 -->
-	<xacro:mico_arm parent="base_link" xyz="0.19 0 0.17" rpy="0 ${15*PI/180} 0"/>
+  <link name="root"/>
+  <joint name="connect_root_and_summit" type="fixed">
+    <child link="root" />
+    <parent link="base_link" />
+    <origin xyz="0.19 0 0.17" rpy="0 ${15*PI/180} 0" />
+  </joint>
+  <property name="robot_root" value="root" />
+  <xacro:m1n6s200  base_parent="${robot_root}" prefix="mico"/>
+	<!--<xacro:mico_arm parent="base_link" xyz="0.19 0 0.17" rpy="0 ${15*PI/180} 0"/>-->
 	<!-- SENSORS -->
 <!--
