Commit message: fix controller issues

File: summit_mico_description/robots/summit_mico_diff.urdf (robot description, URDF)
Before this commit: robot summit_xl_mico, 19 links, 18 joints
Links:
- link back_left_wheel: geometry collision cylinder length=0.14 radius=0.125; visual mesh filename=package://summit_description/meshes/wheels/rubber_wheel_lef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
- link back_right_wheel: geometry collision cylinder length=0.14 radius=0.125; visual mesh filename=package://summit_description/meshes/wheels/rubber_wheel_rig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
- link base_link: geometry collision mesh filename=package://summit_description/meshes/bases/summit_xl_hl_chas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; visual mesh filename=package://summit_description/meshes/bases/summit_xl_hl_chas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
- link front_left_wheel: geometry collision cylinder length=0.14 radius=0.125; visual mesh filename=package://summit_description/meshes/wheels/rubber_wheel_lef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
- link front_right_wheel: geometry collision cylinder length=0.14 radius=0.125; visual mesh filename=package://summit_description/meshes/wheels/rubber_wheel_rig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
- link mico_link_1: geometry collision mesh filename=package://mico_description/meshes/shoulder.dae; visual mesh filename=package://mico_description/meshes/ring_big.STL
- link mico_link_2: geometry collision mesh filename=package://mico_description/meshes/arm_mico.dae; visual mesh filename=package://mico_description/meshes/arm_mico.dae
- link mico_link_3: geometry collision mesh filename=package://mico_description/meshes/forearm_mico.dae; visual mesh filename=package://mico_description/meshes/forearm_mico.dae
- link mico_link_4: geometry collision mesh filename=package://mico_description/meshes/wrist.dae; visual mesh filename=package://mico_description/meshes/ring_small.STL
- link mico_link_5: geometry collision mesh filename=package://mico_description/meshes/wrist.dae; visual mesh filename=package://mico_description/meshes/ring_small.STL
- link mico_link_6: geometry collision mesh filename=package://mico_description/meshes/hand_2finger.dae; visual mesh filename=package://mico_description/meshes/hand_2finger.dae
- link mico_link_base: geometry collision mesh filename=package://mico_description/meshes/base.dae; visual mesh filename=package://mico_description/meshes/base.dae
- link mico_link_finger_1: geometry collision mesh filename=package://mico_description/meshes/finger_proximal.dae; visual mesh filename=package://mico_description/meshes/finger_proximal.dae
- link mico_link_finger_2: geometry collision mesh filename=package://mico_description/meshes/finger_proximal.dae; visual mesh filename=package://mico_description/meshes/finger_proximal.dae
- link mico_link_finger_tip_1: geometry collision mesh filename=package://mico_description/meshes/finger_distal.dae; visual mesh filename=package://mico_description/meshes/finger_distal.dae
- link mico_link_finger_tip_2: geometry collision mesh filename=package://mico_description/meshes/finger_distal.dae; visual mesh filename=package://mico_description/meshes/finger_distal.dae

File: summit_mico_description/robots/summit_xl_hl_diff_mico.urdf.xacro (robot description, xacro)
@@ -71,5 +71,36 @@
   <xacro:mico2fingers  base_parent="${robot_root}" prefix="mico"/>
 	<!--<xacro:mico_arm parent="base_link" xyz="0.19 0 0.17" rpy="0 ${15*PI/180} 0"/>-->
+	<!-- Mini PC -->
+	<link name="mini_pc_link">
+    <visual>
+      <origin rpy="0.0 0.0 0.0" xyz="0 0 0.0"/>
+      <geometry>
+        <mesh filename="package://summit_mico_description/meshes/miniPC.STL" scale="0.5 0.5 0.5"/>
+      </geometry>
+      <material name="">
+        <color rgba="0.34 0.35 0.36 1.0"/>
+      </material>
+    </visual>
+    <collision>
+      <origin rpy="0.0 0 0.0" xyz="0 0 0"/>
+      <geometry>
+        <mesh filename="package://summit_mico_description/meshes/miniPC.STL" scale="0.5 0.5 0.5"/>
+      </geometry>
+    </collision>
+    <inertial>
+      <origin rpy="0.0 0.0 0.0" xyz="0 0 0"/>
+      <mass value="1"/>
+      <inertia ixx="1" ixy="0.0" ixz="0.0" iyy="1" iyz="0.0" izz="1"/>
+    </inertial>
+  </link>
+  <joint name="connect_minipc_and_summit" type="fixed">
+    <child link="mini_pc_link" />
+    <parent link="base_link" />
+    <origin xyz="0.0 0 0.5" rpy="0 ${0*PI/180} 0" />
+  </joint>
 	<!-- SENSORS -->
+	<xacro:sensor_kinect name="kinect" parent="base_link">
+		<origin xyz="-0.30 0.0 0.65" rpy="0 ${7.5*PI/180} 0"/>
+	</xacro:sensor_kinect>
 <!--
 	<xacro:sensor_hokuyo_ust10lx prefix="hokuyo_base" parent="base_link">
