Commit message: virtual joints

File: summit_mico_description/robots/summit_mico_root.xacro (robot description, xacro)
@@ -14,5 +14,5 @@
         </xacro:unless>
         <xacro:summit_xl_robot prefix="${prefix}" kinematic_model="${kin_mode}" kinect="${camera}" mini_pc="true" enable_ros_control="false" publish_tf="false" virtual_platform_joints="true">
-            <origin xyz="0 0 0" rpy="0 0 0"/>
+            <origin xyz="3 0 0" rpy="0 0 0"/>
         </xacro:summit_xl_robot>
         <!-- <link name="world">
