Commit message: add virtual platform joints

File: summit_description/robots/summit_xl_hl_root.urdf.xacro (robot description, xacro)
@@ -14,5 +14,5 @@
     <!-- Import all available sensors -->
     <xacro:include filename="$(find robotnik_sensors)/urdf/all_sensors.urdf.xacro" />
-    <xacro:macro name="summit_xl_robot" params="prefix *origin kinematic_model:='omni' kinect:=true mini_pc:=true enable_ros_control=true">
+    <xacro:macro name="summit_xl_robot" params="prefix *origin kinematic_model:='omni' kinect:=true mini_pc:=true enable_ros_control:=true publish_tf:=false virtual_platform_joints:=false">
         <!-- ***************** -->
         <!-- Global parameters -->
@@ -45,5 +45,13 @@
         <!-- Here we create the robot elements using the xacro:macros imported at the beggining of this file -->
         <!-- Summit XL base -->
-        <xacro:summit_xl_hl_base prefix="${prefix}" publish_bf="true" hq="${hq}" />
+        <xacro:if value="${kinematic_model in ['omni', 'force_omni']}">
+            <xacro:property name="wheel_radius" value="0.127" />
+        </xacro:if>
+        <xacro:unless value="${kinematic_model in ['omni', 'force_omni']}">
+            <xacro:property name="wheel_radius" value="0.11" />
+        </xacro:unless>
+        <xacro:summit_xl_hl_base prefix="${prefix}" publish_bf="true" hq="${hq}" virtual_platform_joints="${virtual_platform_joints}" >
+            <xacro:insert_block name="origin" />
+        </xacro:summit_xl_hl_base>
         <!-- WHEELS -->
         <xacro:if value="${kinematic_model in ['omni', 'force_omni']}">
@@ -180,14 +188,14 @@
         <!-- Gazebo ros control pluggins -->
         <xacro:if value="${kinematic_model == 'omni'}">
-            <xacro:omni_steering prefix="${prefix}" publish_tf="false"/>
+            <xacro:omni_steering prefix="${prefix}" publish_tf="${publish_tf}"/>
         </xacro:if>
         <xacro:if value="${kinematic_model in ['skid','diff']}">
-            <xacro:skid_steering prefix="${prefix}" publish_tf="false"/>
+            <xacro:skid_steering prefix="${prefix}" publish_tf="${publish_tf}"/>
         </xacro:if>
         <xacro:if value="${kinematic_model == 'force_omni'}">
-            <xacro:ros_force_based_move prefix="${prefix}" publish_tf="true"/>
+            <xacro:ros_force_based_move prefix="${prefix}" publish_tf="${publish_tf}"/>
         </xacro:if>
         <xacro:if value="${kinematic_model == 'force_diff'}">
-            <xacro:ros_force_based_move_diff prefix="${prefix}" publish_tf="true"/>
+            <xacro:ros_force_based_move_diff prefix="${prefix}" publish_tf="${publish_tf}"/>
         </xacro:if>
         <xacro:if value="${enable_ros_control}">

File: summit_description/urdf/bases/summit_xl_hl_base.urdf.xacro (robot description, xacro)
@@ -1,60 +1,139 @@
 <?xml version="1.0"?>
-<robot name="summit_xl" xmlns:xacro="http://www.ros.org/wiki/xacro">
-	<xacro:include filename="$(find summit_description)/urdf/bases/summit_xl_base.gazebo.xacro" />
-  <xacro:macro name="summit_xl_hl_base" params="prefix publish_bf hq">
-  <!-- Robot mechanical and motor parameters -->
-  <xacro:property name="PI" value="3.1415926535897931"/>
-  <xacro:property name="wheel_width" value="0.175" />
-  <!-- BASE FOOTPRINT -->
-  <xacro:if value="${publish_bf}">
-    <link name="${prefix}base_footprint">
-      <visual>
+<robot name="summit_xl"
+  xmlns:xacro="http://www.ros.org/wiki/xacro">
+  <xacro:include filename="$(find summit_description)/urdf/bases/summit_xl_base.gazebo.xacro" />
+  <xacro:macro name="summit_xl_hl_base" params="prefix publish_bf hq virtual_platform_joints:=false *origin">
+    <!-- Robot mechanical and motor parameters -->
+    <xacro:property name="PI" value="3.1415926535897931"/>
+    <xacro:property name="wheel_width" value="0.175" />
+    <!-- BASE FOOTPRINT -->
+    <xacro:if value="${publish_bf}">
+      <link name="${prefix}base_footprint">
+        <visual>
           <origin xyz="0 0 0" rpy="0 0 0" />
           <geometry>
-             <box size="0.001 0.001 0.001" />
+            <box size="0.001 0.001 0.001" />
           </geometry>
-      </visual>
+        </visual>
+        <inertial>
+          <mass value="155.0" />
+          <origin xyz="0 0 0" />
+          <inertia ixx="230.391" ixy="0.004" ixz="0.0" iyy="236.853" iyz="0.0" izz="236.125" />
+        </inertial>
+      </link>
+      <joint name="${prefix}base_footprint_joint" type="fixed">
+        <origin xyz="0 0 ${wheel_radius}" rpy="0 0 0" />
+        <!-- ${wheel_radius} property must be defined inside wheel description -->
+        <parent link="${prefix}base_footprint"/>
+        <child link="${prefix}base_link" />
+      </joint>
+    </xacro:if>
+    <!-- BASE_LINK -->
+    <link name="${prefix}base_link">
       <inertial>
         <mass value="155.0" />
         <origin xyz="0 0 0" />
-        <inertia  ixx="230.391" ixy="0.004"  ixz="0.0"  iyy="236.853"  iyz="0.0"  izz="236.125" />
+        <inertia ixx="230.391" ixy="0.004" ixz="0.0" iyy="236.853" iyz="0.0" izz="236.125" />
       </inertial>
+      <visual>
+        <origin xyz="0 0 0" rpy="0 0 0" />
+        <xacro:if value="${hq}">
+          <geometry>
+            <mesh filename="package://summit_description/meshes/bases/summit_xl_hl_chassis.dae"/>
+          </geometry>
+        </xacro:if>
+        <xacro:unless value="${hq}">
+          <geometry>
+            <mesh filename="package://summit_description/meshes/bases/summit_xl_hl_chassis.dae"/>
+          </geometry>
+        </xacro:unless>
+        <material name="darkgrey">
+          <color rgba="0.1 0.1 0.1 1"/>
+        </material>
+      </visual>
+      <collision>
+        <origin xyz="0 0 0" rpy="0 0 0 " />
+        <geometry>
+          <mesh filename="package://summit_description/meshes/bases/summit_xl_hl_chassis.dae"/>
+        </geometry>
+      </collision>
     </link>
-    <joint name="${prefix}base_footprint_joint" type="fixed">
-      <origin xyz="0 0 ${wheel_radius}" rpy="0 0 0" /> <!-- ${wheel_radius} property must be defined inside wheel description -->
-      <parent link="${prefix}base_footprint"/>
-      <child link="${prefix}base_link" />
-    </joint>
-  </xacro:if>
-  <!-- BASE_LINK -->
-  <link name="${prefix}base_link">
-    <inertial>
-      <mass value="155.0" />
-      <origin xyz="0 0 0" />
-      <inertia  ixx="230.391" ixy="0.004"  ixz="0.0"  iyy="236.853"  iyz="0.0"  izz="236.125" />
-    </inertial>
-    <visual>
-       <origin xyz="0 0 0" rpy="0 0 0" />
-       <xacro:if value="${hq}">
-       <geometry>
-	     <mesh filename="package://summit_description/meshes/bases/summit_xl_hl_chassis.dae"/>
-       </geometry>
-       </xacro:if>
-       <xacro:unless value="${hq}">
-       <geometry>
-	     <mesh filename="package://summit_description/meshes/bases/summit_xl_hl_chassis.dae"/>
-       </geometry>
-       </xacro:unless>
-       <material name="darkgrey">
-         <color rgba="0.1 0.1 0.1 1"/>
-       </material>
-    </visual>
-    <collision>
-       <origin xyz="0 0 0" rpy="0 0 0 " />
-       <geometry>
-         <mesh filename="package://summit_description/meshes/bases/summit_xl_hl_chassis.dae"/>
-       </geometry>
-    </collision>
-  </link>
+    <!-- Add Virtual Platform Joints in URDF -->
+    <xacro:if value="${virtual_platform_joints}">
+      <link name="${prefix}world">
+        <inertial>
+          <mass value="1.0" />
+          <origin xyz="0 0 0" />
+          <inertia ixx="1.0" ixy="0.004" ixz="0.0" iyy="1.0" iyz="0.0" izz="1.0" />
+        </inertial>
+      </link>
+      <!-- robot world -> prismatic (x) -> linear_1 -->
+      <link name="${prefix}platform_linear_1">
+        <inertial>
+          <mass value="1.0" />
+          <origin xyz="0 0 0" />
+          <inertia ixx="1.0" ixy="0.004" ixz="0.0" iyy="1.0" iyz="0.0" izz="1.0" />
+        </inertial>
+      </link>
+      <!-- linear_1 -> prismatic (y) -> linear_2 -->
+      <link name="${prefix}platform_linear_2">
+        <inertial>
+          <mass value="1.0" />
+          <origin xyz="0 0 0" />
+          <inertia ixx="1.0" ixy="0.004" ixz="0.0" iyy="1.0" iyz="0.0" izz="1.0" />
+        </inertial>
+      </link>
+      <joint name="${prefix}platform_prismatic_x" type="prismatic">
+        <xacro:insert_block name="origin" />
+        <parent link="${prefix}world"/>
+        <child link="${prefix}platform_linear_1" />
+        <axis xyz="1 0 0"/>
+        <limit lower="-500" upper="500" effort="200" velocity="5"/>
+      </joint>
+      <joint name="${prefix}platform_prismatic_y" type="prismatic">
+        <origin xyz="0 0 0" rpy="0 0 0" />
+        <parent link="${prefix}platform_linear_1"/>
+        <child link="${prefix}platform_linear_2" />
+        <axis xyz="0 1 0"/>
+        <limit lower="-500" upper="500" effort="200" velocity="5"/>
+      </joint>
+      <joint name="${prefix}platform_continuous_z" type="continuous">
+        <origin xyz="0 0 0" rpy="0 0 0" />
+        <parent link="${prefix}platform_linear_2"/>
+        <child link="${prefix}base_footprint" />
+        <axis xyz="0 0 1"/>
+        <limit lower="-500" upper="500" effort="200" velocity="5"/>
+      </joint>
+      <transmission name="${prefix}platform_prismatic_x_trans">
+        <type>transmission_interface/SimpleTransmission</type>
+        <joint name="${prefix}platform_prismatic_x">
+          <hardwareInterface>hardware_interface/PositionJointInterface</hardwareInterface>
+        </joint>
+        <actuator name="${prefix}platform_prismatic_x_actuator">
+          <hardwareInterface>hardware_interface/PositionJointInterface</hardwareInterface>
+          <mechanicalReduction>1</mechanicalReduction>
+        </actuator>
+      </transmission>
+      <transmission name="${prefix}platform_prismatic_y_trans">
+        <type>transmission_interface/SimpleTransmission</type>
+        <joint name="${prefix}platform_prismatic_y">
+          <hardwareInterface>hardware_interface/PositionJointInterface</hardwareInterface>
+        </joint>
+        <actuator name="${prefix}platform_prismatic_y_actuator">
+          <hardwareInterface>hardware_interface/PositionJointInterface</hardwareInterface>
+          <mechanicalReduction>1</mechanicalReduction>
+        </actuator>
+      </transmission>
+      <transmission name="${prefix}platform_continuous_z_trans">
+        <type>transmission_interface/SimpleTransmission</type>
+        <joint name="${prefix}platform_continuous_z">
+          <hardwareInterface>hardware_interface/PositionJointInterface</hardwareInterface>
+        </joint>
+        <actuator name="${prefix}platform_continuous_z_actuator">
+          <hardwareInterface>hardware_interface/PositionJointInterface</hardwareInterface>
+          <mechanicalReduction>1</mechanicalReduction>
+        </actuator>
+      </transmission>
+    </xacro:if>
   </xacro:macro>
 </robot>

File: summit_mico_description/robots/summit_mico_root.xacro (robot description, xacro)
@@ -13,5 +13,5 @@
             <xacro:property name="kin_mode" value="force_diff"/>
         </xacro:unless>
-        <xacro:summit_xl_robot prefix="${prefix}" kinematic_model="${kin_mode}" kinect="${camera}" mini_pc="true" enable_ros_control="false">
+        <xacro:summit_xl_robot prefix="${prefix}" kinematic_model="${kin_mode}" kinect="${camera}" mini_pc="true" enable_ros_control="false" publish_tf="false" virtual_platform_joints="true">
             <origin xyz="0 0 0" rpy="0 0 0"/>
         </xacro:summit_xl_robot>

Commit message: virtual joints and velocity interface

File: summit_description/robots/summit_xl_hl_root.urdf.xacro (robot description, xacro)
@@ -51,5 +51,5 @@
             <xacro:property name="wheel_radius" value="0.11" />
         </xacro:unless>
-        <xacro:summit_xl_hl_base prefix="${prefix}" publish_bf="true" hq="${hq}" virtual_platform_joints="${virtual_platform_joints}" >
+        <xacro:summit_xl_hl_base prefix="${prefix}" publish_bf="true" hq="${hq}" virtual_platform_joints="${virtual_platform_joints}">
             <xacro:insert_block name="origin" />
         </xacro:summit_xl_hl_base>
@@ -187,16 +187,18 @@
         </xacro:if>
         <!-- Gazebo ros control pluggins -->
-        <xacro:if value="${kinematic_model == 'omni'}">
-            <xacro:omni_steering prefix="${prefix}" publish_tf="${publish_tf}"/>
-        </xacro:if>
-        <xacro:if value="${kinematic_model in ['skid','diff']}">
-            <xacro:skid_steering prefix="${prefix}" publish_tf="${publish_tf}"/>
-        </xacro:if>
-        <xacro:if value="${kinematic_model == 'force_omni'}">
-            <xacro:ros_force_based_move prefix="${prefix}" publish_tf="${publish_tf}"/>
-        </xacro:if>
-        <xacro:if value="${kinematic_model == 'force_diff'}">
-            <xacro:ros_force_based_move_diff prefix="${prefix}" publish_tf="${publish_tf}"/>
-        </xacro:if>
+        <xacro:unless value="${virtual_platform_joints}">
+            <xacro:if value="${kinematic_model == 'omni'}">
+                <xacro:omni_steering prefix="${prefix}" publish_tf="${publish_tf}"/>
+            </xacro:if>
+            <xacro:if value="${kinematic_model in ['skid','diff']}">
+                <xacro:skid_steering prefix="${prefix}" publish_tf="${publish_tf}"/>
+            </xacro:if>
+            <xacro:if value="${kinematic_model == 'force_omni'}">
+                <xacro:ros_force_based_move prefix="${prefix}" publish_tf="${publish_tf}"/>
+            </xacro:if>
+            <xacro:if value="${kinematic_model == 'force_diff'}">
+                <xacro:ros_force_based_move_diff prefix="${prefix}" publish_tf="${publish_tf}"/>
+            </xacro:if>
+        </xacro:unless>
         <xacro:if value="${enable_ros_control}">
             <xacro:ros_control/>

File: summit_description/urdf/bases/summit_xl_hl_base.urdf.xacro (robot description, xacro)
@@ -89,5 +89,5 @@
         <child link="${prefix}platform_linear_1" />
         <axis xyz="1 0 0"/>
-        <limit lower="-500" upper="500" effort="200" velocity="5"/>
+        <limit lower="-500" upper="500" effort="500" velocity="5"/>
       </joint>
       <joint name="${prefix}platform_prismatic_y" type="prismatic">
@@ -96,5 +96,5 @@
         <child link="${prefix}platform_linear_2" />
         <axis xyz="0 1 0"/>
-        <limit lower="-500" upper="500" effort="200" velocity="5"/>
+        <limit lower="-500" upper="500" effort="500" velocity="5"/>
       </joint>
       <joint name="${prefix}platform_continuous_z" type="continuous">
@@ -103,13 +103,13 @@
         <child link="${prefix}base_footprint" />
         <axis xyz="0 0 1"/>
-        <limit lower="-500" upper="500" effort="200" velocity="5"/>
+        <limit lower="-500" upper="500" effort="1000" velocity="5"/>
       </joint>
       <transmission name="${prefix}platform_prismatic_x_trans">
         <type>transmission_interface/SimpleTransmission</type>
         <joint name="${prefix}platform_prismatic_x">
-          <hardwareInterface>hardware_interface/PositionJointInterface</hardwareInterface>
+          <hardwareInterface>hardware_interface/VelocityJointInterface</hardwareInterface>
         </joint>
         <actuator name="${prefix}platform_prismatic_x_actuator">
-          <hardwareInterface>hardware_interface/PositionJointInterface</hardwareInterface>
+          <hardwareInterface>hardware_interface/VelocityJointInterface</hardwareInterface>
           <mechanicalReduction>1</mechanicalReduction>
         </actuator>
@@ -118,8 +118,8 @@
         <type>transmission_interface/SimpleTransmission</type>
         <joint name="${prefix}platform_prismatic_y">
-          <hardwareInterface>hardware_interface/PositionJointInterface</hardwareInterface>
+          <hardwareInterface>hardware_interface/VelocityJointInterface</hardwareInterface>
         </joint>
         <actuator name="${prefix}platform_prismatic_y_actuator">
-          <hardwareInterface>hardware_interface/PositionJointInterface</hardwareInterface>
+          <hardwareInterface>hardware_interface/VelocityJointInterface</hardwareInterface>
           <mechanicalReduction>1</mechanicalReduction>
         </actuator>
@@ -128,8 +128,8 @@
         <type>transmission_interface/SimpleTransmission</type>
         <joint name="${prefix}platform_continuous_z">
-          <hardwareInterface>hardware_interface/PositionJointInterface</hardwareInterface>
+          <hardwareInterface>hardware_interface/VelocityJointInterface</hardwareInterface>
         </joint>
         <actuator name="${prefix}platform_continuous_z_actuator">
-          <hardwareInterface>hardware_interface/PositionJointInterface</hardwareInterface>
+          <hardwareInterface>hardware_interface/VelocityJointInterface</hardwareInterface>
           <mechanicalReduction>1</mechanicalReduction>
         </actuator>
