Commit message: minor modifications

File: summit_description/robots/summit_xl_hl_root.urdf.xacro (robot description, xacro)
@@ -57,14 +57,14 @@
         <xacro:if value="${kinematic_model in ['omni', 'force_omni']}">
             <!-- OMNI WHEELS -->
-            <xacro:omni_wheel prefix="${prefix}front_right" parent="${prefix}base_link" reflect="false" hq="true">
+            <xacro:omni_wheel prefix="${prefix}front_right" parent="${prefix}base_link" reflect="false" hq="true" virtual_platform_joints="${virtual_platform_joints}">
                 <origin xyz="${wheel_offset_x} -${wheel_offset_y} ${wheel_offset_z}" rpy="0 0 0"/>
             </xacro:omni_wheel>
-            <xacro:omni_wheel prefix="${prefix}front_left" parent="${prefix}base_link" reflect="true" hq="true">
+            <xacro:omni_wheel prefix="${prefix}front_left" parent="${prefix}base_link" reflect="true" hq="true" virtual_platform_joints="${virtual_platform_joints}">
                 <origin xyz="${wheel_offset_x} ${wheel_offset_y} ${wheel_offset_z}" rpy="0 0 0"/>
             </xacro:omni_wheel>
-            <xacro:omni_wheel prefix="${prefix}back_left" parent="${prefix}base_link" reflect="false" hq="true">
+            <xacro:omni_wheel prefix="${prefix}back_left" parent="${prefix}base_link" reflect="false" hq="true" virtual_platform_joints="${virtual_platform_joints}">
                 <origin xyz="-${wheel_offset_x} ${wheel_offset_y} ${wheel_offset_z}" rpy="0 0 0"/>
             </xacro:omni_wheel>
-            <xacro:omni_wheel prefix="${prefix}back_right" parent="${prefix}base_link" reflect="true" hq="true">
+            <xacro:omni_wheel prefix="${prefix}back_right" parent="${prefix}base_link" reflect="true" hq="true" virtual_platform_joints="${virtual_platform_joints}">
                 <origin xyz="-${wheel_offset_x} -${wheel_offset_y} ${wheel_offset_z}" rpy="0 0 0"/>
             </xacro:omni_wheel>
@@ -72,14 +72,14 @@
         <xacro:if value="${kinematic_model not in ['omni', 'force_omni']}">
             <!-- RUBBER WHEELS MIMIC-->
-            <xacro:rubber_wheel prefix="${prefix}front_right" parent="${prefix}base_link" reflect="false" hq="${hq}">
+            <xacro:rubber_wheel prefix="${prefix}front_right" parent="${prefix}base_link" reflect="false" hq="${hq}" virtual_platform_joints="${virtual_platform_joints}">
                 <origin xyz="${wheel_offset_x} -${wheel_offset_y} ${wheel_offset_z}" rpy="0 0 0"/>
             </xacro:rubber_wheel>
-            <xacro:rubber_wheel prefix="${prefix}front_left" parent="${prefix}base_link" reflect="true" hq="${hq}">
+            <xacro:rubber_wheel prefix="${prefix}front_left" parent="${prefix}base_link" reflect="true" hq="${hq}" virtual_platform_joints="${virtual_platform_joints}">
                 <origin xyz="${wheel_offset_x} ${wheel_offset_y} ${wheel_offset_z}" rpy="0 0 0"/>
             </xacro:rubber_wheel>
-            <xacro:rubber_wheel prefix="${prefix}back_left" parent="${prefix}base_link" reflect="true" hq="${hq}">
+            <xacro:rubber_wheel prefix="${prefix}back_left" parent="${prefix}base_link" reflect="true" hq="${hq}" virtual_platform_joints="${virtual_platform_joints}">
                 <origin xyz="-${wheel_offset_x} ${wheel_offset_y} ${wheel_offset_z}" rpy="0 0 0"/>
             </xacro:rubber_wheel>
-            <xacro:rubber_wheel prefix="${prefix}back_right" parent="${prefix}base_link" reflect="false" hq="${hq}">
+            <xacro:rubber_wheel prefix="${prefix}back_right" parent="${prefix}base_link" reflect="false" hq="${hq}" virtual_platform_joints="${virtual_platform_joints}">
                 <origin xyz="-${wheel_offset_x} -${wheel_offset_y} ${wheel_offset_z}" rpy="0 0 0"/>
             </xacro:rubber_wheel>

File: summit_description/urdf/bases/summit_xl_hl_base.urdf.xacro (robot description, xacro)
@@ -19,5 +19,5 @@
           <mass value="155.0" />
           <origin xyz="0 0 0" />
-          <inertia ixx="230.391" ixy="0.004" ixz="0.0" iyy="236.853" iyz="0.0" izz="236.125" />
+          <inertia ixx="230.391" ixy="0.004" ixz="0.0" iyy="236.853" iyz="0.0" izz="36.125" />
         </inertial>
       </link>
@@ -34,5 +34,5 @@
         <mass value="155.0" />
         <origin xyz="0 0 0" />
-        <inertia ixx="230.391" ixy="0.004" ixz="0.0" iyy="236.853" iyz="0.0" izz="236.125" />
+        <inertia ixx="230.391" ixy="0.004" ixz="0.0" iyy="236.853" iyz="0.0" izz="36.125" />
       </inertial>
       <visual>
@@ -89,5 +89,6 @@
         <child link="${prefix}platform_linear_1" />
         <axis xyz="1 0 0"/>
-        <limit lower="-500" upper="500" effort="500" velocity="5"/>
+        <limit lower="-500" upper="500" effort="1000" velocity="4"/>
+        <joint_properties damping="0.1" friction="0.0"/>
       </joint>
       <joint name="${prefix}platform_prismatic_y" type="prismatic">
@@ -96,5 +97,6 @@
         <child link="${prefix}platform_linear_2" />
         <axis xyz="0 1 0"/>
-        <limit lower="-500" upper="500" effort="500" velocity="5"/>
+        <limit lower="-500" upper="500" effort="1000" velocity="4"/>
+        <joint_properties damping="0.1" friction="0.0"/>
       </joint>
       <joint name="${prefix}platform_continuous_z" type="continuous">
@@ -103,5 +105,6 @@
         <child link="${prefix}base_footprint" />
         <axis xyz="0 0 1"/>
-        <limit lower="-500" upper="500" effort="1000" velocity="5"/>
+        <limit lower="-500" upper="500" effort="1000" velocity="4"/>
+        <joint_properties damping="0.1" friction="0.0"/>
       </joint>
       <transmission name="${prefix}platform_prismatic_x_trans">

File: summit_description/urdf/wheels/omni_wheel.urdf.xacro (robot description, xacro)
@@ -1,4 +1,5 @@
 <?xml version="1.0"?>
-<robot name="wheel" xmlns:xacro="http://wiki.ros.org/xacro">
+<robot name="wheel"
+  xmlns:xacro="http://wiki.ros.org/xacro">
   <xacro:property name="M_PI" value="3.1415926535897931" />
   <!-- Wheels -->
@@ -6,19 +7,31 @@
   <xacro:property name="wheel_radius" value="0.127" />
   <xacro:property name="omni_wheel_height" value="0.087" />
-  <xacro:property name="omni_wheel_mass" value="6.5" /> <!-- in kg-->
+  <xacro:property name="omni_wheel_mass" value="6.5" />
+  <!-- in kg-->
   <xacro:macro name="cylinder_inertia" params="m r h">
-    <inertia  ixx="${m*(3*r*r+h*h)/12}" ixy = "0" ixz = "0"
-              iyy="${m*r*r/2}" iyz = "0"
-              izz="${m*(3*r*r+h*h)/12}" />
+    <inertia ixx="${m*(3*r*r+h*h)/12}" ixy = "0" ixz = "0" iyy="${m*r*r/2}" iyz = "0" izz="${m*(3*r*r+h*h)/12}" />
   </xacro:macro>
-  <xacro:macro name="omni_wheel" params="prefix parent *origin reflect hq">
-    <joint name="${prefix}_wheel_joint" type="continuous">
-      <parent link="${parent}"/>
-      <child link="${prefix}_wheel_link"/>
-      <xacro:insert_block name="origin" />
-      <axis xyz="0 1 0" rpy="0 0 0" />
-      <limit effort="100" velocity="100"/>
-      <joint_properties damping="0.0" friction="0.0"/>
-    </joint>
+  <xacro:macro name="omni_wheel" params="prefix parent *origin reflect hq virtual_platform_joints:=false">
+    <xacro:if value="${virtual_platform_joints}">
+      <xacro:property name="omni_wheel_radius" value="0.08" />
+      <joint name="${prefix}_wheel_joint" type="fixed">
+        <parent link="${parent}"/>
+        <child link="${prefix}_wheel_link"/>
+        <xacro:insert_block name="origin" />
+        <axis xyz="0 1 0" rpy="0 0 0" />
+        <limit effort="100" velocity="100"/>
+        <joint_properties damping="0.0" friction="0.0"/>
+      </joint>
+    </xacro:if>
+    <xacro:unless value="${virtual_platform_joints}">
+      <joint name="${prefix}_wheel_joint" type="continuous">
+        <parent link="${parent}"/>
+        <child link="${prefix}_wheel_link"/>
+        <xacro:insert_block name="origin" />
+        <axis xyz="0 1 0" rpy="0 0 0" />
+        <limit effort="100" velocity="100"/>
+        <joint_properties damping="0.0" friction="0.0"/>
+      </joint>
+    </xacro:unless>
     <link name="${prefix}_wheel_link">
       <visual>
@@ -34,5 +47,5 @@
               <mesh filename="package://summit_description/meshes/wheels/omni_wheel_2.dae" />
             </geometry>
-		  </xacro:unless>
+          </xacro:unless>
         </xacro:if>
         <xacro:unless value="${hq}">
@@ -43,20 +56,11 @@
         </xacro:unless>
         <material name="darkgrey">
-           <color rgba="0.2 0.2 0.2 1"/>
+          <color rgba="0.2 0.2 0.2 1"/>
         </material>
       </visual>
       <collision>
-				<origin xyz="0 0 0" rpy="${PI/2} 0 0" />
+        <origin xyz="0 0 0" rpy="${PI/2} 0 0" />
         <geometry>
           <sphere radius="${omni_wheel_radius}" />
-<!--
-          <xacro:if value="${reflect}">
-              <mesh filename="package://summit_xl_description/meshes/wheels/omni_wheel_1.dae" />
-          </xacro:if>
-          <xacro:unless value="${reflect}">
-              <mesh filename="package://summit_xl_description/meshes/wheels/omni_wheel_2.dae" />
-					</xacro:unless>
--->
-					<!--cylinder length="${omni_wheel_height}" radius="${omni_wheel_radius}" /-->
         </geometry>
       </collision>
@@ -64,25 +68,28 @@
         <mass value="${omni_wheel_mass}" />
         <origin xyz="0 0 0" />
-        <cylinder_inertia  m="${omni_wheel_mass}" r="${omni_wheel_radius}" h="${omni_wheel_height}" />
+        <cylinder_inertia m="${omni_wheel_mass}" r="${omni_wheel_radius}" h="${omni_wheel_height}" />
       </inertial>
     </link>
-    <!-- Transmission is important to link the joints and the controller (see summit_xl_control/config/summit_xl_control.yaml)-->
-    <transmission name="${prefix}_wheel_joint_trans">
-      <type>transmission_interface/SimpleTransmission</type>
-      <joint name="${prefix}_wheel_joint" >
-        <hardwareInterface>hardware_interface/VelocityJointInterface</hardwareInterface>
-      </joint>
-      <actuator name="${prefix}_wheel_joint_motor">
-         <mechanicalReduction>1</mechanicalReduction>
-      </actuator>
-    </transmission>
-    <gazebo reference="${prefix}_wheel_link">
-		<mu1 value="1.0"/>
-		<mu2 value="1.0"/>
-		<kp value="10000000.0" />
-		<kd value="1.0" />
-		<fdir1 value="1 0 0"/>
+    <xacro:unless value="${virtual_platform_joints}">
+      <!-- Transmission is important to link the joints and the controller (see summit_xl_control/config/summit_xl_control.yaml)-->
+      <transmission name="${prefix}_wheel_joint_trans">
+        <type>transmission_interface/SimpleTransmission</type>
+        <joint name="${prefix}_wheel_joint">
+          <hardwareInterface>hardware_interface/VelocityJointInterface</hardwareInterface>
+        </joint>
+        <actuator name="${prefix}_wheel_joint_motor">
+          <mechanicalReduction>1</mechanicalReduction>
+        </actuator>
+      </transmission>
+      <!-- <xacro:unless value="${virtual_platform_joints}"> -->
+      <gazebo reference="${prefix}_wheel_link">
+        <mu1 value="1.0"/>
+        <mu2 value="1.0"/>
+        <kp value="10000000.0" />
+        <kd value="1.0" />
+        <fdir1 value="1 0 0"/>
         <turnGravityOff>false</turnGravityOff>
-    </gazebo>
+      </gazebo>
+    </xacro:unless>
   </xacro:macro>
 </robot>

File: summit_description/urdf/wheels/rubber_wheel.urdf.xacro (robot description, xacro)
@@ -1,25 +1,36 @@
 <?xml version="1.0"?>
-<robot name="wheel" xmlns:xacro="http://wiki.ros.org/xacro">
+<robot name="wheel"
+  xmlns:xacro="http://wiki.ros.org/xacro">
   <xacro:property name="M_PI" value="3.1415926535897931" />
   <!-- Wheels -->
   <xacro:property name="rubber_wheel_radius" value="0.11" />
   <xacro:property name="wheel_radius" value="0.11" />
-  <xacro:property name="rubber_wheel_height" value="0.15" /> <!-- really is the wheel width -->
-  <xacro:property name="rubber_wheel_mass" value="6.5" /> <!-- in kg-->
+  <xacro:property name="rubber_wheel_height" value="0.15" />
+  <!-- really is the wheel width -->
+  <xacro:property name="rubber_wheel_mass" value="6.5" />
+  <!-- in kg-->
   <xacro:macro name="cylinder_inertia" params="m r h">
-    <inertia  ixx="${m*(3*r*r+h*h)/12}" ixy = "0" ixz = "0"
-              iyy="${m*r*r/2}" iyz = "0"
-              izz="${m*(3*r*r+h*h)/12}" />
+    <inertia ixx="${m*(3*r*r+h*h)/12}" ixy = "0" ixz = "0" iyy="${m*r*r/2}" iyz = "0" izz="${m*(3*r*r+h*h)/12}" />
   </xacro:macro>
-  <xacro:macro name="rubber_wheel" params="prefix parent *origin reflect hq">
-<!--WHEEL TIRE -->
-    <joint name="${prefix}_wheel_joint" type="continuous">
-      <parent link="${parent}"/>
-      <child link="${prefix}_wheel"/>
-      <xacro:insert_block name="origin" />
-      <axis xyz="0 1 0" rpy="0 0 0" />
-      <limit effort="100" velocity="100"/>
-      <joint_properties damping="0.0" friction="0.0"/>
-    </joint>
+  <xacro:macro name="rubber_wheel" params="prefix parent *origin reflect hq virtual_platform_joints:=false">
+    <!--WHEEL TIRE -->
+    <xacro:if value="${virtual_platform_joints}">
+      <xacro:property name="rubber_wheel_radius" value="0.05" />
+      <joint name="${prefix}_wheel_joint" type="fixed">
+        <parent link="${parent}"/>
+        <child link="${prefix}_wheel"/>
+        <xacro:insert_block name="origin" />
+      </joint>
+    </xacro:if>
+    <xacro:unless value="${virtual_platform_joints}">
+      <joint name="${prefix}_wheel_joint" type="continuous">
+        <parent link="${parent}"/>
+        <child link="${prefix}_wheel"/>
+        <xacro:insert_block name="origin" />
+        <axis xyz="0 1 0" rpy="0 0 0" />
+        <limit effort="100" velocity="100"/>
+        <joint_properties damping="0.0" friction="0.0"/>
+      </joint>
+    </xacro:unless>
     <link name="${prefix}_wheel">
       <visual>
@@ -28,13 +39,13 @@
           <origin xyz="0 0 0" rpy="0 0 0" />
           <geometry>
-						<xacro:if value="${reflect}">
-							<mesh filename="package://summit_description/meshes/wheels/rubber_wheel_left.dae" />
-						</xacro:if>
-						<xacro:unless value="${reflect}">
-							<mesh filename="package://summit_description/meshes/wheels/rubber_wheel_right.dae" />
-						</xacro:unless>
+            <xacro:if value="${reflect}">
+              <mesh filename="package://summit_description/meshes/wheels/rubber_wheel_left.dae" />
+            </xacro:if>
+            <xacro:unless value="${reflect}">
+              <mesh filename="package://summit_description/meshes/wheels/rubber_wheel_right.dae" />
+            </xacro:unless>
           </geometry>
         </xacro:if>
-       <!-- LOW RESOLUTION WHEELS -->
+        <!-- LOW RESOLUTION WHEELS -->
         <xacro:unless value="${hq}">
           <origin xyz="0 0 0" rpy="${M_PI/2} 0 0" />
@@ -45,5 +56,5 @@
       </visual>
       <collision>
-				<origin xyz="0 0 0" rpy="${M_PI/2} 0 0" />
+        <origin xyz="0 0 0" rpy="${M_PI/2} 0 0" />
         <geometry>
           <cylinder length="${rubber_wheel_height}" radius="${rubber_wheel_radius}" />
@@ -53,26 +64,28 @@
         <mass value="${rubber_wheel_mass}" />
         <origin xyz="0 0 0" />
-        <cylinder_inertia  m="${rubber_wheel_mass}" r="${rubber_wheel_radius}" h="${rubber_wheel_height}" />
+        <cylinder_inertia m="${rubber_wheel_mass}" r="${rubber_wheel_radius}" h="${rubber_wheel_height}" />
       </inertial>
     </link>
     <!-- Transmission is important to link the joints and the controller (see summit_xl_control/config/summit_xl_control.yaml)-->
-    <transmission name="${prefix}_wheel_joint_trans">
-      <type>transmission_interface/SimpleTransmission</type>
-      <joint name="${prefix}_wheel_joint">
-        <hardwareInterface>hardware_interface/VelocityJointInterface</hardwareInterface>
-      </joint>
-      <actuator name="${prefix}_wheel_joint_motor">
-        <mechanicalReduction>1</mechanicalReduction>
-        <motorTorqueConstant>20</motorTorqueConstant>
-      </actuator>
-     </transmission>
-    <gazebo reference="${prefix}_wheel">
-			<mu1 value="0.01"/>
-			<mu2 value="0.01"/>
-			<kp value="10000000.0" />
-			<kd value="1.0" />
-			<fdir1 value="1 0 0"/>
-      <turnGravityOff>false</turnGravityOff>
-    </gazebo>
+    <xacro:unless value="${virtual_platform_joints}">
+      <transmission name="${prefix}_wheel_joint_trans">
+        <type>transmission_interface/SimpleTransmission</type>
+        <joint name="${prefix}_wheel_joint">
+          <hardwareInterface>hardware_interface/VelocityJointInterface</hardwareInterface>
+        </joint>
+        <actuator name="${prefix}_wheel_joint_motor">
+          <mechanicalReduction>1</mechanicalReduction>
+          <motorTorqueConstant>20</motorTorqueConstant>
+        </actuator>
+      </transmission>
+      <gazebo reference="${prefix}_wheel">
+        <mu1 value="0.01"/>
+        <mu2 value="0.01"/>
+        <kp value="10000000.0" />
+        <kd value="1.0" />
+        <fdir1 value="1 0 0"/>
+        <turnGravityOff>false</turnGravityOff>
+      </gazebo>
+    </xacro:unless>
   </xacro:macro>
 </robot>

File: summit_mico_description/robots/summit_mico_csl.urdf.xacro (robot description, xacro)
@@ -7,6 +7,25 @@
     <xacro:arg name="enable_camera" default="true"/>
     <xacro:arg name="color" default="None"/>
+    <xacro:arg name="x" default="0.0"/>
+    <xacro:arg name="y" default="0.0"/>
+    <xacro:arg name="yaw" default="0.0"/>
     <!-- Import summit XL root -->
     <xacro:include filename="$(find summit_mico_description)/robots/summit_mico_root.xacro" />
-    <xacro:summit_mico prefix="$(arg prefix)" platform_mode="$(arg platform_mode)" arm_interface="$(arg arm_interface)" color="$(arg color)" camera="$(arg enable_camera)"/>
+    <xacro:property name="prefix_" value="$(arg prefix)"/>
+    <xacro:unless value="${prefix_ == ''}">
+        <link name="world"/>
+        <joint name="$(arg prefix)connect_word_and_summit_world" type="fixed">
+            <origin xyz="$(arg x) $(arg y) 0" rpy="0 0 $(arg yaw)"/>
+            <parent link="world" />
+            <child link="$(arg prefix)world" />
+        </joint>
+        <xacro:summit_mico prefix="$(arg prefix)" platform_mode="$(arg platform_mode)" arm_interface="$(arg arm_interface)" color="$(arg color)" camera="$(arg enable_camera)">
+            <origin xyz="0 0 0" rpy="0 0 0"/>
+        </xacro:summit_mico>
+    </xacro:unless>
+    <xacro:if value="${prefix_ == ''}">
+        <xacro:summit_mico prefix="$(arg prefix)" platform_mode="$(arg platform_mode)" arm_interface="$(arg arm_interface)" color="$(arg color)" camera="$(arg enable_camera)">
+            <origin xyz="$(arg x) $(arg y) 0" rpy="0 0 $(arg yaw)"/>
+        </xacro:summit_mico>
+    </xacro:if>
 </robot>

File: summit_mico_description/robots/summit_mico_root.xacro (robot description, xacro)
@@ -6,5 +6,5 @@
     <!--  -->
     <xacro:include filename="$(find mico_description)/urdf/mico2fingers.xacro" />
-    <xacro:macro name="summit_mico" params="prefix platform_mode:='omni' arm_interface:='velocity' color:='None' camera:=true">
+    <xacro:macro name="summit_mico" params="prefix *origin platform_mode:='omni' arm_interface:='velocity' color:='None' camera:=true">
         <xacro:if value="${platform_mode in ['omni', 'force_omni', 'force', 'Omni']}">
             <xacro:property name="kin_mode" value="force_omni"/>
@@ -14,5 +14,5 @@
         </xacro:unless>
         <xacro:summit_xl_robot prefix="${prefix}" kinematic_model="${kin_mode}" kinect="${camera}" mini_pc="true" enable_ros_control="false" publish_tf="false" virtual_platform_joints="true">
-            <origin xyz="3 0 0" rpy="0 0 0"/>
+            <xacro:insert_block name="origin" />
         </xacro:summit_xl_robot>
         <!-- <link name="world">
