Commit message: update ros controllers and ns

File: mico_description/urdf/kinova_common.xacro (robot description, xacro)
@@ -51,5 +51,5 @@
         <limit effort="${joint_torque_limit}" velocity="${joint_velocity_limit}" lower="${joint_lower_limit}" upper="${joint_upper_limit}"/>
         <origin xyz="${joint_origin_xyz}" rpy="${joint_origin_rpy}"/>
-        <dynamics damping="0.0" friction="0.0"/>
+        <dynamics damping="20.0" friction="0.0"/>
      </joint>
    <xacro:unless value="${fixed}">
@@ -57,8 +57,10 @@
         <type>transmission_interface/SimpleTransmission</type>
         <joint name="${joint_name}">
-          <hardwareInterface>hardware_interface/EffortJointInterface</hardwareInterface>
+          <!--<hardwareInterface>hardware_interface/EffortJointInterface</hardwareInterface>-->
+          <hardwareInterface>hardware_interface/VelocityJointInterface</hardwareInterface>
         </joint>
         <actuator name="${joint_name}_actuator">
-          <hardwareInterface>hardware_interface/EffortJointInterface</hardwareInterface>
+          <!-- <hardwareInterface>hardware_interface/EffortJointInterface</hardwareInterface> -->
+          <hardwareInterface>hardware_interface/VelocityJointInterface</hardwareInterface>
         <mechanicalReduction>160</mechanicalReduction>
         </actuator>
@@ -112,8 +114,10 @@
 					<type>transmission_interface/SimpleTransmission</type>
 					<joint name="${prefix}joint_finger_${finger_number}">
-					  <hardwareInterface>EffortJointInterface</hardwareInterface>
+                      <!-- <hardwareInterface>EffortJointInterface</hardwareInterface> -->
+                      <hardwareInterface>hardware_interface/VelocityJointInterface</hardwareInterface>
 					</joint>
 					<actuator name="${prefix}joint_finger_${finger_number}_actuator">
-					<hardwareInterface>EffortJointInterface</hardwareInterface>
+                    <!-- <hardwareInterface>EffortJointInterface</hardwareInterface> -->
+                    <hardwareInterface>hardware_interface/VelocityJointInterface</hardwareInterface>
 					<mechanicalReduction>1</mechanicalReduction>
 					</actuator>

File: mico_description/urdf/mico2fingers.xacro (robot description, xacro)
@@ -7,5 +7,4 @@
     xmlns:body="http://playerstage.sourceforge.net/gazebo/xmlschema/#body"
     xmlns:geom="http://playerstage.sourceforge.net/gazebo/xmlschema/#geom"
-    xmlns:joint="http://playerstage.sourceforge.net/gazebo/xmlschema/#joint"
     xmlns:controller="http://playerstage.sourceforge.net/gazebo/xmlschema/#controller"
     xmlns:interface="http://playerstage.sourceforge.net/gazebo/xmlschema/#interface"
@@ -103,4 +102,5 @@
     <xacro:property name="joint_end_effector_origin_rpy" value="${J_PI} 0 ${J_PI/2}" />
     <xacro:macro name="mico2fingers" params="base_parent prefix:=mico">
+        <xacro:gazebo_config robot_namespace="${prefix}"/>
         <xacro:kinova_armlink link_name="${prefix}_link_base" link_mesh="${link_base_mesh}" mesh_no="${link_base_mesh_no}"/>
         <xacro:kinova_armjoint joint_name="${prefix}_joint_base" type="${joint_base_type}" parent="${base_parent}" child="${prefix}_link_base" joint_axis_xyz="${joint_base_axis_xyz}" joint_origin_xyz="${joint_base_origin_xyz}" joint_origin_rpy="${joint_base_origin_rpy}" joint_lower_limit="0" joint_upper_limit="0" joint_velocity_limit="0" joint_torque_limit="0" fixed="true"/>
@@ -119,5 +119,5 @@
         <xacro:kinova_virtual_link link_name="${prefix}_end_effector"/>
         <xacro:kinova_virtual_joint joint_name="${prefix}_joint_end_effector" type="${joint_end_effector_type}" parent="${prefix}_link_6" child="${prefix}_end_effector" joint_axis_xyz="${joint_end_effector_axis_xyz}" joint_origin_xyz="${joint_end_effector_origin_xyz}" joint_origin_rpy="${joint_end_effector_origin_rpy}" joint_lower_limit="0" joint_upper_limit="0"/>
-<xacro:kinova_2fingers link_hand="${prefix}_link_6" prefix="${prefix}_"/>
+        <xacro:kinova_2fingers link_hand="${prefix}_link_6" prefix="${prefix}_"/>
     </xacro:macro>
 </root>

File: summit_description/urdf/bases/summit_xl_base.gazebo.xacro (robot description, xacro)
@@ -38,8 +38,8 @@
 		<gazebo>
 	    <plugin name="omni_steering" filename="libgazebo_ros_planar_move.so">
-	      <commandTopic>/summit_xl_control/cmd_vel</commandTopic>
-	      <odometryTopic>/odom</odometryTopic>
+		  <commandTopic>robotnik_base_control/cmd_vel</commandTopic>
+		  <odometryTopic>robotnik_base_control/odom</odometryTopic>
 	      <odometryFrame>odom</odometryFrame>
-	      <odometryRate>20.0</odometryRate>
+	      <odometryRate>50.0</odometryRate>
 	      <robotBaseFrame>base_footprint</robotBaseFrame>
 	    </plugin>

File: summit_mico_description/robots/summit_xl_hl_omni_mico.urdf.xacro (robot description, xacro)
@@ -68,9 +68,52 @@
     <parent link="base_link" />
 	<!--<origin xyz="0.19 0.0 0.17" rpy="0 ${15*PI/180} 0" />-->
-	<origin xyz="0.19 0.0 0.23" rpy="0 ${0.0*PI/180} 0" />
+	<origin xyz="0.22 0.0 0.30" rpy="0 ${0.0*PI/180} 0" />
   </joint>
   <property name="robot_root" value="root" />
   <xacro:mico2fingers  base_parent="${robot_root}" prefix="mico"/>
-	<!-- SENSORS -->
+ <!-- Collision Boxes for Modified Platform -->
+ <link name="mini_pc">
+	<visual>
+		<origin xyz="0.0 0.0 0.0" rpy="0.0 0.0 0.0" />
+		<geometry>
+		  <box size = "0.40 0.37 0.14"/>
+		</geometry>
+		<material name="Black" />
+  	</visual>
+  <collision>
+	<origin xyz="0.0 0.0 0.0" rpy="0.0 0.0 0.0" />
+	<geometry>
+	  <box size = "0.40 0.37 0.14"/>
+	</geometry>
+  </collision>
+</link>
+<link name="rgbd_camera">
+	<visual>
+		<origin xyz="0.0 0.0 0.0" rpy="0.0 0.0 0.0" />
+		<geometry>
+		  <box size = "0.10 0.26 0.60"/>
+		</geometry>
+		<material name="Black" />
+  	</visual>
+  <collision>
+	<origin xyz="0.0 0.0 0.0" rpy="0.0 0.0 0.0" />
+	<geometry>
+	  <box size = "0.10 0.26 0.60"/>
+	</geometry>
+  </collision>
+</link>
+<joint name="mini_pc_and_summit" type="fixed">
+    <child link="mini_pc" />
+    <parent link="base_link" />
+	<!--<origin xyz="0.19 0.0 0.17" rpy="0 ${15*PI/180} 0" />-->
+	<origin xyz="-0.1 0.0 0.30" rpy="0 ${0.0*PI/180} 0" />
+</joint>
+<joint name="rgbd_and_summit" type="fixed">
+    <child link="rgbd_camera" />
+    <parent link="base_link" />
+	<!--<origin xyz="0.19 0.0 0.17" rpy="0 ${15*PI/180} 0" />-->
+	<origin xyz="-0.3 0.0 0.60" rpy="0 ${0.0*PI/180} 0" />
+</joint>
+  <!-- SENSORS -->
   <!-- Hokuyo laser sensors can be parametized with min_angle and max_angle e.g: -->
   <!--xacro:sensor_hokuyo_utm30lx name="hokuyo_base" parent="base_link" min_angle="2.35" max_angle="-2.35"-->
