Commit message: update summit files

File: mico_description/urdf/kinova_common.xacro (robot description, xacro)
@@ -1,134 +1,140 @@
 <?xml version="1.0"?>
 <root xmlns:xi="http://www.w3.org/2001/XInclude"
-	xmlns:gazebo="http://playerstage.sourceforge.net/gazebo/xmlschema/#gz"
-    xmlns:model="http://playerstage.sourceforge.net/gazebo/xmlschema/#model"
-	xmlns:sensor="http://playerstage.sourceforge.net/gazebo/xmlschema/#sensor"
-	xmlns:body="http://playerstage.sourceforge.net/gazebo/xmlschema/#body"
-    xmlns:geom="http://playerstage.sourceforge.net/gazebo/xmlschema/#geom"
-    xmlns:joint="http://playerstage.sourceforge.net/gazebo/xmlschema/#joint"
-	xmlns:controller="http://playerstage.sourceforge.net/gazebo/xmlschema/#controller"
-	xmlns:interface="http://playerstage.sourceforge.net/gazebo/xmlschema/#interface"
-	xmlns:rendering="http://playerstage.sourceforge.net/gazebo/xmlschema/#rendering"
-    xmlns:renderable="http://playerstage.sourceforge.net/gazebo/xmlschema/#renderable"
-    xmlns:physics="http://playerstage.sourceforge.net/gazebo/xmlschema/#physics"
-	xmlns:xacro="http://www.ros.org/wiki/xacro">
-<xacro:include filename="$(find mico_description)/urdf/kinova_inertial.xacro" />
-    <property name="J_PI" value="3.1415926535897931" />
-    <xacro:macro name="kinova_armlink" params="link_name link_mesh ring_mesh:=ring_big use_ring_mesh:=false mesh_no">
-        <link name="${link_name}">
-            <visual>
-                <geometry>
-                    <mesh
-                        filename="package://mico_description/meshes/${link_mesh}.dae"/>
-                </geometry>
-                <material name="carbon_fiber">
-                    <color rgba="0.792156862745098 0.819607843137255 0.933333333333333 1" />
-                </material>
-            </visual>
-	    <!-- Adding ring to the model -->
-	         <xacro:if value="${use_ring_mesh}">
-	           <visual>
-                <geometry>
-                    <mesh
-                        filename="package://mico_description/meshes/${ring_mesh}.STL"/>
-                </geometry>
-             </visual>
-	    </xacro:if>
-            <collision>
-                <geometry>
-                    <mesh
-                        filename="package://mico_description/meshes/${link_mesh}.dae"/>
-                </geometry>
-            </collision>
-						<xacro:kinova_inertial mesh_no="${mesh_no}"/>
-      </link>
-    </xacro:macro>
-  <xacro:macro name="kinova_armjoint" params="joint_name type parent child joint_axis_xyz joint_origin_xyz joint_origin_rpy joint_lower_limit joint_upper_limit joint_velocity_limit joint_torque_limit fixed:=false">
+  xmlns:gazebo="http://playerstage.sourceforge.net/gazebo/xmlschema/#gz"
+  xmlns:model="http://playerstage.sourceforge.net/gazebo/xmlschema/#model"
+  xmlns:sensor="http://playerstage.sourceforge.net/gazebo/xmlschema/#sensor"
+  xmlns:body="http://playerstage.sourceforge.net/gazebo/xmlschema/#body"
+  xmlns:geom="http://playerstage.sourceforge.net/gazebo/xmlschema/#geom"
+  xmlns:joint="http://playerstage.sourceforge.net/gazebo/xmlschema/#joint"
+  xmlns:controller="http://playerstage.sourceforge.net/gazebo/xmlschema/#controller"
+  xmlns:interface="http://playerstage.sourceforge.net/gazebo/xmlschema/#interface"
+  xmlns:rendering="http://playerstage.sourceforge.net/gazebo/xmlschema/#rendering"
+  xmlns:renderable="http://playerstage.sourceforge.net/gazebo/xmlschema/#renderable"
+  xmlns:physics="http://playerstage.sourceforge.net/gazebo/xmlschema/#physics"
+  xmlns:xacro="http://www.ros.org/wiki/xacro">
+  <xacro:include filename="$(find kinova_description)/urdf/kinova_inertial.xacro" />
+  <xacro:property name="J_PI" value="3.1415926535897931" />
+  <xacro:macro name="kinova_armlink" params="link_name link_mesh ring_mesh:=ring_big use_ring_mesh:=false mesh_no">
+    <link name="${link_name}">
+      <visual>
+        <geometry>
+          <mesh filename="package://kinova_description/meshes/${link_mesh}.dae"/>
+        </geometry>
+        <material name="carbon_fiber">
+          <color rgba="0.792156862745098 0.819607843137255 0.933333333333333 1" />
+        </material>
+      </visual>
+      <!-- Adding ring to the model -->
+      <xacro:if value="${use_ring_mesh}">
+        <visual>
+          <geometry>
+            <mesh filename="package://kinova_description/meshes/${ring_mesh}.dae"/>
+          </geometry>
+        </visual>
+      </xacro:if>
+      <collision>
+        <geometry>
+          <mesh filename="package://kinova_description/meshes/${link_mesh}.dae"/>
+        </geometry>
+      </collision>
+      <xacro:kinova_inertial mesh_no="${mesh_no}"/>
+    </link>
+  </xacro:macro>
+  <xacro:macro name="kinova_armjoint" params="joint_name type parent child joint_axis_xyz joint_origin_xyz joint_origin_rpy joint_lower_limit joint_upper_limit joint_velocity_limit joint_torque_limit fixed:=false interface:=effort">
     <joint name="${joint_name}" type="${type}">
-        <parent link="${parent}"/>
-        <child link="${child}"/>
-        <axis xyz="${joint_axis_xyz}"/>
-        <limit effort="${joint_torque_limit}" velocity="${joint_velocity_limit}" lower="${joint_lower_limit}" upper="${joint_upper_limit}"/>
-        <origin xyz="${joint_origin_xyz}" rpy="${joint_origin_rpy}"/>
-        <dynamics damping="20.0" friction="0.0"/>
-     </joint>
-   <xacro:unless value="${fixed}">
-     <transmission name="${joint_name}_trans">
-        <type>transmission_interface/SimpleTransmission</type>
-        <joint name="${joint_name}">
-          <!--<hardwareInterface>hardware_interface/EffortJointInterface</hardwareInterface>-->
-          <hardwareInterface>hardware_interface/VelocityJointInterface</hardwareInterface>
-        </joint>
-        <actuator name="${joint_name}_actuator">
-          <!-- <hardwareInterface>hardware_interface/EffortJointInterface</hardwareInterface> -->
-          <hardwareInterface>hardware_interface/VelocityJointInterface</hardwareInterface>
-        <mechanicalReduction>160</mechanicalReduction>
-        </actuator>
-     </transmission>
-     <!--For torque sensing in simulation-->
-     <gazebo reference="${joint_name}">
-        <provideFeedback>true</provideFeedback>
-      </gazebo>
-      <gazebo>
-        <plugin name="ft_sensor" filename="libgazebo_ros_ft_sensor.so">
-          <updateRate>30.0</updateRate>
-          <topicName>${joint_name}_ft_sensor_topic</topicName>
-          <jointName>${joint_name}</jointName>
-        </plugin>
-      </gazebo>
-     </xacro:unless>
-</xacro:macro>
-    <xacro:macro name="kinova_virtual_link" params="link_name">
-        <link name="${link_name}">
-            <visual>
-                <geometry>
-                    <box size = "0.01 0.01 0.01"/>
-                </geometry>
-            </visual>
-            <collision>
-                <geometry>
-                    <box size = "0.01 0.01 0.01"/>
-                </geometry>
-            </collision>
-        </link>
-    </xacro:macro>
-    <xacro:macro name="kinova_virtual_joint" params="joint_name type parent child joint_axis_xyz joint_origin_xyz joint_origin_rpy joint_lower_limit joint_upper_limit">
+      <parent link="${parent}"/>
+      <child link="${child}"/>
+      <axis xyz="${joint_axis_xyz}"/>
+      <limit effort="${joint_torque_limit}" velocity="${joint_velocity_limit}" lower="${joint_lower_limit}" upper="${joint_upper_limit}"/>
+      <origin xyz="${joint_origin_xyz}" rpy="${joint_origin_rpy}"/>
+      <dynamics damping="0.2" friction="0.1"/>
+    </joint>
+    <xacro:unless value="${fixed}">
+      <xacro:if value="${interface=='position'}">
+        <transmission name="${joint_name}_trans">
+          <type>transmission_interface/SimpleTransmission</type>
+          <joint name="${joint_name}">
+            <hardwareInterface>hardware_interface/PositionJointInterface</hardwareInterface>
+          </joint>
+          <actuator name="${joint_name}_actuator">
+            <hardwareInterface>hardware_interface/PositionJointInterface</hardwareInterface>
+          </actuator>
+        </transmission>
+      </xacro:if>
+      <xacro:if value="${interface == 'effort'}">
+        <transmission name="${joint_name}_trans">
+          <type>transmission_interface/SimpleTransmission</type>
+          <joint name="${joint_name}">
+            <hardwareInterface>hardware_interface/EffortJointInterface</hardwareInterface>
+          </joint>
+          <actuator name="${joint_name}_actuator">
+            <hardwareInterface>hardware_interface/EffortJointInterface</hardwareInterface>
+            <mechanicalReduction>1</mechanicalReduction>
+          </actuator>
+        </transmission>
+      </xacro:if>
+      <xacro:if value="${interface == 'velocity'}">
+        <transmission name="${joint_name}_trans">
+          <type>transmission_interface/SimpleTransmission</type>
+          <joint name="${joint_name}">
+            <hardwareInterface>hardware_interface/VelocityJointInterface</hardwareInterface>
+          </joint>
+          <actuator name="${joint_name}_actuator">
+            <hardwareInterface>hardware_interface/VelocityJointInterface</hardwareInterface>
+            <mechanicalReduction>1</mechanicalReduction>
+          </actuator>
+        </transmission>
+      </xacro:if>
+    </xacro:unless>
+  </xacro:macro>
+  <xacro:macro name="kinova_virtual_link" params="link_name">
+    <link name="${link_name}"/>
+  </xacro:macro>
+  <xacro:macro name="kinova_virtual_joint" params="joint_name type parent child joint_axis_xyz joint_origin_xyz joint_origin_rpy joint_lower_limit joint_upper_limit">
     <joint name="${joint_name}" type="${type}">
-        <parent link="${parent}"/>
-        <child link="${child}"/>
-        <axis xyz="${joint_axis_xyz}"/>
-        <limit effort="2000" velocity="1" lower="${joint_lower_limit}" upper="${joint_upper_limit}"/>
-        <origin xyz="${joint_origin_xyz}" rpy="${joint_origin_rpy}"/>
-     </joint>
-    </xacro:macro>
-    <xacro:macro name="kinova_finger" params="prefix finger_number hand finger_origin_xyz finger_origin_rpy">
-        <xacro:kinova_armlink link_name="${prefix}link_finger_${finger_number}" link_mesh="finger_proximal" mesh_no="57"/>
-        <joint name="${prefix}joint_finger_${finger_number}" type="revolute">
-            <parent link="${hand}"/>
-            <child link="${prefix}link_finger_${finger_number}"/>
-            <axis xyz="0 0 1"/>
-            <origin xyz="${finger_origin_xyz}" rpy="${finger_origin_rpy}"/>
-            <limit lower="0" upper="2" effort="2000" velocity="1"/>
-        </joint>
-		    <transmission name="${prefix}joint_finger_${finger_number}_trans">
-					<type>transmission_interface/SimpleTransmission</type>
-					<joint name="${prefix}joint_finger_${finger_number}">
-                      <!-- <hardwareInterface>EffortJointInterface</hardwareInterface> -->
-                      <hardwareInterface>hardware_interface/VelocityJointInterface</hardwareInterface>
-					</joint>
-					<actuator name="${prefix}joint_finger_${finger_number}_actuator">
-                    <!-- <hardwareInterface>EffortJointInterface</hardwareInterface> -->
-                    <hardwareInterface>hardware_interface/VelocityJointInterface</hardwareInterface>
-					<mechanicalReduction>1</mechanicalReduction>
-					</actuator>
-		    </transmission>
-        <xacro:kinova_armlink link_name="${prefix}link_finger_tip_${finger_number}" link_mesh="finger_distal" mesh_no="58"/>
-        <joint name="${prefix}joint_finger_tip_${finger_number}" type="fixed">
-            <parent link="${prefix}link_finger_${finger_number}"/>
-            <child link="${prefix}link_finger_tip_${finger_number}"/>
-            <axis xyz="0 0 1"/>
-            <origin xyz="0.044 -0.003 0" rpy="0 0 0"/>
-            <limit lower="0" upper="2" effort="2000" velocity="1"/>
-        </joint>
-    </xacro:macro>
+      <parent link="${parent}"/>
+      <child link="${child}"/>
+      <axis xyz="${joint_axis_xyz}"/>
+      <limit effort="20000" velocity="2" lower="${joint_lower_limit}" upper="${joint_upper_limit}"/>
+      <origin xyz="${joint_origin_xyz}" rpy="${joint_origin_rpy}"/>
+    </joint>
+  </xacro:macro>
+  <xacro:macro name="kinova_finger" params="prefix finger_number hand finger_origin_xyz finger_origin_rpy">
+    <xacro:kinova_armlink link_name="${prefix}link_finger_${finger_number}" link_mesh="finger_proximal" mesh_no="57"/>
+    <joint name="${prefix}joint_finger_${finger_number}" type="revolute">
+      <parent link="${hand}"/>
+      <child link="${prefix}link_finger_${finger_number}"/>
+      <axis xyz="0 0 1"/>
+      <origin xyz="${finger_origin_xyz}" rpy="${finger_origin_rpy}"/>
+      <limit lower="0" upper="1.51" effort="2" velocity="1"/>
+    </joint>
+    <transmission name="${prefix}joint_finger_${finger_number}_trans">
+      <type>transmission_interface/SimpleTransmission</type>
+      <joint name="${prefix}joint_finger_${finger_number}">
+        <hardwareInterface>hardware_interface/EffortJointInterface</hardwareInterface>
+      </joint>
+      <actuator name="${prefix}joint_finger_${finger_number}_actuator">
+        <hardwareInterface>hardware_interface/EffortJointInterface</hardwareInterface>
+        <mechanicalReduction>1</mechanicalReduction>
+      </actuator>
+    </transmission>
+    <xacro:kinova_armlink link_name="${prefix}link_finger_tip_${finger_number}" link_mesh="finger_distal" mesh_no="58"/>
+    <joint name="${prefix}joint_finger_tip_${finger_number}" type="revolute">
+      <parent link="${prefix}link_finger_${finger_number}"/>
+      <child link="${prefix}link_finger_tip_${finger_number}"/>
+      <axis xyz="0 0 1"/>
+      <origin xyz="0.044 -0.003 0" rpy="0 0 0"/>
+      <limit lower="0" upper="2" effort="2" velocity="1"/>
+    </joint>
+    <transmission name="${prefix}joint_finger_tip_${finger_number}_trans">
+      <type>transmission_interface/SimpleTransmission</type>
+      <joint name="${prefix}joint_finger_tip_${finger_number}">
+        <hardwareInterface>hardware_interface/EffortJointInterface</hardwareInterface>
+      </joint>
+      <actuator name="${prefix}joint_finger_tip_${finger_number}_actuator">
+        <hardwareInterface>hardware_interface/EffortJointInterface</hardwareInterface>
+        <mechanicalReduction>1</mechanicalReduction>
+      </actuator>
+    </transmission>
+  </xacro:macro>
 </root>

File: mico_description/urdf/kinova_inertial.xacro (robot description, xacro)
@@ -29,22 +29,23 @@
    finger_distal      58
 -->
+<xacro:property name="mass_mul" value="1.0" />
 <xacro:macro name="inertia_cylinder" params="mass height radius axis:=0">
   <!-- z Axis -->
   <xacro:unless value="${axis}">
-    <inertia  ixx="${0.083333 * mass * (3*radius*radius + height*height)}" ixy="0" ixz="0"
-              iyy="${0.083333 * mass * (3*radius*radius + height*height)}" iyz="0"
-              izz="${0.5*mass*radius*radius}" />
+    <inertia  ixx="1.0" ixy="0" ixz="0"
+              iyy="1.0" iyz="0"
+              izz="1.0" />
   </xacro:unless>
   <!-- y Axis -->
   <xacro:unless value="${axis-1}">
-   <inertia  ixx="${0.083333 * mass * (3*radius*radius + height*height)}" ixy="0" ixz="0"
-             iyy="${0.5*mass*radius*radius}"
-             izz="${0.083333 * mass * (3*radius*radius + height*height)}" iyz="0" />
+   <inertia  ixx="1.0" ixy="0" ixz="0"
+             iyy="1.0"
+             izz="1.0" iyz="0" />
   </xacro:unless>
   <!-- x Axis -->
   <xacro:unless value="${axis-2}">
-   <inertia  ixx="${0.5*mass*radius*radius}"
-             iyy="${0.083333 * mass * (3*radius*radius + height*height)}" iyz="0"
-             izz="${0.083333 * mass * (3*radius*radius + height*height)}" ixy="0" ixz="0" />
+   <inertia  ixx="1.0"
+             iyy="1.0" iyz="0"
+             izz="1.0" ixy="0" ixz="0" />
   </xacro:unless>
 </xacro:macro>
@@ -53,5 +54,5 @@
   <xacro:unless value="${mesh_no}">
     <inertial>
-        <mass value="0.46784" />
+        <mass value="${mass_mul*0.46784}" />
         <origin xyz="0 0 0.1255" rpy="0 0 0"/>
         <xacro:inertia_cylinder height="0.14"  radius = "0.04" mass="0.46784"/>
@@ -61,5 +62,5 @@
   <xacro:unless value="${mesh_no-1}">
     <inertial>
-        <mass value="0.7477" />
+        <mass value="${mass_mul*0.7477}" />
         <origin xyz="0 -0.002 -0.0605" />
         <xacro:inertia_cylinder height="0.14"  radius = "0.04" mass="0.7477"/>
@@ -69,5 +70,5 @@
   <xacro:unless value="${mesh_no-2}">
     <inertial>
-        <mass value="0.99" />
+        <mass value="${mass_mul*0.99}" />
         <origin xyz="0 -0.2065 -0.01" />
         <xacro:inertia_cylinder height="0.35"  radius = "0.04" mass="0.99" axis="1"/>
@@ -77,5 +78,5 @@
   <xacro:unless value="${mesh_no-3}">
     <inertial>
-        <mass value="0.6763" />
+        <mass value="${mass_mul*0.6763}" />
         <origin xyz="0 0.081 -0.0086" />
         <xacro:inertia_cylinder height="0.15"  radius = "0.03" mass="0.6763" axis="1"/>
@@ -85,5 +86,5 @@
   <xacro:unless value="${mesh_no-4}">
     <inertial>
-        <mass value="0.1785" />
+        <mass value="${mass_mul*0.426367}" />
         <origin xyz="0 -0.037 -0.0642" />
         <xacro:inertia_cylinder height="0.02"  radius = "0.04" mass="0.1785"/>
@@ -93,5 +94,5 @@
   <xacro:unless value="${mesh_no-5}">
     <inertial>
-        <mass value="0.85968" />
+        <mass value="${mass_mul*0.85968}" />
         <origin xyz="0 -0.145  -0.0076"/>
         <xacro:inertia_cylinder height="0.25"  radius = "0.03" mass="0.85968" axis="1"/>
@@ -101,5 +102,5 @@
   <xacro:unless value="${mesh_no-6}">
     <inertial>
-        <mass value="0.8447" />
+        <mass value="${mass_mul*0.8447}" />
         <origin xyz="0 -0.103563213 0" />
         <xacro:inertia_cylinder height="0.18"  radius = "0.03" mass="0.8447" axis="1"/>
@@ -109,5 +110,5 @@
   <xacro:unless value="${mesh_no-7}">
     <inertial>
-        <mass value="0.8447" />
+        <mass value="${mass_mul*0.8447}" />
         <origin xyz="0 0 -0.1022447445" />
         <xacro:inertia_cylinder height="0.18"  radius = "0.03" mass="0.8447"/>
@@ -117,5 +118,5 @@
   <xacro:unless value="${mesh_no-8}">
     <inertial>
-        <mass value="0.463" />
+        <mass value="${10*0.463}" />
         <origin xyz="0 0.0028848942 -0.0541932613" />
         <xacro:inertia_cylinder height="0.1"  radius = "0.02" mass="0.463"/>
@@ -125,5 +126,5 @@
   <xacro:unless value="${mesh_no-9}">
     <inertial>
-        <mass value="0.463" />
+        <mass value="${mass_mul*0.463}" />
         <origin xyz="0 0.0497208855 -0.0028562765" />
         <xacro:inertia_cylinder height="0.1"  radius = "0.02" mass="0.463" axis="1"/>
@@ -133,5 +134,5 @@
   <xacro:unless value="${mesh_no-10}">
     <inertial>
-        <mass value="0.606" />
+        <mass value="${mass_mul*0.606}" />
         <origin xyz="0 0.0463 -0.0065" />
         <xacro:inertia_cylinder height="0.08"  radius = "0.02" mass="0.606" axis="1"/>
@@ -141,5 +142,5 @@
   <xacro:unless value="${mesh_no - 55}">
     <inertial>
-        <mass value="0.727" />
+        <mass value="${mass_mul*0.99}" />
         <origin xyz="0 0 -0.06" />
         <xacro:inertia_cylinder height="0.03"  radius = "0.04" mass="0.727"/>
