Commit message: update summit files

File: summit_description/urdf/bases/summit_xl_base.gazebo.xacro (robot description, xacro)
@@ -1,67 +1,58 @@
 <?xml version="1.0"?>
 <robot xmlns:xacro="http://www.ros.org/wiki/xacro">
-  <!-- ros control plugin -->
-  <xacro:macro name="ros_control">
-    <gazebo>
-      <plugin name="ros_control" filename="libgazebo_ros_control.so">
-        <!--<robotNamespace>/summit_xl</robotNamespace>-->
-        <robotParam>robot_description</robotParam>
-        <controlPeriod>0.001</controlPeriod>
-	    <robotSimType>gazebo_ros_control/DefaultRobotHWSim</robotSimType>
-	    <legacyModeNS>true</legacyModeNS>
-      </plugin>
-    </gazebo>
+	<!-- ros control plugin -->
+	<xacro:macro name="ros_control">
+		<gazebo>
+			<plugin name="ros_control" filename="libgazebo_ros_control.so">
+				<!--<robotNamespace>/summit_xl</robotNamespace>-->
+				<robotParam>robot_description</robotParam>
+				<controlPeriod>0.001</controlPeriod>
+				<robotSimType>gazebo_ros_control/DefaultRobotHWSim</robotSimType>
+				<legacyModeNS>true</legacyModeNS>
+			</plugin>
+		</gazebo>
 	</xacro:macro>
-	<!-- skid steering plugin -->
-	<xacro:macro name="skid_steering" params="broadcastOdomTF">
-    <gazebo>
-      <plugin name="skid_steer_drive_controller" filename="libgazebo_ros_skid_steer_drive.so">
-			<!--<robotNamespace>/summit_xl</robotNamespace>-->
-		    <updateRate>100.0</updateRate>
-		    <leftFrontJoint>joint_front_left_wheel</leftFrontJoint>
-		    <rightFrontJoint>joint_front_right_wheel</rightFrontJoint>
-		    <leftRearJoint>joint_back_left_wheel</leftRearJoint>
-		    <rightRearJoint>joint_back_right_wheel</rightRearJoint>
-		    <!-- wheelSeparation>0.566</wheelSeparation --> <!-- real parameter value -->
-		    <wheelSeparation>1.5</wheelSeparation> <!-- works a bit better in Gazebo -->
-		    <wheelDiameter>0.234</wheelDiameter>
-		    <robotBaseFrame>base_footprint</robotBaseFrame>
-		    <torque>50</torque>
-		    <commandTopic>/summit_xl_control/cmd_vel</commandTopic>
-		    <odometryTopic>odom</odometryTopic>
-		    <odometryFrame>/odom</odometryFrame>
-		    <broadcastTF>${broadcastOdomTF}</broadcastTF>
-      </plugin>
-    </gazebo>
-  </xacro:macro>
-  <xacro:macro name="omni_steering">
+	<xacro:macro name="omni_steering" params="prefix publish_tf">
 		<gazebo>
-	    <plugin name="omni_steering" filename="libgazebo_ros_planar_move.so">
-		  <commandTopic>/summit_xl/robotnik_base_control/cmd_vel</commandTopic>
-		  <odometryTopic>/summit_xl/robotnik_base_control/odom</odometryTopic>
-	      <odometryFrame>odom</odometryFrame>
-	      <odometryRate>50.0</odometryRate>
-	      <robotBaseFrame>base_footprint</robotBaseFrame>
-	    </plugin>
-	  </gazebo>
-  </xacro:macro>
-  <xacro:macro name="ros_force_based_move" params="broadcastOdomTF">
-	  <gazebo>
-		 <plugin name="ros_force_based_move" filename="libgazebo_ros_force_based_move.so">
-			 <!--<robotNamespace>/summit_xl</robotNamespace>-->
-			 <commandTopic>/summit_xl_control/cmd_vel</commandTopic>
-			 <odometryTopic>/summit_xl/odom</odometryTopic>
-	         <odometryFrame>odom</odometryFrame>
-			 <yaw_velocity_p_gain>10000.0</yaw_velocity_p_gain>
-			 <x_velocity_p_gain>10000.0</x_velocity_p_gain>
-			 <y_velocity_p_gain>10000.0</y_velocity_p_gain>
-			 <robotBaseFrame>base_footprint</robotBaseFrame>
-			 <odometryRate>20.0</odometryRate>
-			 <publishOdometryTf>${broadcastOdomTF}</publishOdometryTf>
-		 </plugin>
-	  </gazebo>
-  </xacro:macro>
-  <gazebo reference="base_footprint">
-    <material>Gazebo/Green</material>
-  </gazebo>
+			<plugin name="omni_steering" filename="libgazebo_ros_planar_move.so">
+				<commandTopic>robotnik_base_control/cmd_vel</commandTopic>
+				<odometryTopic>robotnik_base_control/odom</odometryTopic>
+				<odometryFrame>${prefix}odom</odometryFrame>
+				<odometryRate>100.0</odometryRate>
+				<robotBaseFrame>${prefix}base_footprint</robotBaseFrame>
+				<publishTF>${publish_tf}</publishTF>
+			</plugin>
+		</gazebo>
+	</xacro:macro>
+	<xacro:macro name="skid_steering" params="prefix publish_tf">
+		<gazebo>
+			<plugin name="skid_steering" filename="libgazebo_ros_planar_move.so">
+				<commandTopic>robotnik_base_control/cmd_vel</commandTopic>
+				<odometryTopic>robotnik_base_control/odom</odometryTopic>
+				<odometryFrame>${prefix}odom</odometryFrame>
+				<odometryRate>100.0</odometryRate>
+				<robotBaseFrame>${prefix}base_footprint</robotBaseFrame>
+				<publishTF>${publish_tf}</publishTF>
+				<enableYAxis>false</enableYAxis>
+			</plugin>
+		</gazebo>
+	</xacro:macro>
+	<xacro:macro name="ros_force_based_move" params="publish_tf prefix">
+		<gazebo>
+			<plugin name="ros_force_based_move" filename="libgazebo_ros_force_based_move.so">
+				<commandTopic>robotnik_base_control/cmd_vel</commandTopic>
+				<odometryTopic>robotnik_base_control/odom</odometryTopic>
+				<odometryFrame>${prefix}odom</odometryFrame>
+				<yaw_velocity_p_gain>10000.0</yaw_velocity_p_gain>
+				<x_velocity_p_gain>10000.0</x_velocity_p_gain>
+				<y_velocity_p_gain>10000.0</y_velocity_p_gain>
+				<robotBaseFrame>${prefix}base_footprint</robotBaseFrame>
+				<odometryRate>100.0</odometryRate>
+				<publishOdometryTf>${publish_tf}</publishOdometryTf>
+			</plugin>
+		</gazebo>
+	</xacro:macro>
+	<gazebo reference="base_footprint">
+		<material>Gazebo/Green</material>
+	</gazebo>
 </robot>

File: summit_description/urdf/bases/summit_xl_hl_base.urdf.xacro (robot description, xacro)
@@ -2,5 +2,5 @@
 <robot name="summit_xl" xmlns:xacro="http://www.ros.org/wiki/xacro">
 	<xacro:include filename="$(find summit_description)/urdf/bases/summit_xl_base.gazebo.xacro" />
-  <xacro:macro name="summit_xl_hl_base" params="name publish_bf hq">
+  <xacro:macro name="summit_xl_hl_base" params="prefix publish_bf hq">
   <!-- Robot mechanical and motor parameters -->
   <xacro:property name="PI" value="3.1415926535897931"/>
@@ -8,5 +8,5 @@
   <!-- BASE FOOTPRINT -->
   <xacro:if value="${publish_bf}">
-    <link name="base_footprint">
+    <link name="${prefix}base_footprint">
       <visual>
           <origin xyz="0 0 0" rpy="0 0 0" />
@@ -15,17 +15,22 @@
           </geometry>
       </visual>
+      <inertial>
+        <mass value="155.0" />
+        <origin xyz="0 0 0" />
+        <inertia  ixx="230.391" ixy="0.004"  ixz="0.0"  iyy="236.853"  iyz="0.0"  izz="236.125" />
+      </inertial>
     </link>
-    <joint name="base_footprint_joint" type="fixed">
+    <joint name="${prefix}base_footprint_joint" type="fixed">
       <origin xyz="0 0 ${wheel_radius}" rpy="0 0 0" /> <!-- ${wheel_radius} property must be defined inside wheel description -->
-      <parent link="base_footprint"/>
-      <child link="base_link" />
+      <parent link="${prefix}base_footprint"/>
+      <child link="${prefix}base_link" />
     </joint>
   </xacro:if>
   <!-- BASE_LINK -->
-  <link name="base_link">
+  <link name="${prefix}base_link">
     <inertial>
-      <mass value="25.0" />
+      <mass value="155.0" />
       <origin xyz="0 0 0" />
-      <inertia  ixx="1.391" ixy="0.004"  ixz="0.0"  iyy="6.853"  iyz="0.0"  izz="6.125" />
+      <inertia  ixx="230.391" ixy="0.004"  ixz="0.0"  iyy="236.853"  iyz="0.0"  izz="236.125" />
     </inertial>
     <visual>

File: summit_description/urdf/wheels/omni_wheel.urdf.xacro (robot description, xacro)
@@ -1,9 +1,10 @@
 <?xml version="1.0"?>
-<robot name="wheel" xmlns:xacro="http://www.ros.org/wiki/xacro">
+<robot name="wheel" xmlns:xacro="http://wiki.ros.org/xacro">
   <xacro:property name="M_PI" value="3.1415926535897931" />
   <!-- Wheels -->
+  <xacro:property name="omni_wheel_radius" value="0.127" />
   <xacro:property name="wheel_radius" value="0.127" />
-  <xacro:property name="wheel_height" value="0.087" />
-  <xacro:property name="wheel_mass" value="6.5" /> <!-- in kg-->
+  <xacro:property name="omni_wheel_height" value="0.087" />
+  <xacro:property name="omni_wheel_mass" value="6.5" /> <!-- in kg-->
   <xacro:macro name="cylinder_inertia" params="m r h">
     <inertia  ixx="${m*(3*r*r+h*h)/12}" ixy = "0" ixz = "0"
@@ -12,7 +13,7 @@
   </xacro:macro>
   <xacro:macro name="omni_wheel" params="prefix parent *origin reflect hq">
-    <joint name="joint_${prefix}_wheel" type="continuous">
+    <joint name="${prefix}_wheel_joint" type="continuous">
       <parent link="${parent}"/>
-      <child link="${prefix}_wheel"/>
+      <child link="${prefix}_wheel_link"/>
       <xacro:insert_block name="origin" />
       <axis xyz="0 1 0" rpy="0 0 0" />
@@ -20,5 +21,5 @@
       <joint_properties damping="0.0" friction="0.0"/>
     </joint>
-    <link name="${prefix}_wheel">
+    <link name="${prefix}_wheel_link">
       <visual>
         <xacro:if value="${hq}">
@@ -38,5 +39,5 @@
           <origin xyz="0 0 0" rpy="0 0 0" />
           <geometry>
-            <sphere radius="${wheel_radius}" />
+            <sphere radius="${omni_wheel_radius}" />
           </geometry>
         </xacro:unless>
@@ -48,22 +49,20 @@
 				<origin xyz="0 0 0" rpy="${PI/2} 0 0" />
         <geometry>
-<!--
-          <sphere radius="${wheel_radius}" />
--->
+          <sphere radius="${omni_wheel_radius}" />
 <!--
           <xacro:if value="${reflect}">
-              <mesh filename="package://summit_description/meshes/wheels/omni_wheel_1.dae" />
+              <mesh filename="package://summit_xl_description/meshes/wheels/omni_wheel_1.dae" />
           </xacro:if>
           <xacro:unless value="${reflect}">
-              <mesh filename="package://summit_description/meshes/wheels/omni_wheel_2.dae" />
+              <mesh filename="package://summit_xl_description/meshes/wheels/omni_wheel_2.dae" />
 					</xacro:unless>
 -->
-					<cylinder length="${wheel_height}" radius="${wheel_radius}" />
+					<!--cylinder length="${omni_wheel_height}" radius="${omni_wheel_radius}" /-->
         </geometry>
       </collision>
       <inertial>
-        <mass value="${wheel_mass}" />
+        <mass value="${omni_wheel_mass}" />
         <origin xyz="0 0 0" />
-        <cylinder_inertia  m="${wheel_mass}" r="${wheel_radius}" h="${wheel_height}" />
+        <cylinder_inertia  m="${omni_wheel_mass}" r="${omni_wheel_radius}" h="${omni_wheel_height}" />
       </inertial>
     </link>
@@ -71,6 +70,6 @@
     <transmission name="${prefix}_wheel_joint_trans">
       <type>transmission_interface/SimpleTransmission</type>
-      <joint name="joint_${prefix}_wheel" >
-        <hardwareInterface>VelocityJointInterface</hardwareInterface>
+      <joint name="${prefix}_wheel_joint" >
+        <hardwareInterface>hardware_interface/VelocityJointInterface</hardwareInterface>
       </joint>
       <actuator name="${prefix}_wheel_joint_motor">
@@ -78,5 +77,5 @@
       </actuator>
     </transmission>
-    <gazebo reference="${prefix}_wheel">
+    <gazebo reference="${prefix}_wheel_link">
 		<mu1 value="1.0"/>
 		<mu2 value="1.0"/>

File: summit_description/urdf/wheels/rubber_wheel.urdf.xacro (robot description, xacro)
@@ -1,9 +1,10 @@
 <?xml version="1.0"?>
-<robot name="wheel" xmlns:xacro="http://www.ros.org/wiki/xacro">
+<robot name="wheel" xmlns:xacro="http://wiki.ros.org/xacro">
   <xacro:property name="M_PI" value="3.1415926535897931" />
   <!-- Wheels -->
-  <xacro:property name="wheel_radius" value="0.125" />
-  <xacro:property name="wheel_height" value="0.14" /> <!-- really is the wheel width -->
-  <xacro:property name="wheel_mass" value="6.5" /> <!-- in kg-->
+  <xacro:property name="rubber_wheel_radius" value="0.11" />
+  <xacro:property name="wheel_radius" value="0.11" />
+  <xacro:property name="rubber_wheel_height" value="0.15" /> <!-- really is the wheel width -->
+  <xacro:property name="rubber_wheel_mass" value="6.5" /> <!-- in kg-->
   <xacro:macro name="cylinder_inertia" params="m r h">
     <inertia  ixx="${m*(3*r*r+h*h)/12}" ixy = "0" ixz = "0"
@@ -13,5 +14,5 @@
   <xacro:macro name="rubber_wheel" params="prefix parent *origin reflect hq">
 <!--WHEEL TIRE -->
-    <joint name="joint_${prefix}_wheel" type="continuous">
+    <joint name="${prefix}_wheel_joint" type="continuous">
       <parent link="${parent}"/>
       <child link="${prefix}_wheel"/>
@@ -39,5 +40,5 @@
           <origin xyz="0 0 0" rpy="${M_PI/2} 0 0" />
           <geometry>
-            <cylinder length="${wheel_height}" radius="${wheel_radius}" />
+            <cylinder length="${rubber_wheel_height}" radius="${rubber_wheel_radius}" />
           </geometry>
         </xacro:unless>
@@ -46,11 +47,11 @@
 				<origin xyz="0 0 0" rpy="${M_PI/2} 0 0" />
         <geometry>
-          <cylinder length="${wheel_height}" radius="${wheel_radius}" />
+          <cylinder length="${rubber_wheel_height}" radius="${rubber_wheel_radius}" />
         </geometry>
       </collision>
       <inertial>
-        <mass value="${wheel_mass}" />
+        <mass value="${rubber_wheel_mass}" />
         <origin xyz="0 0 0" />
-        <cylinder_inertia  m="${wheel_mass}" r="${wheel_radius}" h="${wheel_height}" />
+        <cylinder_inertia  m="${rubber_wheel_mass}" r="${rubber_wheel_radius}" h="${rubber_wheel_height}" />
       </inertial>
     </link>
@@ -58,6 +59,6 @@
     <transmission name="${prefix}_wheel_joint_trans">
       <type>transmission_interface/SimpleTransmission</type>
-      <joint name="joint_${prefix}_wheel">
-        <hardwareInterface>VelocityJointInterface</hardwareInterface>
+      <joint name="${prefix}_wheel_joint">
+        <hardwareInterface>hardware_interface/VelocityJointInterface</hardwareInterface>
       </joint>
       <actuator name="${prefix}_wheel_joint_motor">

File: summit_mico_description/robots/summit_xl_hl_omni_mico.urdf.xacro (robot description, xacro)
@@ -1,4 +1,5 @@
 <?xml version="1.0"?>
-<robot name="summit_xl_hl_mico" xmlns:xacro="http://www.ros.org/wiki/xacro">
+<robot name="summit_xl_hl_mico"
+	xmlns:xacro="http://www.ros.org/wiki/xacro">
 	<!-- ***************** -->
 	<!-- Imported elements -->
@@ -18,5 +19,6 @@
 	<xacro:property name="PI" value="3.1415926535897931"/>
 	<!-- Wheel parameters -->
-	<xacro:property name="wheel_offset_x" value="0.229" />    <!-- x,y,z in translation from base_link to the center of the wheel -->
+	<xacro:property name="wheel_offset_x" value="0.229" />
+	<!-- x,y,z in translation from base_link to the center of the wheel -->
 	<xacro:property name="wheel_offset_y" value="0.234" />
 	<xacro:property name="wheel_offset_z" value="0.0" />
@@ -28,8 +30,8 @@
 	<!-- Here we create the robot elements using the xacro:macros imported at the beggining of this file -->
 	<!-- Summit XL HL base -->
-  <xacro:summit_xl_hl_base name="summit_xl" publish_bf="true" hq="${hq}"/>
-  <!-- Gazebo ros control pluggins -->
-  <xacro:ros_control/>
-  <!-- Gazebo omni steering plugin -->
+	<xacro:summit_xl_hl_base name="summit_xl" publish_bf="true" hq="${hq}"/>
+	<!-- Gazebo ros control pluggins -->
+	<xacro:ros_control/>
+	<!-- Gazebo omni steering plugin -->
 	<xacro:omni_steering/>
 	<!-- WHEELS -->
@@ -48,105 +50,105 @@
 	<!-- ARM KINOVA MICO2 -->
 	<!-- Load Mico Arm -->
-<!--	<xacro:mico_arm parent="base_link" xyz="0.19 0 0.17" rpy="0 ${15*PI/180} 0"/>-->
-  <link name="root">
-      <visual>
-          <origin xyz="0.0 0.0 0.0" rpy="0.0 0.0 0.0" />
-          <geometry>
-            <box size = "0.01 0.01 0.01"/>
-          </geometry>
-    <!--<material name="Black" /> -->
-    </visual>
-    <collision>
-      <origin xyz="0.0 0.0 0.0" rpy="0.0 0.0 0.0" />
-      <geometry>
-        <box size = "0.01 0.01 0.01"/>
-      </geometry>
-    </collision>
-  </link>
-  <joint name="connect_root_and_summit" type="fixed">
-    <child link="root" />
-    <parent link="base_link" />
-	<!--<origin xyz="0.19 0.0 0.17" rpy="0 ${15*PI/180} 0" />-->
-	<origin xyz="0.22 0.0 0.30" rpy="0 ${0.0*PI/180} 0" />
-  </joint>
-  <property name="robot_root" value="root" />
-  <xacro:mico2fingers  base_parent="${robot_root}" prefix="mico"/>
- <!-- Collision Boxes for Modified Platform -->
- <link name="mini_pc">
-	<visual>
-		<origin xyz="0.0 0.0 0.0" rpy="0.0 0.0 0.0" />
-		<geometry>
-		  <box size = "0.40 0.37 0.14"/>
-		</geometry>
-		<material name="Black" />
-  	</visual>
-  <collision>
-	<origin xyz="0.0 0.0 0.0" rpy="0.0 0.0 0.0" />
-	<geometry>
-	  <box size = "0.40 0.37 0.14"/>
-	</geometry>
-  </collision>
-</link>
-<link name="rgbd_camera">
-	<visual>
-		<origin xyz="0.0 0.0 0.0" rpy="0.0 0.0 0.0" />
-		<geometry>
-		  <box size = "0.10 0.26 0.60"/>
-		</geometry>
-		<material name="Black" />
-  	</visual>
-  <collision>
-	<origin xyz="0.0 0.0 0.0" rpy="0.0 0.0 0.0" />
-	<geometry>
-	  <box size = "0.10 0.26 0.60"/>
-	</geometry>
-  </collision>
-</link>
-<joint name="mini_pc_and_summit" type="fixed">
-    <child link="mini_pc" />
-    <parent link="base_link" />
-	<!--<origin xyz="0.19 0.0 0.17" rpy="0 ${15*PI/180} 0" />-->
-	<origin xyz="-0.1 0.0 0.30" rpy="0 ${0.0*PI/180} 0" />
-</joint>
-<joint name="rgbd_and_summit" type="fixed">
-    <child link="rgbd_camera" />
-    <parent link="base_link" />
-	<!--<origin xyz="0.19 0.0 0.17" rpy="0 ${15*PI/180} 0" />-->
-	<origin xyz="-0.3 0.0 0.60" rpy="0 ${0.0*PI/180} 0" />
-</joint>
-  <!-- SENSORS -->
-  <!-- Hokuyo laser sensors can be parametized with min_angle and max_angle e.g: -->
-  <!--xacro:sensor_hokuyo_utm30lx name="hokuyo_base" parent="base_link" min_angle="2.35" max_angle="-2.35"-->
-  <!--
+	<!--	<xacro:mico_arm parent="base_link" xyz="0.19 0 0.17" rpy="0 ${15*PI/180} 0"/>-->
+	<link name="root">
+		<visual>
+			<origin xyz="0.0 0.0 0.0" rpy="0.0 0.0 0.0" />
+			<geometry>
+				<box size = "0.01 0.01 0.01"/>
+			</geometry>
+			<!--<material name="Black" /> -->
+		</visual>
+		<collision>
+			<origin xyz="0.0 0.0 0.0" rpy="0.0 0.0 0.0" />
+			<geometry>
+				<box size = "0.01 0.01 0.01"/>
+			</geometry>
+		</collision>
+	</link>
+	<joint name="connect_root_and_summit" type="fixed">
+		<child link="root" />
+		<parent link="base_link" />
+		<!--<origin xyz="0.19 0.0 0.17" rpy="0 ${15*PI/180} 0" />-->
+		<origin xyz="0.22 0.0 0.30" rpy="0 ${0.0*PI/180} 0" />
+	</joint>
+	<property name="robot_root" value="root" />
+	<xacro:mico2fingers base_parent="${robot_root}" prefix="mico"/>
+	<!-- Collision Boxes for Modified Platform -->
+	<link name="mini_pc">
+		<visual>
+			<origin xyz="0.0 0.0 0.0" rpy="0.0 0.0 0.0" />
+			<geometry>
+				<box size = "0.40 0.37 0.14"/>
+			</geometry>
+			<material name="Black" />
+		</visual>
+		<collision>
+			<origin xyz="0.0 0.0 0.0" rpy="0.0 0.0 0.0" />
+			<geometry>
+				<box size = "0.40 0.37 0.14"/>
+			</geometry>
+		</collision>
+	</link>
+	<link name="rgbd_camera">
+		<visual>
+			<origin xyz="0.0 0.0 0.0" rpy="0.0 0.0 0.0" />
+			<geometry>
+				<box size = "0.10 0.26 0.60"/>
+			</geometry>
+			<material name="Black" />
+		</visual>
+		<collision>
+			<origin xyz="0.0 0.0 0.0" rpy="0.0 0.0 0.0" />
+			<geometry>
+				<box size = "0.10 0.26 0.60"/>
+			</geometry>
+		</collision>
+	</link>
+	<joint name="mini_pc_and_summit" type="fixed">
+		<child link="mini_pc" />
+		<parent link="base_link" />
+		<!--<origin xyz="0.19 0.0 0.17" rpy="0 ${15*PI/180} 0" />-->
+		<origin xyz="-0.1 0.0 0.30" rpy="0 ${0.0*PI/180} 0" />
+	</joint>
+	<joint name="rgbd_and_summit" type="fixed">
+		<child link="rgbd_camera" />
+		<parent link="base_link" />
+		<!--<origin xyz="0.19 0.0 0.17" rpy="0 ${15*PI/180} 0" />-->
+		<origin xyz="-0.3 0.0 0.60" rpy="0 ${0.0*PI/180} 0" />
+	</joint>
+	<!-- SENSORS -->
+	<!-- Hokuyo laser sensors can be parametized with min_angle and max_angle e.g: -->
+	<!--xacro:sensor_hokuyo_utm30lx name="hokuyo_base" parent="base_link" min_angle="2.35" max_angle="-2.35"-->
+	<!--
 	<xacro:sensor_hokuyo_utm30lx prefix="hokuyo_base" parent="base_link">
 		<origin xyz="0.0 0.0 0.33" rpy="0 0 0"/>
 	</xacro:sensor_hokuyo_utm30lx>
   -->
-<!--
+	<!--
 	<xacro:sensor_hokuyo_urg04lx name="hokuyo1" parent="base_link">
 		<origin xyz="-0.1 0.0 0.33" rpy="0 0 0"/>
 	</xacro:sensor_hokuyo_urg04lx>
 -->
-<!--
+	<!--
   <xacro:sensor_hokuyo_ust10lx name="hokuyo_base" parent="base_link">
 		<origin xyz="0.0 0.0 0.33" rpy="0 0 0"/>
 	</xacro:sensor_hokuyo_ust10lx>
 -->
-<!--
+	<!--
 	<xacro:sensor_imu name="imu" parent="base_link">
 		<origin xyz="-0.18 0.0 0.170" rpy="0 0 0"/>
 	</xacro:sensor_imu>
 -->
-<!--
+	<!--
 	<xacro:sensor_gps name="gps" parent="base_link">
 		<origin xyz="-0.22 0 0.275" rpy="0 0 0"/>
 	</xacro:sensor_gps>
 -->
-<!--
+	<!--
 	<xacro:sensor_kinect name="kinect" parent="base_link">
 		<origin xyz="0.325 0.0 0.16" rpy="0 0 0"/>
 	</xacro:sensor_kinect>
 -->
-<!--
+	<!--
 	<xacro:sensor_fotonic name="fotonic" parent="base_link">
 		<origin xyz="0.3 0.0 0.24" rpy="0 0 0"/>
