Commit message: new mico and mobile manipulator descriptions

File: mico_description/urdf/kinova_common.xacro (robot description, xacro)
@@ -48,5 +48,5 @@
       <limit effort="${joint_torque_limit}" velocity="${joint_velocity_limit}" lower="${joint_lower_limit}" upper="${joint_upper_limit}"/>
       <origin xyz="${joint_origin_xyz}" rpy="${joint_origin_rpy}"/>
-      <dynamics damping="0.2" friction="0.1"/>
+      <dynamics damping="0.3" friction="0.1"/>
     </joint>
     <xacro:unless value="${fixed}">
@@ -100,5 +100,5 @@
     </joint>
   </xacro:macro>
-  <xacro:macro name="kinova_finger" params="prefix finger_number hand finger_origin_xyz finger_origin_rpy">
+  <xacro:macro name="kinova_finger" params="prefix finger_number hand finger_origin_xyz finger_origin_rpy interface:=velocity">
     <xacro:kinova_armlink link_name="${prefix}link_finger_${finger_number}" link_mesh="finger_proximal" mesh_no="57"/>
     <joint name="${prefix}joint_finger_${finger_number}" type="revolute">
@@ -109,14 +109,4 @@
       <limit lower="0" upper="1.51" effort="2" velocity="1"/>
     </joint>
-    <transmission name="${prefix}joint_finger_${finger_number}_trans">
-      <type>transmission_interface/SimpleTransmission</type>
-      <joint name="${prefix}joint_finger_${finger_number}">
-        <hardwareInterface>hardware_interface/EffortJointInterface</hardwareInterface>
-      </joint>
-      <actuator name="${prefix}joint_finger_${finger_number}_actuator">
-        <hardwareInterface>hardware_interface/EffortJointInterface</hardwareInterface>
-        <mechanicalReduction>1</mechanicalReduction>
-      </actuator>
-    </transmission>
     <xacro:kinova_armlink link_name="${prefix}link_finger_tip_${finger_number}" link_mesh="finger_distal" mesh_no="58"/>
     <joint name="${prefix}joint_finger_tip_${finger_number}" type="revolute">
@@ -127,14 +117,70 @@
       <limit lower="0" upper="2" effort="2" velocity="1"/>
     </joint>
-    <transmission name="${prefix}joint_finger_tip_${finger_number}_trans">
-      <type>transmission_interface/SimpleTransmission</type>
-      <joint name="${prefix}joint_finger_tip_${finger_number}">
-        <hardwareInterface>hardware_interface/EffortJointInterface</hardwareInterface>
-      </joint>
-      <actuator name="${prefix}joint_finger_tip_${finger_number}_actuator">
-        <hardwareInterface>hardware_interface/EffortJointInterface</hardwareInterface>
-        <mechanicalReduction>1</mechanicalReduction>
-      </actuator>
-    </transmission>
+    <xacro:if value="${interface == 'effort'}">
+      <transmission name="${prefix}joint_finger_${finger_number}_trans">
+        <type>transmission_interface/SimpleTransmission</type>
+        <joint name="${prefix}joint_finger_${finger_number}">
+          <hardwareInterface>hardware_interface/EffortJointInterface</hardwareInterface>
+        </joint>
+        <actuator name="${prefix}joint_finger_${finger_number}_actuator">
+          <hardwareInterface>hardware_interface/EffortJointInterface</hardwareInterface>
+          <mechanicalReduction>1</mechanicalReduction>
+        </actuator>
+      </transmission>
+      <transmission name="${prefix}joint_finger_tip_${finger_number}_trans">
+        <type>transmission_interface/SimpleTransmission</type>
+        <joint name="${prefix}joint_finger_tip_${finger_number}">
+          <hardwareInterface>hardware_interface/EffortJointInterface</hardwareInterface>
+        </joint>
+        <actuator name="${prefix}joint_finger_tip_${finger_number}_actuator">
+          <hardwareInterface>hardware_interface/EffortJointInterface</hardwareInterface>
+          <mechanicalReduction>1</mechanicalReduction>
+        </actuator>
+      </transmission>
+    </xacro:if>
+    <xacro:if value="${interface == 'velocity'}">
+      <transmission name="${prefix}joint_finger_${finger_number}_trans">
+        <type>transmission_interface/SimpleTransmission</type>
+        <joint name="${prefix}joint_finger_${finger_number}">
+          <hardwareInterface>hardware_interface/VelocityJointInterface</hardwareInterface>
+        </joint>
+        <actuator name="${prefix}joint_finger_${finger_number}_actuator">
+          <hardwareInterface>hardware_interface/VelocityJointInterface</hardwareInterface>
+          <mechanicalReduction>1</mechanicalReduction>
+        </actuator>
+      </transmission>
+      <transmission name="${prefix}joint_finger_tip_${finger_number}_trans">
+        <type>transmission_interface/SimpleTransmission</type>
+        <joint name="${prefix}joint_finger_tip_${finger_number}">
+          <hardwareInterface>hardware_interface/VelocityJointInterface</hardwareInterface>
+        </joint>
+        <actuator name="${prefix}joint_finger_tip_${finger_number}_actuator">
+          <hardwareInterface>hardware_interface/VelocityJointInterface</hardwareInterface>
+          <mechanicalReduction>1</mechanicalReduction>
+        </actuator>
+      </transmission>
+    </xacro:if>
+    <xacro:if value="${interface == 'position'}">
+      <transmission name="${prefix}joint_finger_${finger_number}_trans">
+        <type>transmission_interface/SimpleTransmission</type>
+        <joint name="${prefix}joint_finger_${finger_number}">
+          <hardwareInterface>hardware_interface/PositionJointInterface</hardwareInterface>
+        </joint>
+        <actuator name="${prefix}joint_finger_${finger_number}_actuator">
+          <hardwareInterface>hardware_interface/PositionJointInterface</hardwareInterface>
+          <mechanicalReduction>1</mechanicalReduction>
+        </actuator>
+      </transmission>
+      <transmission name="${prefix}joint_finger_tip_${finger_number}_trans">
+        <type>transmission_interface/SimpleTransmission</type>
+        <joint name="${prefix}joint_finger_tip_${finger_number}">
+          <hardwareInterface>hardware_interface/PositionJointInterface</hardwareInterface>
+        </joint>
+        <actuator name="${prefix}joint_finger_tip_${finger_number}_actuator">
+          <hardwareInterface>hardware_interface/PositionJointInterface</hardwareInterface>
+          <mechanicalReduction>1</mechanicalReduction>
+        </actuator>
+      </transmission>
+    </xacro:if>
   </xacro:macro>
 </root>

File: mico_description/urdf/kinova_inertial.xacro (robot description, xacro)
@@ -29,5 +29,5 @@
    finger_distal      58
 -->
-<xacro:property name="mass_mul" value="1.0" />
+<xacro:property name="mass_mul" value="0.5" />
 <xacro:macro name="inertia_cylinder" params="mass height radius axis:=0">
   <!-- z Axis -->

File: mico_description/urdf/mico2fingers_root.xacro (robot description, xacro)
@@ -1,15 +1,4 @@
 <?xml version="1.0"?>
-<!-- m1_6n refers to mico v1 6DOF non-spherical -->
-<root xmlns:xi="http://www.w3.org/2001/XInclude"
-    xmlns:gazebo="http://playerstage.sourceforge.net/gazebo/xmlschema/#gz"
-    xmlns:model="http://playerstage.sourceforge.net/gazebo/xmlschema/#model"
-    xmlns:sensor="http://playerstage.sourceforge.net/gazebo/xmlschema/#sensor"
-    xmlns:body="http://playerstage.sourceforge.net/gazebo/xmlschema/#body"
-    xmlns:geom="http://playerstage.sourceforge.net/gazebo/xmlschema/#geom"
-    xmlns:controller="http://playerstage.sourceforge.net/gazebo/xmlschema/#controller"
-    xmlns:interface="http://playerstage.sourceforge.net/gazebo/xmlschema/#interface"
-    xmlns:rendering="http://playerstage.sourceforge.net/gazebo/xmlschema/#rendering"
-    xmlns:renderable="http://playerstage.sourceforge.net/gazebo/xmlschema/#renderable"
-    xmlns:physics="http://playerstage.sourceforge.net/gazebo/xmlschema/#physics"
+<robot name="summit_xl"
     xmlns:xacro="http://www.ros.org/wiki/xacro">
     <xacro:include filename="$(find mico_description)/urdf/kinova_common.xacro" />
@@ -19,6 +8,6 @@
     <!-- Import all Kinova Mico Arm Properties elements -->
     <xacro:include filename="$(find mico_description)/urdf/micoproperties.xacro" />
-    <xacro:macro name="mico2fingers" params="base_parent robot_control_ns:='' prefix:='mico' interface:=velocity color:='None'">
-        <xacro:gazebo_config robot_namespace="${robot_control_ns}"/>
+    <xacro:macro name="mico2fingers" params="base_parent prefix:='mico' interface:=velocity">
+        <xacro:gazebo_config robot_namespace=""/>
         <xacro:kinova_armlink link_name="${prefix}_link_base" link_mesh="${link_base_mesh}" mesh_no="${link_base_mesh_no}"/>
         <xacro:kinova_armjoint joint_name="${prefix}_joint_base" type="${joint_base_type}" parent="${base_parent}" child="${prefix}_link_base" joint_axis_xyz="${joint_base_axis_xyz}" joint_origin_xyz="${joint_base_origin_xyz}" joint_origin_rpy="${joint_base_origin_rpy}" joint_lower_limit="0" joint_upper_limit="0" joint_velocity_limit="0" joint_torque_limit="0" fixed="true"/>
@@ -35,10 +24,7 @@
         <xacro:kinova_armlink link_name="${prefix}_link_6" link_mesh="${link_6_mesh}" use_ring_mesh="true" ring_mesh="ring_small" mesh_no="${link_6_mesh_no}"/>
         <xacro:kinova_armjoint joint_name="${prefix}_joint_6" type="${joint_6_type}" parent="${prefix}_link_5" child="${prefix}_link_6" joint_axis_xyz="${joint_6_axis_xyz}" joint_origin_xyz="${joint_6_origin_xyz}" joint_origin_rpy="${joint_6_origin_rpy}" joint_lower_limit="${joint_6_lower_limit}" joint_upper_limit="${joint_6_upper_limit}" joint_velocity_limit="${joint_6_velocity_limit}" joint_torque_limit="${joint_6_torque_limit}" interface="${interface}"/>
-        <xacro:unless value="${color == 'None'}">
-            <xacro:gazebo_materials prefix="${prefix}" color="${color}"/>
-        </xacro:unless>
         <xacro:kinova_virtual_link link_name="${prefix}_end_effector"/>
         <xacro:kinova_virtual_joint joint_name="${prefix}_joint_end_effector" type="${joint_end_effector_type}" parent="${prefix}_link_6" child="${prefix}_end_effector" joint_axis_xyz="${joint_end_effector_axis_xyz}" joint_origin_xyz="${joint_end_effector_origin_xyz}" joint_origin_rpy="${joint_end_effector_origin_rpy}" joint_lower_limit="0" joint_upper_limit="0"/>
         <xacro:kinova_2fingers link_hand="${prefix}_link_6" prefix="${prefix}_"/>
     </xacro:macro>
-</root>
+</robot>

File: mico_description/urdf/mico_standalone.xacro (robot description, xacro)
@@ -13,5 +13,7 @@
     xmlns:renderable="http://playerstage.sourceforge.net/gazebo/xmlschema/#renderable"
     xmlns:physics="http://playerstage.sourceforge.net/gazebo/xmlschema/#physics"
-	xmlns:xacro="http://ros.org/wiki/xacro" name="mico2fingers">
+  xmlns:xacro="http://ros.org/wiki/xacro" name="mico2fingers">
+  <xacro:arg name="interface" default="velocity"/>
+  <xacro:arg name="enable_ft_sensor" default="false"/>
   <xacro:include filename="$(find mico_description)/urdf/mico2fingers.xacro"/>
   <link name="root">
@@ -49,7 +51,7 @@
     <child link="root" />
     <parent link="world" />
-    <origin xyz="0 0 0" rpy="0 0 0" />
+    <origin xyz="0 0 0.1" rpy="0 0 0" />
   </joint>
   <property name="robot_root" value="root" />
-  <xacro:mico2fingers  base_parent="${robot_root}"/>
+  <xacro:mico2fingers  base_parent="${robot_root}" interface="$(arg interface)"/>
 </robot>

File: summit_description/robots/summit_xl_hl_root.urdf.xacro (robot description, xacro)
@@ -2,17 +2,17 @@
 <robot name="summit_xl"
     xmlns:xacro="http://www.ros.org/wiki/xacro">
-    <xacro:macro name="summit_xl_robot" params="prefix *origin kinematic_model:='omni' kinect:=true mini_pc:=true">
-        <!-- ***************** -->
-        <!-- Imported elements -->
-        <!-- ***************** -->
-        <!-- First we import all posible elements defined in the urdf.xacro files. All these elements are defined as macro:xacros -->
-        <!-- Import summit XL base elements -->
-        <xacro:include filename="$(find summit_description)/urdf/bases/summit_xl_hl_base.urdf.xacro" />
-        <!-- Import summit XL wheels -->
-        <xacro:include filename="$(find summit_description)/urdf/wheels/rubber_wheel.urdf.xacro" />
-        <!-- Import summit XL wheels -->
-        <xacro:include filename="$(find summit_description)/urdf/wheels/omni_wheel.urdf.xacro" />
-        <!-- Import all available sensors -->
-        <xacro:include filename="$(find robotnik_sensors)/urdf/all_sensors.urdf.xacro" />
+    <!-- ***************** -->
+    <!-- Imported elements -->
+    <!-- ***************** -->
+    <!-- First we import all posible elements defined in the urdf.xacro files. All these elements are defined as macro:xacros -->
+    <!-- Import summit XL base elements -->
+    <xacro:include filename="$(find summit_description)/urdf/bases/summit_xl_hl_base.urdf.xacro" />
+    <!-- Import summit XL wheels -->
+    <xacro:include filename="$(find summit_description)/urdf/wheels/rubber_wheel.urdf.xacro" />
+    <!-- Import summit XL wheels -->
+    <xacro:include filename="$(find summit_description)/urdf/wheels/omni_wheel.urdf.xacro" />
+    <!-- Import all available sensors -->
+    <xacro:include filename="$(find robotnik_sensors)/urdf/all_sensors.urdf.xacro" />
+    <xacro:macro name="summit_xl_robot" params="prefix *origin kinematic_model:='omni' kinect:=true mini_pc:=true enable_ros_control=true">
         <!-- ***************** -->
         <!-- Global parameters -->
@@ -34,5 +34,5 @@
             <child link="${prefix}odom"/>
         </joint> -->
-<!--
+        <!--
         <link name="${prefix}odom">
             <inertial>
@@ -47,5 +47,5 @@
         <xacro:summit_xl_hl_base prefix="${prefix}" publish_bf="true" hq="${hq}" />
         <!-- WHEELS -->
-        <xacro:if value="${kinematic_model == 'omni'}">
+        <xacro:if value="${kinematic_model in ['omni', 'force_omni']}">
             <!-- OMNI WHEELS -->
             <xacro:omni_wheel prefix="${prefix}front_right" parent="${prefix}base_link" reflect="false" hq="true">
@@ -62,13 +62,13 @@
             </xacro:omni_wheel>
         </xacro:if>
-        <xacro:unless value="${kinematic_model == 'omni'}">
+        <xacro:if value="${kinematic_model not in ['omni', 'force_omni']}">
             <!-- RUBBER WHEELS MIMIC-->
-            <xacro:rubber_wheel prefix="${prefix}front_right" parent="${prefix}base_link" reflect="false" hq="${hq}" >
+            <xacro:rubber_wheel prefix="${prefix}front_right" parent="${prefix}base_link" reflect="false" hq="${hq}">
                 <origin xyz="${wheel_offset_x} -${wheel_offset_y} ${wheel_offset_z}" rpy="0 0 0"/>
             </xacro:rubber_wheel>
-            <xacro:rubber_wheel prefix="${prefix}front_left" parent="${prefix}base_link" reflect="true" hq="${hq}" >
+            <xacro:rubber_wheel prefix="${prefix}front_left" parent="${prefix}base_link" reflect="true" hq="${hq}">
                 <origin xyz="${wheel_offset_x} ${wheel_offset_y} ${wheel_offset_z}" rpy="0 0 0"/>
             </xacro:rubber_wheel>
-            <xacro:rubber_wheel prefix="${prefix}back_left" parent="${prefix}base_link" reflect="true" hq="${hq}" >
+            <xacro:rubber_wheel prefix="${prefix}back_left" parent="${prefix}base_link" reflect="true" hq="${hq}">
                 <origin xyz="-${wheel_offset_x} ${wheel_offset_y} ${wheel_offset_z}" rpy="0 0 0"/>
             </xacro:rubber_wheel>
@@ -76,5 +76,5 @@
                 <origin xyz="-${wheel_offset_x} -${wheel_offset_y} ${wheel_offset_z}" rpy="0 0 0"/>
             </xacro:rubber_wheel>
-        </xacro:unless>
+        </xacro:if>
         <!-- SENSORS -->
         <!-- IMU Sensor -->
@@ -182,11 +182,16 @@
             <xacro:omni_steering prefix="${prefix}" publish_tf="false"/>
         </xacro:if>
-        <xacro:if value="${kinematic_model == 'skid'}">
+        <xacro:if value="${kinematic_model in ['skid','diff']}">
             <xacro:skid_steering prefix="${prefix}" publish_tf="false"/>
         </xacro:if>
-        <xacro:if value="${kinematic_model == 'diff'}">
-            <xacro:skid_steering prefix="${prefix}" publish_tf="false"/>
+        <xacro:if value="${kinematic_model == 'force_omni'}">
+            <xacro:ros_force_based_move prefix="${prefix}" publish_tf="false"/>
         </xacro:if>
-        <xacro:ros_control/>
+        <xacro:if value="${kinematic_model == 'force_diff'}">
+            <xacro:ros_force_based_move_diff prefix="${prefix}" publish_tf="false"/>
+        </xacro:if>
+        <xacro:if value="${enable_ros_control}">
+            <xacro:ros_control/>
+        </xacro:if>
     </xacro:macro>
 </robot>

File: summit_description/urdf/bases/summit_xl_base.gazebo.xacro (robot description, xacro)
@@ -45,6 +45,21 @@
 				<odometryFrame>${prefix}odom</odometryFrame>
 				<yaw_velocity_p_gain>10000.0</yaw_velocity_p_gain>
-				<x_velocity_p_gain>10000.0</x_velocity_p_gain>
-				<y_velocity_p_gain>10000.0</y_velocity_p_gain>
+				<x_velocity_p_gain>100000.0</x_velocity_p_gain>
+				<y_velocity_p_gain>100000.0</y_velocity_p_gain>
+				<robotBaseFrame>${prefix}base_footprint</robotBaseFrame>
+				<odometryRate>100.0</odometryRate>
+				<publishOdometryTf>${publish_tf}</publishOdometryTf>
+			</plugin>
+		</gazebo>
+	</xacro:macro>
+	<xacro:macro name="ros_force_based_move_diff" params="publish_tf prefix">
+		<gazebo>
+			<plugin name="ros_force_based_move" filename="libgazebo_ros_force_based_move.so">
+				<commandTopic>robotnik_base_control/cmd_vel</commandTopic>
+				<odometryTopic>robotnik_base_control/odom</odometryTopic>
+				<odometryFrame>${prefix}odom</odometryFrame>
+				<yaw_velocity_p_gain>10000.0</yaw_velocity_p_gain>
+				<x_velocity_p_gain>100000.0</x_velocity_p_gain>
+				<y_velocity_p_gain>0.0</y_velocity_p_gain>
 				<robotBaseFrame>${prefix}base_footprint</robotBaseFrame>
 				<odometryRate>100.0</odometryRate>

File: summit_description/urdf/wheels/rubber_wheel.urdf.xacro (robot description, xacro)
@@ -68,6 +68,6 @@
      </transmission>
     <gazebo reference="${prefix}_wheel">
-			<mu1 value="1.0"/>
-			<mu2 value="1.0"/>
+			<mu1 value="0.01"/>
+			<mu2 value="0.01"/>
 			<kp value="10000000.0" />
 			<kd value="1.0" />
