Commit message: summit mico multi robot spawn

File: mico_description/urdf/kinova_common.xacro (robot description, xacro)
@@ -17,26 +17,35 @@
   <xacro:macro name="kinova_armlink" params="link_name link_mesh ring_mesh:=ring_big use_ring_mesh:=false mesh_no">
     <link name="${link_name}">
-      <visual>
-        <geometry>
-          <mesh filename="package://kinova_description/meshes/${link_mesh}.dae"/>
-        </geometry>
-        <material name="carbon_fiber">
-          <color rgba="0.792156862745098 0.819607843137255 0.933333333333333 1" />
-        </material>
-      </visual>
-      <!-- Adding ring to the model -->
-      <xacro:if value="${use_ring_mesh}">
+      <xacro:unless value="${link_mesh == 'None'}">
         <visual>
           <geometry>
-            <mesh filename="package://kinova_description/meshes/${ring_mesh}.dae"/>
+            <mesh filename="package://kinova_description/meshes/${link_mesh}.dae"/>
           </geometry>
+          <material name="carbon_fiber">
+            <color rgba="0.792156862745098 0.819607843137255 0.933333333333333 1" />
+          </material>
         </visual>
-      </xacro:if>
-      <collision>
-        <geometry>
-          <mesh filename="package://kinova_description/meshes/${link_mesh}.dae"/>
-        </geometry>
-      </collision>
-      <xacro:kinova_inertial mesh_no="${mesh_no}"/>
+        <!-- Adding ring to the model -->
+        <xacro:if value="${use_ring_mesh}">
+          <visual>
+            <geometry>
+              <mesh filename="package://kinova_description/meshes/${ring_mesh}.dae"/>
+            </geometry>
+          </visual>
+        </xacro:if>
+        <collision>
+          <geometry>
+            <mesh filename="package://kinova_description/meshes/${link_mesh}.dae"/>
+          </geometry>
+        </collision>
+        <xacro:kinova_inertial mesh_no="${mesh_no}"/>
+      </xacro:unless>
+      <xacro:if value="${link_mesh == 'None'}">
+        <inertial>
+          <mass value="0.5" />
+          <origin xyz="0 0 0" />
+          <xacro:inertia_cylinder height="0.14"  radius = "0.04" mass="0.7477"/>
+        </inertial>
+      </xacro:if>
     </link>
   </xacro:macro>
@@ -100,7 +109,13 @@
     </joint>
   </xacro:macro>
-  <xacro:macro name="kinova_finger" params="prefix finger_number hand finger_origin_xyz finger_origin_rpy interface:=velocity">
+  <xacro:macro name="kinova_finger" params="prefix finger_number hand finger_origin_xyz finger_origin_rpy interface:=velocity fixed:=false">
     <xacro:kinova_armlink link_name="${prefix}link_finger_${finger_number}" link_mesh="finger_proximal" mesh_no="57"/>
-    <joint name="${prefix}joint_finger_${finger_number}" type="revolute">
+    <xacro:if value="${fixed}">
+      <xacro:property name="finger_joint_type" value="fixed"/>
+    </xacro:if>
+    <xacro:unless value="${fixed}">
+      <xacro:property name="finger_joint_type" value="revolute"/>
+    </xacro:unless>
+    <joint name="${prefix}joint_finger_${finger_number}" type="${finger_joint_type}">
       <parent link="${hand}"/>
       <child link="${prefix}link_finger_${finger_number}"/>
@@ -110,5 +125,5 @@
     </joint>
     <xacro:kinova_armlink link_name="${prefix}link_finger_tip_${finger_number}" link_mesh="finger_distal" mesh_no="58"/>
-    <joint name="${prefix}joint_finger_tip_${finger_number}" type="revolute">
+    <joint name="${prefix}joint_finger_tip_${finger_number}" type="${finger_joint_type}">
       <parent link="${prefix}link_finger_${finger_number}"/>
       <child link="${prefix}link_finger_tip_${finger_number}"/>
@@ -117,70 +132,72 @@
       <limit lower="0" upper="2" effort="2" velocity="1"/>
     </joint>
-    <xacro:if value="${interface == 'effort'}">
-      <transmission name="${prefix}joint_finger_${finger_number}_trans">
-        <type>transmission_interface/SimpleTransmission</type>
-        <joint name="${prefix}joint_finger_${finger_number}">
-          <hardwareInterface>hardware_interface/EffortJointInterface</hardwareInterface>
-        </joint>
-        <actuator name="${prefix}joint_finger_${finger_number}_actuator">
-          <hardwareInterface>hardware_interface/EffortJointInterface</hardwareInterface>
-          <mechanicalReduction>1</mechanicalReduction>
-        </actuator>
-      </transmission>
-      <transmission name="${prefix}joint_finger_tip_${finger_number}_trans">
-        <type>transmission_interface/SimpleTransmission</type>
-        <joint name="${prefix}joint_finger_tip_${finger_number}">
-          <hardwareInterface>hardware_interface/EffortJointInterface</hardwareInterface>
-        </joint>
-        <actuator name="${prefix}joint_finger_tip_${finger_number}_actuator">
-          <hardwareInterface>hardware_interface/EffortJointInterface</hardwareInterface>
-          <mechanicalReduction>1</mechanicalReduction>
-        </actuator>
-      </transmission>
-    </xacro:if>
-    <xacro:if value="${interface == 'velocity'}">
-      <transmission name="${prefix}joint_finger_${finger_number}_trans">
-        <type>transmission_interface/SimpleTransmission</type>
-        <joint name="${prefix}joint_finger_${finger_number}">
-          <hardwareInterface>hardware_interface/VelocityJointInterface</hardwareInterface>
-        </joint>
-        <actuator name="${prefix}joint_finger_${finger_number}_actuator">
-          <hardwareInterface>hardware_interface/VelocityJointInterface</hardwareInterface>
-          <mechanicalReduction>1</mechanicalReduction>
-        </actuator>
-      </transmission>
-      <transmission name="${prefix}joint_finger_tip_${finger_number}_trans">
-        <type>transmission_interface/SimpleTransmission</type>
-        <joint name="${prefix}joint_finger_tip_${finger_number}">
-          <hardwareInterface>hardware_interface/VelocityJointInterface</hardwareInterface>
-        </joint>
-        <actuator name="${prefix}joint_finger_tip_${finger_number}_actuator">
-          <hardwareInterface>hardware_interface/VelocityJointInterface</hardwareInterface>
-          <mechanicalReduction>1</mechanicalReduction>
-        </actuator>
-      </transmission>
-    </xacro:if>
-    <xacro:if value="${interface == 'position'}">
-      <transmission name="${prefix}joint_finger_${finger_number}_trans">
-        <type>transmission_interface/SimpleTransmission</type>
-        <joint name="${prefix}joint_finger_${finger_number}">
-          <hardwareInterface>hardware_interface/PositionJointInterface</hardwareInterface>
-        </joint>
-        <actuator name="${prefix}joint_finger_${finger_number}_actuator">
-          <hardwareInterface>hardware_interface/PositionJointInterface</hardwareInterface>
-          <mechanicalReduction>1</mechanicalReduction>
-        </actuator>
-      </transmission>
-      <transmission name="${prefix}joint_finger_tip_${finger_number}_trans">
-        <type>transmission_interface/SimpleTransmission</type>
-        <joint name="${prefix}joint_finger_tip_${finger_number}">
-          <hardwareInterface>hardware_interface/PositionJointInterface</hardwareInterface>
-        </joint>
-        <actuator name="${prefix}joint_finger_tip_${finger_number}_actuator">
-          <hardwareInterface>hardware_interface/PositionJointInterface</hardwareInterface>
-          <mechanicalReduction>1</mechanicalReduction>
-        </actuator>
-      </transmission>
-    </xacro:if>
+    <xacro:unless value="${fixed}">
+      <xacro:if value="${interface == 'effort'}">
+        <transmission name="${prefix}joint_finger_${finger_number}_trans">
+          <type>transmission_interface/SimpleTransmission</type>
+          <joint name="${prefix}joint_finger_${finger_number}">
+            <hardwareInterface>hardware_interface/EffortJointInterface</hardwareInterface>
+          </joint>
+          <actuator name="${prefix}joint_finger_${finger_number}_actuator">
+            <hardwareInterface>hardware_interface/EffortJointInterface</hardwareInterface>
+            <mechanicalReduction>1</mechanicalReduction>
+          </actuator>
+        </transmission>
+        <transmission name="${prefix}joint_finger_tip_${finger_number}_trans">
+          <type>transmission_interface/SimpleTransmission</type>
+          <joint name="${prefix}joint_finger_tip_${finger_number}">
+            <hardwareInterface>hardware_interface/EffortJointInterface</hardwareInterface>
+          </joint>
+          <actuator name="${prefix}joint_finger_tip_${finger_number}_actuator">
+            <hardwareInterface>hardware_interface/EffortJointInterface</hardwareInterface>
+            <mechanicalReduction>1</mechanicalReduction>
+          </actuator>
+        </transmission>
+      </xacro:if>
+      <xacro:if value="${interface == 'velocity'}">
+        <transmission name="${prefix}joint_finger_${finger_number}_trans">
+          <type>transmission_interface/SimpleTransmission</type>
+          <joint name="${prefix}joint_finger_${finger_number}">
+            <hardwareInterface>hardware_interface/VelocityJointInterface</hardwareInterface>
+          </joint>
+          <actuator name="${prefix}joint_finger_${finger_number}_actuator">
+            <hardwareInterface>hardware_interface/VelocityJointInterface</hardwareInterface>
+            <mechanicalReduction>1</mechanicalReduction>
+          </actuator>
+        </transmission>
+        <transmission name="${prefix}joint_finger_tip_${finger_number}_trans">
+          <type>transmission_interface/SimpleTransmission</type>
+          <joint name="${prefix}joint_finger_tip_${finger_number}">
+            <hardwareInterface>hardware_interface/VelocityJointInterface</hardwareInterface>
+          </joint>
+          <actuator name="${prefix}joint_finger_tip_${finger_number}_actuator">
+            <hardwareInterface>hardware_interface/VelocityJointInterface</hardwareInterface>
+            <mechanicalReduction>1</mechanicalReduction>
+          </actuator>
+        </transmission>
+      </xacro:if>
+      <xacro:if value="${interface == 'position'}">
+        <transmission name="${prefix}joint_finger_${finger_number}_trans">
+          <type>transmission_interface/SimpleTransmission</type>
+          <joint name="${prefix}joint_finger_${finger_number}">
+            <hardwareInterface>hardware_interface/PositionJointInterface</hardwareInterface>
+          </joint>
+          <actuator name="${prefix}joint_finger_${finger_number}_actuator">
+            <hardwareInterface>hardware_interface/PositionJointInterface</hardwareInterface>
+            <mechanicalReduction>1</mechanicalReduction>
+          </actuator>
+        </transmission>
+        <transmission name="${prefix}joint_finger_tip_${finger_number}_trans">
+          <type>transmission_interface/SimpleTransmission</type>
+          <joint name="${prefix}joint_finger_tip_${finger_number}">
+            <hardwareInterface>hardware_interface/PositionJointInterface</hardwareInterface>
+          </joint>
+          <actuator name="${prefix}joint_finger_tip_${finger_number}_actuator">
+            <hardwareInterface>hardware_interface/PositionJointInterface</hardwareInterface>
+            <mechanicalReduction>1</mechanicalReduction>
+          </actuator>
+        </transmission>
+      </xacro:if>
+    </xacro:unless>
   </xacro:macro>
 </root>

File: mico_description/urdf/kinova_finger_set.xacro (robot description, xacro)
@@ -15,9 +15,17 @@
     xmlns:xacro="http://www.ros.org/wiki/xacro">
     <xacro:include filename="$(find mico_description)/urdf/kinova_common.xacro" />
-    <xacro:macro name="kinova_2fingers" params="link_hand prefix">
-        <!-- finger1 Rot := Ry((1/2)*Pi) . Rx(Pi) . Rz(-52.8*((1/180)*Pi)) -->
-        <xacro:kinova_finger prefix="${prefix}" finger_number="1" hand="${link_hand}" finger_origin_xyz="-0.0025 0.03095 -0.11482" finger_origin_rpy="-1.570796327 .649262481663582 1.57079632679490"/>
-        <!-- finger2 Rot := Ry((1/2)*Pi) . Rz(-52.8*((1/180)*Pi))  -->
-        <xacro:kinova_finger prefix="${prefix}" finger_number="2" hand="${link_hand}" finger_origin_xyz="-0.0025 -0.03095 -0.11482" finger_origin_rpy="-1.570796327 .649262481663582 -1.57079632679490"/>
+    <xacro:macro name="kinova_2fingers" params="link_hand prefix fixed:=false">
+        <xacro:unless value="${fixed}">
+            <!-- finger1 Rot := Ry((1/2)*Pi) . Rx(Pi) . Rz(-52.8*((1/180)*Pi)) -->
+            <xacro:kinova_finger prefix="${prefix}" finger_number="1" hand="${link_hand}" finger_origin_xyz="-0.0025 0.03095 -0.11482" finger_origin_rpy="-1.570796327 .649262481663582 1.57079632679490"/>
+            <!-- finger2 Rot := Ry((1/2)*Pi) . Rz(-52.8*((1/180)*Pi))  -->
+            <xacro:kinova_finger prefix="${prefix}" finger_number="2" hand="${link_hand}" finger_origin_xyz="-0.0025 -0.03095 -0.11482" finger_origin_rpy="-1.570796327 .649262481663582 -1.57079632679490"/>
+        </xacro:unless>
+        <xacro:if value="${fixed}">
+            <!-- finger1 Rot := Ry((1/2)*Pi) . Rx(Pi) . Rz(-52.8*((1/180)*Pi)) -->
+            <xacro:kinova_finger prefix="${prefix}" finger_number="1" hand="${link_hand}" finger_origin_xyz="-0.0025 0.04095 -0.11482" finger_origin_rpy="-1.570796327 1.570796327 1.57079632679490" fixed="true"/>
+            <!-- finger2 Rot := Ry((1/2)*Pi) . Rz(-52.8*((1/180)*Pi))  -->
+            <xacro:kinova_finger prefix="${prefix}" finger_number="2" hand="${link_hand}" finger_origin_xyz="-0.0025 -0.04095 -0.11482" finger_origin_rpy="-1.570796327 1.570796327 -1.57079632679490" fixed="true"/>
+        </xacro:if>
     </xacro:macro>
 </root>
