Commit message: summit mico multi robot spawn

File: mico_description/urdf/mico2fingers.xacro (robot description, xacro)
@@ -19,20 +19,56 @@
     <!-- Import all Kinova Mico Arm Properties elements -->
     <xacro:include filename="$(find mico_description)/urdf/micoproperties.xacro" />
-    <xacro:macro name="mico2fingers" params="base_parent robot_control_ns:='' prefix:='mico' interface:=velocity color:='None'">
+    <xacro:macro name="mico2fingers" params="base_parent robot_control_ns:='' prefix:='mico' interface:=velocity color:='None' J1_offset:=0.0 J2_offset:=0.0 J3_offset:=0.0 J4_offset:=0.0 J5_offset:=0.0 J6_offset:=0.0">
         <xacro:gazebo_config robot_namespace="${robot_control_ns}"/>
         <xacro:kinova_armlink link_name="${prefix}_link_base" link_mesh="${link_base_mesh}" mesh_no="${link_base_mesh_no}"/>
         <xacro:kinova_armjoint joint_name="${prefix}_joint_base" type="${joint_base_type}" parent="${base_parent}" child="${prefix}_link_base" joint_axis_xyz="${joint_base_axis_xyz}" joint_origin_xyz="${joint_base_origin_xyz}" joint_origin_rpy="${joint_base_origin_rpy}" joint_lower_limit="0" joint_upper_limit="0" joint_velocity_limit="0" joint_torque_limit="0" fixed="true"/>
         <xacro:kinova_armlink link_name="${prefix}_link_1" link_mesh="${link_1_mesh}" use_ring_mesh="true" mesh_no="${link_1_mesh_no}"/>
-        <xacro:kinova_armjoint joint_name="${prefix}_joint_1" type="${joint_1_type}" parent="${prefix}_link_base" child="${prefix}_link_1" joint_axis_xyz="${joint_1_axis_xyz}" joint_origin_xyz="${joint_1_origin_xyz}" joint_origin_rpy="${joint_1_origin_rpy}" joint_lower_limit="${joint_1_lower_limit}" joint_upper_limit="${joint_1_upper_limit}" joint_velocity_limit="${joint_1_velocity_limit}" joint_torque_limit="${joint_1_torque_limit}" interface="${interface}"/>
+        <xacro:if value="${J1_offset in [0.0, 0, None]}">
+            <xacro:kinova_armjoint joint_name="${prefix}_joint_1" type="${joint_1_type}" parent="${prefix}_link_base" child="${prefix}_link_1" joint_axis_xyz="${joint_1_axis_xyz}" joint_origin_xyz="${joint_1_origin_xyz}" joint_origin_rpy="${joint_1_origin_rpy}" joint_lower_limit="${joint_1_lower_limit}" joint_upper_limit="${joint_1_upper_limit}" joint_velocity_limit="${joint_1_velocity_limit}" joint_torque_limit="${joint_1_torque_limit}" interface="${interface}"/>
+        </xacro:if>
+        <xacro:unless value="${J1_offset in [0.0, 0, None]}">
+            <xacro:kinova_armjoint joint_name="${prefix}_joint_1" type="${joint_1_type}" parent="${prefix}_link_base" child="${prefix}_link_1" joint_axis_xyz="${joint_1_axis_xyz}" joint_origin_xyz="${joint_1_origin_xyz}" joint_origin_rpy="0 ${J_PI} ${J1_offset}" joint_lower_limit="${joint_1_lower_limit-J1_offset}" joint_upper_limit="${joint_1_upper_limit-J1_offset}" joint_velocity_limit="${joint_1_velocity_limit}" joint_torque_limit="${joint_1_torque_limit}" interface="${interface}"/>
+        </xacro:unless>
         <xacro:kinova_armlink link_name="${prefix}_link_2" link_mesh="${link_2_mesh}" use_ring_mesh="true" mesh_no="${link_2_mesh_no}"/>
-        <xacro:kinova_armjoint joint_name="${prefix}_joint_2" type="${joint_2_type}" parent="${prefix}_link_1" child="${prefix}_link_2" joint_axis_xyz="${joint_2_axis_xyz}" joint_origin_xyz="${joint_2_origin_xyz}" joint_origin_rpy="${joint_2_origin_rpy}" joint_lower_limit="${joint_2_lower_limit}" joint_upper_limit="${joint_2_upper_limit}" joint_velocity_limit="${joint_2_velocity_limit}" joint_torque_limit="${joint_2_torque_limit}" interface="${interface}"/>
+        <xacro:if value="${J2_offset in [0.0, 0, None]}">
+            <xacro:kinova_armjoint joint_name="${prefix}_joint_2" type="${joint_2_type}" parent="${prefix}_link_1" child="${prefix}_link_2" joint_axis_xyz="${joint_2_axis_xyz}" joint_origin_xyz="${joint_2_origin_xyz}" joint_origin_rpy="${joint_2_origin_rpy}" joint_lower_limit="${joint_2_lower_limit}" joint_upper_limit="${joint_2_upper_limit}" joint_velocity_limit="${joint_2_velocity_limit}" joint_torque_limit="${joint_2_torque_limit}" interface="${interface}"/>
+        </xacro:if>
+        <xacro:unless value="${J2_offset in [0.0, 0, None]}">
+            <xacro:kinova_armjoint joint_name="${prefix}_joint_2" type="${joint_2_type}" parent="${prefix}_link_1" child="${prefix}_link_2" joint_axis_xyz="${joint_2_axis_xyz}" joint_origin_xyz="${joint_2_origin_xyz}" joint_origin_rpy="${-J_PI/2} ${J2_offset} ${J_PI}" joint_lower_limit="${joint_2_lower_limit-J2_offset}" joint_upper_limit="${joint_2_upper_limit-J2_offset}" joint_velocity_limit="${joint_2_velocity_limit}" joint_torque_limit="${joint_2_torque_limit}" interface="${interface}"/>
+        </xacro:unless>
         <xacro:kinova_armlink link_name="${prefix}_link_3" link_mesh="${link_3_mesh}" use_ring_mesh="true" mesh_no="${link_3_mesh_no}"/>
-        <xacro:kinova_armjoint joint_name="${prefix}_joint_3" type="${joint_3_type}" parent="${prefix}_link_2" child="${prefix}_link_3" joint_axis_xyz="${joint_3_axis_xyz}" joint_origin_xyz="${joint_3_origin_xyz}" joint_origin_rpy="${joint_3_origin_rpy}" joint_lower_limit="${joint_3_lower_limit}" joint_upper_limit="${joint_3_upper_limit}" joint_velocity_limit="${joint_3_velocity_limit}" joint_torque_limit="${joint_3_torque_limit}" interface="${interface}"/>
+        <xacro:if value="${J3_offset in [0.0, 0, None]}">
+            <xacro:kinova_armjoint joint_name="${prefix}_joint_3" type="${joint_3_type}" parent="${prefix}_link_2" child="${prefix}_link_3" joint_axis_xyz="${joint_3_axis_xyz}" joint_origin_xyz="${joint_3_origin_xyz}" joint_origin_rpy="${joint_3_origin_rpy}" joint_lower_limit="${joint_3_lower_limit}" joint_upper_limit="${joint_3_upper_limit}" joint_velocity_limit="${joint_3_velocity_limit}" joint_torque_limit="${joint_3_torque_limit}" interface="${interface}"/>
+        </xacro:if>
+        <xacro:unless value="${J3_offset in [0.0, 0, None]}">
+            <xacro:kinova_armjoint joint_name="${prefix}_joint_3" type="${joint_3_type}" parent="${prefix}_link_2" child="${prefix}_link_3" joint_axis_xyz="${joint_3_axis_xyz}" joint_origin_xyz="${joint_3_origin_xyz}" joint_origin_rpy="0 ${J_PI} ${J3_offset}" joint_lower_limit="${joint_3_lower_limit-J3_offset}" joint_upper_limit="${joint_3_upper_limit-J3_offset}" joint_velocity_limit="${joint_3_velocity_limit}" joint_torque_limit="${joint_3_torque_limit}" interface="${interface}"/>
+        </xacro:unless>
         <xacro:kinova_armlink link_name="${prefix}_link_4" link_mesh="${link_4_mesh}" use_ring_mesh="true" ring_mesh="ring_small" mesh_no="${link_4_mesh_no}"/>
-        <xacro:kinova_armjoint joint_name="${prefix}_joint_4" type="${joint_4_type}" parent="${prefix}_link_3" child="${prefix}_link_4" joint_axis_xyz="${joint_4_axis_xyz}" joint_origin_xyz="${joint_4_origin_xyz}" joint_origin_rpy="${joint_4_origin_rpy}" joint_lower_limit="${joint_4_lower_limit}" joint_upper_limit="${joint_4_upper_limit}" joint_velocity_limit="${joint_4_velocity_limit}" joint_torque_limit="${joint_4_torque_limit}" interface="${interface}"/>
-        <xacro:kinova_armlink link_name="${prefix}_link_5" link_mesh="${link_5_mesh}" use_ring_mesh="true" ring_mesh="ring_small" mesh_no="${link_5_mesh_no}"/>
-        <xacro:kinova_armjoint joint_name="${prefix}_joint_5" type="${joint_5_type}" parent="${prefix}_link_4" child="${prefix}_link_5" joint_axis_xyz="${joint_5_axis_xyz}" joint_origin_xyz="${joint_5_origin_xyz}" joint_origin_rpy="${joint_5_origin_rpy}" joint_lower_limit="${joint_5_lower_limit}" joint_upper_limit="${joint_5_upper_limit}" joint_velocity_limit="${joint_5_velocity_limit}" joint_torque_limit="${joint_5_torque_limit}" interface="${interface}"/>
-        <xacro:kinova_armlink link_name="${prefix}_link_6" link_mesh="${link_6_mesh}" use_ring_mesh="true" ring_mesh="ring_small" mesh_no="${link_6_mesh_no}"/>
-        <xacro:kinova_armjoint joint_name="${prefix}_joint_6" type="${joint_6_type}" parent="${prefix}_link_5" child="${prefix}_link_6" joint_axis_xyz="${joint_6_axis_xyz}" joint_origin_xyz="${joint_6_origin_xyz}" joint_origin_rpy="${joint_6_origin_rpy}" joint_lower_limit="${joint_6_lower_limit}" joint_upper_limit="${joint_6_upper_limit}" joint_velocity_limit="${joint_6_velocity_limit}" joint_torque_limit="${joint_6_torque_limit}" interface="${interface}"/>
+        <xacro:if value="${J4_offset in [0.0, 0, None]}">
+            <xacro:kinova_armjoint joint_name="${prefix}_joint_4" type="${joint_4_type}" parent="${prefix}_link_3" child="${prefix}_link_4" joint_axis_xyz="${joint_4_axis_xyz}" joint_origin_xyz="${joint_4_origin_xyz}" joint_origin_rpy="${joint_4_origin_rpy}" joint_lower_limit="${joint_4_lower_limit-J4_offset}" joint_upper_limit="${joint_4_upper_limit-J4_offset}" joint_velocity_limit="${joint_4_velocity_limit}" joint_torque_limit="${joint_4_torque_limit}" interface="${interface}"/>
+        </xacro:if>
+        <xacro:unless value="${J4_offset in [0.0, 0, None]}">
+            <xacro:kinova_armjoint joint_name="${prefix}_joint_4" type="${joint_4_type}" parent="${prefix}_link_3" child="${prefix}_link_4" joint_axis_xyz="${joint_4_axis_xyz}" joint_origin_xyz="${joint_4_origin_xyz}" joint_origin_rpy="${-J_PI/2} ${J4_offset} ${J_PI}" joint_lower_limit="${joint_4_lower_limit-J4_offset}" joint_upper_limit="${joint_4_upper_limit-J4_offset}" joint_velocity_limit="${joint_4_velocity_limit}" joint_torque_limit="${joint_4_torque_limit}" interface="${interface}"/>
+        </xacro:unless>
+        <xacro:if value="${J5_offset in [0.0, 0, None]}">
+            <xacro:kinova_armlink link_name="${prefix}_link_5" link_mesh="${link_5_mesh}" use_ring_mesh="true" ring_mesh="ring_small" mesh_no="${link_5_mesh_no}"/>
+            <xacro:kinova_armjoint joint_name="${prefix}_joint_5" type="${joint_5_type}" parent="${prefix}_link_4" child="${prefix}_link_5" joint_axis_xyz="${joint_5_axis_xyz}" joint_origin_xyz="${joint_5_origin_xyz}" joint_origin_rpy="${joint_5_origin_rpy}" joint_lower_limit="${joint_5_lower_limit}" joint_upper_limit="${joint_5_upper_limit}" joint_velocity_limit="${joint_5_velocity_limit}" joint_torque_limit="${joint_5_torque_limit}" interface="${interface}"/>
+        </xacro:if>
+        <xacro:unless value="${J5_offset in [0.0, 0, None]}">
+            <xacro:kinova_armlink link_name="${prefix}_virtual_link_5" link_mesh="None" use_ring_mesh="true" ring_mesh="ring_small" mesh_no="${link_5_mesh_no}"/>
+            <xacro:kinova_armjoint joint_name="${prefix}_joint_4_to_5" type="fixed" parent="${prefix}_link_4" child="${prefix}_virtual_link_5" joint_axis_xyz="${joint_5_axis_xyz}" joint_origin_xyz="${joint_5_origin_xyz}" joint_origin_rpy="${joint_5_origin_rpy}" joint_lower_limit="0" joint_upper_limit="0" joint_velocity_limit="0" joint_torque_limit="0" fixed="true"/>
+            <xacro:kinova_armlink link_name="${prefix}_link_5" link_mesh="${link_5_mesh}" use_ring_mesh="true" ring_mesh="ring_small" mesh_no="${link_5_mesh_no}"/>
+            <xacro:kinova_armjoint joint_name="${prefix}_joint_5" type="${joint_5_type}" parent="${prefix}_virtual_link_5" child="${prefix}_link_5" joint_axis_xyz="${joint_5_axis_xyz}" joint_origin_xyz="0 0 0" joint_origin_rpy="0 0 ${J5_offset}" joint_lower_limit="${joint_5_lower_limit-J5_offset}" joint_upper_limit="${joint_5_upper_limit-J5_offset}" joint_velocity_limit="${joint_5_velocity_limit}" joint_torque_limit="${joint_5_torque_limit}" interface="${interface}"/>
+        </xacro:unless>
+        <xacro:if value="${J6_offset in [0.0, 0, None]}">
+            <xacro:kinova_armlink link_name="${prefix}_link_6" link_mesh="${link_6_mesh}" use_ring_mesh="true" ring_mesh="ring_small" mesh_no="${link_6_mesh_no}"/>
+            <xacro:kinova_armjoint joint_name="${prefix}_joint_6" type="${joint_6_type}" parent="${prefix}_link_5" child="${prefix}_link_6" joint_axis_xyz="${joint_6_axis_xyz}" joint_origin_xyz="${joint_6_origin_xyz}" joint_origin_rpy="${joint_6_origin_rpy}" joint_lower_limit="${joint_6_lower_limit-J6_offset}" joint_upper_limit="${joint_6_upper_limit-J6_offset}" joint_velocity_limit="${joint_6_velocity_limit}" joint_torque_limit="${joint_6_torque_limit}" interface="${interface}"/>
+        </xacro:if>
+        <xacro:unless value="${J6_offset in [0.0, 0, None]}">
+            <xacro:kinova_armlink link_name="${prefix}_virtual_link_6" link_mesh="None" use_ring_mesh="true" ring_mesh="ring_small" mesh_no="${link_6_mesh_no}"/>
+            <xacro:kinova_armjoint joint_name="${prefix}_joint_5_to_6" type="fixed" parent="${prefix}_link_5" child="${prefix}_virtual_link_6" joint_axis_xyz="${joint_6_axis_xyz}" joint_origin_xyz="${joint_6_origin_xyz}" joint_origin_rpy="${joint_6_origin_rpy}" joint_lower_limit="0" joint_upper_limit="0" joint_velocity_limit="0" joint_torque_limit="0" fixed="true"/>
+            <xacro:kinova_armlink link_name="${prefix}_link_6" link_mesh="${link_6_mesh}" use_ring_mesh="true" ring_mesh="ring_small" mesh_no="${link_6_mesh_no}"/>
+            <xacro:kinova_armjoint joint_name="${prefix}_joint_6" type="${joint_6_type}" parent="${prefix}_virtual_link_6" child="${prefix}_link_6" joint_axis_xyz="${joint_6_axis_xyz}" joint_origin_xyz="0 0 0" joint_origin_rpy="0.0 0.0 ${J6_offset}" joint_lower_limit="${joint_6_lower_limit-J6_offset}" joint_upper_limit="${joint_6_upper_limit-J6_offset}" joint_velocity_limit="${joint_6_velocity_limit}" joint_torque_limit="${joint_6_torque_limit}" interface="${interface}"/>
+        </xacro:unless>
         <xacro:unless value="${color == 'None'}">
             <xacro:gazebo_materials prefix="${prefix}" color="${color}"/>
@@ -40,5 +76,5 @@
         <xacro:kinova_virtual_link link_name="${prefix}_end_effector"/>
         <xacro:kinova_virtual_joint joint_name="${prefix}_joint_end_effector" type="${joint_end_effector_type}" parent="${prefix}_link_6" child="${prefix}_end_effector" joint_axis_xyz="${joint_end_effector_axis_xyz}" joint_origin_xyz="${joint_end_effector_origin_xyz}" joint_origin_rpy="${joint_end_effector_origin_rpy}" joint_lower_limit="0" joint_upper_limit="0"/>
-        <xacro:kinova_2fingers link_hand="${prefix}_link_6" prefix="${prefix}_"/>
+        <xacro:kinova_2fingers link_hand="${prefix}_link_6" prefix="${prefix}_" fixed="true"/>
     </xacro:macro>
 </root>

File: mico_description/urdf/micoproperties.xacro (robot description, xacro)
@@ -33,6 +33,6 @@
     <xacro:property name="joint_1_upper_limit" value="${2*J_PI}" />
     <!-- <xacro:property name="joint_1_velocity_limit" value="${36*J_PI/180}" /> -->
-    <xacro:property name="joint_1_velocity_limit" value="1.0" />
-    <xacro:property name="joint_1_torque_limit" value="40" />
+    <xacro:property name="joint_1_velocity_limit" value="2.0" />
+    <xacro:property name="joint_1_torque_limit" value="140" />
     <xacro:property name="joint_2" value="joint_2" />
     <xacro:property name="joint_2_type" value="revolute" />
@@ -43,6 +43,6 @@
     <xacro:property name="joint_2_upper_limit" value="${310/180*J_PI}" />
     <!-- <xacro:property name="joint_2_velocity_limit" value="${36*J_PI/180}" /> -->
-    <xacro:property name="joint_2_velocity_limit" value="1.0" />
-    <xacro:property name="joint_2_torque_limit" value="80" />
+    <xacro:property name="joint_2_velocity_limit" value="2.0" />
+    <xacro:property name="joint_2_torque_limit" value="180" />
     <xacro:property name="joint_3" value="joint_3" />
     <xacro:property name="joint_3_type" value="revolute" />
@@ -53,6 +53,6 @@
     <xacro:property name="joint_3_upper_limit" value="${325/180*J_PI}" />
     <!-- <xacro:property name="joint_3_velocity_limit" value="${36*J_PI/180}" /> -->
-    <xacro:property name="joint_3_velocity_limit" value="1.0" />
-    <xacro:property name="joint_3_torque_limit" value="40" />
+    <xacro:property name="joint_3_velocity_limit" value="2.0" />
+    <xacro:property name="joint_3_torque_limit" value="140" />
     <xacro:property name="joint_4" value="joint_4" />
     <xacro:property name="joint_4_type" value="continuous" />
@@ -63,6 +63,6 @@
     <xacro:property name="joint_4_upper_limit" value="${2*J_PI}" />
     <!-- <xacro:property name="joint_4_velocity_limit" value="${48*J_PI/180}" /> -->
-    <xacro:property name="joint_4_velocity_limit" value="1.0" />
-    <xacro:property name="joint_4_torque_limit" value="20" />
+    <xacro:property name="joint_4_velocity_limit" value="2.0" />
+    <xacro:property name="joint_4_torque_limit" value="120" />
     <xacro:property name="joint_5" value="joint_5" />
     <xacro:property name="joint_5_type" value="continuous" />
@@ -73,6 +73,6 @@
     <xacro:property name="joint_5_upper_limit" value="${2*J_PI}" />
     <!-- <xacro:property name="joint_5_velocity_limit" value="${48*J_PI/180}" /> -->
-    <xacro:property name="joint_5_velocity_limit" value="1.0" />
-    <xacro:property name="joint_5_torque_limit" value="20" />
+    <xacro:property name="joint_5_velocity_limit" value="2.0" />
+    <xacro:property name="joint_5_torque_limit" value="120" />
     <xacro:property name="joint_6" value="joint_6" />
     <xacro:property name="joint_6_type" value="continuous" />
@@ -83,6 +83,6 @@
     <xacro:property name="joint_6_upper_limit" value="${2*J_PI}" />
     <!-- <xacro:property name="joint_6_velocity_limit" value="${48*J_PI/180}" /> -->
-    <xacro:property name="joint_6_velocity_limit" value="1.0" />
-    <xacro:property name="joint_6_torque_limit" value="20" />
+    <xacro:property name="joint_6_velocity_limit" value="2.0" />
+    <xacro:property name="joint_6_torque_limit" value="120" />
     <xacro:property name="joint_end_effector" value="end_effector_offset" />
     <xacro:property name="joint_end_effector_type" value="fixed" />

File: summit_description/robots/summit_xl_hl_root.urdf.xacro (robot description, xacro)
@@ -186,8 +186,8 @@
         </xacro:if>
         <xacro:if value="${kinematic_model == 'force_omni'}">
-            <xacro:ros_force_based_move prefix="${prefix}" publish_tf="false"/>
+            <xacro:ros_force_based_move prefix="${prefix}" publish_tf="true"/>
         </xacro:if>
         <xacro:if value="${kinematic_model == 'force_diff'}">
-            <xacro:ros_force_based_move_diff prefix="${prefix}" publish_tf="false"/>
+            <xacro:ros_force_based_move_diff prefix="${prefix}" publish_tf="true"/>
         </xacro:if>
         <xacro:if value="${enable_ros_control}">

File: summit_mico_description/robots/summit_mico_csl.urdf.xacro (robot description, xacro)
@@ -2,6 +2,11 @@
 <robot name="summit_mico_csl"
     xmlns:xacro="http://www.ros.org/wiki/xacro">
+    <xacro:arg name="prefix" default=""/>
+    <xacro:arg name="platform_mode" default="omni"/>
+    <xacro:arg name="arm_interface" default="velocity"/>
+    <xacro:arg name="enable_camera" default="true"/>
+    <xacro:arg name="color" default="None"/>
     <!-- Import summit XL root -->
     <xacro:include filename="$(find summit_mico_description)/robots/summit_mico_root.xacro" />
-    <xacro:summit_mico prefix="" />
+    <xacro:summit_mico prefix="$(arg prefix)" platform_mode="$(arg platform_mode)" arm_interface="$(arg arm_interface)" color="$(arg color)" camera="$(arg enable_camera)"/>
 </robot>

File: summit_mico_description/robots/summit_mico_root.xacro (robot description, xacro)
@@ -13,5 +13,5 @@
             <xacro:property name="kin_mode" value="force_diff"/>
         </xacro:unless>
-        <xacro:summit_xl_robot prefix="" kinematic_model="${kin_mode}" kinect="${camera}" mini_pc="true" enable_ros_control="false">
+        <xacro:summit_xl_robot prefix="${prefix}" kinematic_model="${kin_mode}" kinect="${camera}" mini_pc="true" enable_ros_control="false">
             <origin xyz="0 0 0" rpy="0 0 0"/>
         </xacro:summit_xl_robot>
@@ -22,5 +22,5 @@
             </inertial>
         </link> -->
-        <link name="root">
+        <link name="${prefix}root">
             <inertial>
                 <mass value="1"/>
@@ -28,11 +28,11 @@
             </inertial>
         </link>
-        <joint name="connect_root_and_summit" type="fixed">
-          <child link="root" />
-          <parent link="base_link" />
+        <joint name="${prefix}connect_root_and_summit" type="fixed">
+          <child link="${prefix}root" />
+          <parent link="${prefix}base_link" />
           <origin xyz="0.19 0 0.17" rpy="0 ${0.0*PI/180} 0" />
         </joint>
-        <property name="robot_root" value="root" />
-        <xacro:mico2fingers base_parent="root" prefix="mico" interface="${arm_interface}" robot_control_ns='' color="${color}"/>
+        <property name="robot_root" value="${prefix}root" />
+        <xacro:mico2fingers base_parent="${prefix}root" prefix="${prefix}mico" interface="${arm_interface}" robot_control_ns='' color="${color}" J2_offset="2.355" J3_offset="2.355"  J4_offset="0.0" J6_offset="1.57" />
     </xacro:macro>
 </robot>
