Commit message: cooperative object manipulation

File: mico_description/urdf/kinova_common.xacro (robot description, xacro)
@@ -13,5 +13,5 @@
   xmlns:physics="http://playerstage.sourceforge.net/gazebo/xmlschema/#physics"
   xmlns:xacro="http://www.ros.org/wiki/xacro">
-  <xacro:include filename="$(find kinova_description)/urdf/kinova_inertial.xacro" />
+  <xacro:include filename="$(find  mico_description)/urdf/kinova_inertial.xacro" />
   <xacro:property name="J_PI" value="3.1415926535897931" />
   <xacro:macro name="kinova_armlink" params="link_name link_mesh ring_mesh:=ring_big use_ring_mesh:=false mesh_no">
@@ -43,7 +43,7 @@
       <xacro:if value="${link_mesh == 'None'}">
         <inertial>
-          <mass value="0.5" />
+          <mass value="1" />
           <origin xyz="0 0 0" />
-          <xacro:inertia_cylinder height="0.14"  radius = "0.04" mass="0.7477"/>
+          <xacro:inertia_cylinder2 height="0.14"  radius = "0.04" mass="0.7477"/>
         </inertial>
       </xacro:if>
@@ -57,5 +57,5 @@
       <limit effort="${joint_torque_limit}" velocity="${joint_velocity_limit}" lower="${joint_lower_limit}" upper="${joint_upper_limit}"/>
       <origin xyz="${joint_origin_xyz}" rpy="${joint_origin_rpy}"/>
-      <dynamics damping="0.3" friction="0.1"/>
+      <dynamics damping="0.5" friction="0.5"/>
     </joint>
     <xacro:unless value="${fixed}">
@@ -123,4 +123,5 @@
       <origin xyz="${finger_origin_xyz}" rpy="${finger_origin_rpy}"/>
       <limit lower="0" upper="1.51" effort="2" velocity="1"/>
+      <dynamics damping="0.5" friction="0.5"/>
     </joint>
     <xacro:kinova_armlink link_name="${prefix}link_finger_tip_${finger_number}" link_mesh="finger_distal" mesh_no="58"/>
@@ -131,4 +132,5 @@
       <origin xyz="0.044 -0.003 0" rpy="0 0 0"/>
       <limit lower="0" upper="2" effort="2" velocity="1"/>
+      <dynamics damping="0.5" friction="0.5"/>
     </joint>
     <xacro:unless value="${fixed}">

File: mico_description/urdf/kinova_inertial.xacro (robot description, xacro)
@@ -30,22 +30,23 @@
 -->
 <xacro:property name="mass_mul" value="0.5" />
-<xacro:macro name="inertia_cylinder" params="mass height radius axis:=0">
+<xacro:property name="global_mass" value="1" />
+<xacro:macro name="inertia_cylinder2" params="mass height radius axis:=0">
   <!-- z Axis -->
   <xacro:unless value="${axis}">
-    <inertia  ixx="1.0" ixy="0" ixz="0"
-              iyy="1.0" iyz="0"
-              izz="1.0" />
+    <inertia  ixx="1" ixy="0" ixz="0"
+              iyy="1" iyz="0"
+              izz="1" />
   </xacro:unless>
   <!-- y Axis -->
   <xacro:unless value="${axis-1}">
-   <inertia  ixx="1.0" ixy="0" ixz="0"
-             iyy="1.0"
-             izz="1.0" iyz="0" />
+   <inertia  ixx="1" ixy="0" ixz="0"
+             iyy="1"
+             izz="1" iyz="0" />
   </xacro:unless>
   <!-- x Axis -->
   <xacro:unless value="${axis-2}">
-   <inertia  ixx="1.0"
-             iyy="1.0" iyz="0"
-             izz="1.0" ixy="0" ixz="0" />
+   <inertia  ixx="1"
+             iyy="1" iyz="0"
+             izz="1" ixy="0" ixz="0" />
   </xacro:unless>
 </xacro:macro>
@@ -54,7 +55,8 @@
   <xacro:unless value="${mesh_no}">
     <inertial>
-        <mass value="${mass_mul*0.46784}" />
-        <origin xyz="0 0 0.1255" rpy="0 0 0"/>
-        <xacro:inertia_cylinder height="0.14"  radius = "0.04" mass="0.46784"/>
+        <mass value="${global_mass}" /> <!--"${mass_mul*0.46784}" /> -->
+        <!-- <origin xyz="0 0 0.1255" rpy="0 0 0"/> -->
+        <origin xyz="0 0 0" rpy="0 0 0"/>
+        <xacro:inertia_cylinder2 height="0.14"  radius = "0.04" mass="0.46784"/>
     </inertial>
   </xacro:unless>
@@ -62,7 +64,8 @@
   <xacro:unless value="${mesh_no-1}">
     <inertial>
-        <mass value="${mass_mul*0.7477}" />
-        <origin xyz="0 -0.002 -0.0605" />
-        <xacro:inertia_cylinder height="0.14"  radius = "0.04" mass="0.7477"/>
+        <mass value="${global_mass}" /> <!--"${mass_mul*0.7477}" /> -->
+        <!-- <origin xyz="0 -0.002 -0.0605" /> -->
+        <origin xyz="0 0 0" rpy="0 0 0"/>
+        <xacro:inertia_cylinder2 height="0.14"  radius = "0.04" mass="0.7477"/>
     </inertial>
   </xacro:unless>
@@ -70,7 +73,8 @@
   <xacro:unless value="${mesh_no-2}">
     <inertial>
-        <mass value="${mass_mul*0.99}" />
-        <origin xyz="0 -0.2065 -0.01" />
-        <xacro:inertia_cylinder height="0.35"  radius = "0.04" mass="0.99" axis="1"/>
+        <mass value="${global_mass}" />
+        <!-- <origin xyz="0 -0.2065 -0.01" /> -->
+        <origin xyz="0 0 0" rpy="0 0 0"/>
+        <xacro:inertia_cylinder2 height="0.35"  radius = "0.04" mass="0.99" axis="1"/>
     </inertial>
   </xacro:unless>
@@ -78,7 +82,8 @@
   <xacro:unless value="${mesh_no-3}">
     <inertial>
-        <mass value="${mass_mul*0.6763}" />
-        <origin xyz="0 0.081 -0.0086" />
-        <xacro:inertia_cylinder height="0.15"  radius = "0.03" mass="0.6763" axis="1"/>
+        <mass value="${global_mass}" />
+        <!-- <origin xyz="0 0.081 -0.0086" /> -->
+        <origin xyz="0 0 0" rpy="0 0 0"/>
+        <xacro:inertia_cylinder2 height="0.15"  radius = "0.03" mass="0.6763" axis="1"/>
     </inertial>
   </xacro:unless>
@@ -86,7 +91,8 @@
   <xacro:unless value="${mesh_no-4}">
     <inertial>
-        <mass value="${mass_mul*0.426367}" />
-        <origin xyz="0 -0.037 -0.0642" />
-        <xacro:inertia_cylinder height="0.02"  radius = "0.04" mass="0.1785"/>
+        <mass value="${global_mass}" />
+        <!-- <origin xyz="0 -0.037 -0.0642" /> -->
+        <origin xyz="0 0 0" rpy="0 0 0"/>
+        <xacro:inertia_cylinder2 height="0.02"  radius = "0.04" mass="0.1785"/>
     </inertial>
   </xacro:unless>
@@ -94,7 +100,8 @@
   <xacro:unless value="${mesh_no-5}">
     <inertial>
-        <mass value="${mass_mul*0.85968}" />
-        <origin xyz="0 -0.145  -0.0076"/>
-        <xacro:inertia_cylinder height="0.25"  radius = "0.03" mass="0.85968" axis="1"/>
+        <mass value="${global_mass}" />
+        <!-- <origin xyz="0 -0.145  -0.0076"/> -->
+        <origin xyz="0 0 0" rpy="0 0 0"/>
+        <xacro:inertia_cylinder2 height="0.25"  radius = "0.03" mass="0.85968" axis="1"/>
     </inertial>
   </xacro:unless>
@@ -102,7 +109,8 @@
   <xacro:unless value="${mesh_no-6}">
     <inertial>
-        <mass value="${mass_mul*0.8447}" />
-        <origin xyz="0 -0.103563213 0" />
-        <xacro:inertia_cylinder height="0.18"  radius = "0.03" mass="0.8447" axis="1"/>
+        <mass value="${global_mass}" />
+        <!-- <origin xyz="0 -0.103563213 0" /> -->
+        <origin xyz="0 0 0" rpy="0 0 0"/>
+        <xacro:inertia_cylinder2 height="0.18"  radius = "0.03" mass="0.8447" axis="1"/>
     </inertial>
   </xacro:unless>
@@ -110,7 +118,8 @@
   <xacro:unless value="${mesh_no-7}">
     <inertial>
-        <mass value="${mass_mul*0.8447}" />
-        <origin xyz="0 0 -0.1022447445" />
-        <xacro:inertia_cylinder height="0.18"  radius = "0.03" mass="0.8447"/>
+        <mass value="${global_mass}" />
+        <!-- <origin xyz="0 0 -0.1022447445" /> -->
+        <origin xyz="0 0 0" rpy="0 0 0"/>
+        <xacro:inertia_cylinder2 height="0.18"  radius = "0.03" mass="0.8447"/>
     </inertial>
   </xacro:unless>
@@ -118,7 +127,8 @@
   <xacro:unless value="${mesh_no-8}">
     <inertial>
-        <mass value="${10*0.463}" />
-        <origin xyz="0 0.0028848942 -0.0541932613" />
-        <xacro:inertia_cylinder height="0.1"  radius = "0.02" mass="0.463"/>
+        <mass value="${global_mass}" />
+        <!-- <origin xyz="0 0.0028848942 -0.0541932613" /> -->
+        <origin xyz="0 0 0" rpy="0 0 0"/>
+        <xacro:inertia_cylinder2 height="0.1"  radius = "0.02" mass="0.463"/>
     </inertial>
   </xacro:unless>
@@ -126,7 +136,8 @@
   <xacro:unless value="${mesh_no-9}">
     <inertial>
-        <mass value="${mass_mul*0.463}" />
-        <origin xyz="0 0.0497208855 -0.0028562765" />
-        <xacro:inertia_cylinder height="0.1"  radius = "0.02" mass="0.463" axis="1"/>
+        <mass value="${global_mass}" />
+        <!-- <origin xyz="0 0.0497208855 -0.0028562765" /> -->
+        <origin xyz="0 0 0" rpy="0 0 0"/>
+        <xacro:inertia_cylinder2 height="0.1"  radius = "0.02" mass="0.463" axis="1"/>
     </inertial>
   </xacro:unless>
@@ -134,7 +145,8 @@
   <xacro:unless value="${mesh_no-10}">
     <inertial>
-        <mass value="${mass_mul*0.606}" />
-        <origin xyz="0 0.0463 -0.0065" />
-        <xacro:inertia_cylinder height="0.08"  radius = "0.02" mass="0.606" axis="1"/>
+        <mass value="${global_mass}" />
+        <!-- <origin xyz="0 0.0463 -0.0065" /> -->
+        <origin xyz="0 0 0" rpy="0 0 0"/>
+        <xacro:inertia_cylinder2 height="0.08"  radius = "0.02" mass="0.606" axis="1"/>
     </inertial>
   </xacro:unless>
@@ -142,15 +154,17 @@
   <xacro:unless value="${mesh_no - 55}">
     <inertial>
-        <mass value="${mass_mul*0.99}" />
-        <origin xyz="0 0 -0.06" />
-        <xacro:inertia_cylinder height="0.03"  radius = "0.04" mass="0.727"/>
+        <mass value="${global_mass}" />
+        <!-- <origin xyz="0 0 -0.06" /> -->
+        <origin xyz="0 0 0" rpy="0 0 0"/>
+        <xacro:inertia_cylinder2 height="0.03"  radius = "0.04" mass="0.727"/>
     </inertial>
   </xacro:unless>
   <!-- hand 2 finger = 56 -->
-  <xacro:unless value="${mesh_no - 56}">
+  <xacro:unless value="${global_mass}">
    <inertial>
         <mass value="0.78" />
-        <origin xyz="0 0 -0.06" />
-        <xacro:inertia_cylinder height="0.03"  radius = "0.04" mass="0.78"/>
+        <!-- <origin xyz="0 0 -0.06" /> -->
+        <origin xyz="0 0 0" rpy="0 0 0"/>
+        <xacro:inertia_cylinder2 height="0.03"  radius = "0.04" mass="0.78"/>
     </inertial>
   </xacro:unless>
@@ -158,7 +172,8 @@
   <xacro:unless value="${mesh_no - 57}">
     <inertial>
-        <mass value="0.01" />
-        <origin xyz="0.022 0 0" />
-        <xacro:inertia_cylinder height="0.03"  radius = "0.004" mass="0.01"/>
+        <mass value="${global_mass}" />
+        <!-- <origin xyz="0.022 0 0" /> -->
+        <origin xyz="0 0 0" rpy="0 0 0"/>
+        <xacro:inertia_cylinder2 height="0.03"  radius = "0.004" mass="0.01"/>
     </inertial>
   </xacro:unless>
@@ -166,7 +181,8 @@
   <xacro:unless value="${mesh_no - 58}">
     <inertial>
-        <mass value="0.01" />
-        <origin xyz="0.022 0 0" />
-        <xacro:inertia_cylinder height="0.03"  radius = "0.004" mass="0.01"/>
+        <mass value="${global_mass}" />
+        <!-- <origin xyz="0.022 0 0" /> -->
+        <origin xyz="0 0 0" rpy="0 0 0"/>
+        <xacro:inertia_cylinder2 height="0.03"  radius = "0.004" mass="0.01"/>
     </inertial>
   </xacro:unless>

File: mico_description/urdf/mico2fingers.xacro (robot description, xacro)
@@ -19,6 +19,8 @@
     <!-- Import all Kinova Mico Arm Properties elements -->
     <xacro:include filename="$(find mico_description)/urdf/micoproperties.xacro" />
-    <xacro:macro name="mico2fingers" params="base_parent robot_control_ns:='' prefix:='mico' interface:=velocity color:='None' J1_offset:=0.0 J2_offset:=0.0 J3_offset:=0.0 J4_offset:=0.0 J5_offset:=0.0 J6_offset:=0.0">
-        <xacro:gazebo_config robot_namespace="${robot_control_ns}"/>
+    <xacro:macro name="mico2fingers" params="base_parent robot_control_ns:='' prefix:='mico' interface:=velocity color:='None' J1_offset:=0.0 J2_offset:=0.0 J3_offset:=0.0 J4_offset:=0.0 J5_offset:=0.0 J6_offset:=0.0 gazebo_ros_control:=true">
+        <xacro:if value="${gazebo_ros_control}">
+            <xacro:gazebo_config robot_namespace="${robot_control_ns}"/>
+        </xacro:if>
         <xacro:kinova_armlink link_name="${prefix}_link_base" link_mesh="${link_base_mesh}" mesh_no="${link_base_mesh_no}"/>
         <xacro:kinova_armjoint joint_name="${prefix}_joint_base" type="${joint_base_type}" parent="${base_parent}" child="${prefix}_link_base" joint_axis_xyz="${joint_base_axis_xyz}" joint_origin_xyz="${joint_base_origin_xyz}" joint_origin_rpy="${joint_base_origin_rpy}" joint_lower_limit="0" joint_upper_limit="0" joint_velocity_limit="0" joint_torque_limit="0" fixed="true"/>

File: summit_mico_description/robots/summit_mico_root.xacro (robot description, xacro)
@@ -6,5 +6,5 @@
     <!--  -->
     <xacro:include filename="$(find mico_description)/urdf/mico2fingers.xacro" />
-    <xacro:macro name="summit_mico" params="prefix *origin platform_mode:='omni' arm_interface:='velocity' color:='None' camera:=true">
+    <xacro:macro name="summit_mico" params="prefix *origin platform_mode:='omni' arm_interface:='velocity' color:='None' camera:=true gazebo_ros_control:=true">
         <xacro:if value="${platform_mode in ['omni', 'force_omni', 'force', 'Omni']}">
             <xacro:property name="kin_mode" value="force_omni"/>
@@ -29,10 +29,40 @@
         </link>
         <joint name="${prefix}connect_root_and_summit" type="fixed">
-          <child link="${prefix}root" />
-          <parent link="${prefix}base_link" />
-          <origin xyz="0.19 0 0.17" rpy="0 ${0.0*PI/180} 0" />
+            <child link="${prefix}root" />
+            <parent link="${prefix}base_link" />
+            <origin xyz="0.19 0 0.17" rpy="0 ${0.0*PI/180} 0" />
         </joint>
         <property name="robot_root" value="${prefix}root" />
-        <xacro:mico2fingers base_parent="${prefix}root" prefix="${prefix}mico" interface="${arm_interface}" robot_control_ns='' color="${color}" J2_offset="2.355" J3_offset="2.355"  J4_offset="0.0" J6_offset="1.57" />
+        <xacro:mico2fingers base_parent="${prefix}root" prefix="${prefix}mico" interface="${arm_interface}" robot_control_ns='' color="${color}" J2_offset="2.355" J3_offset="2.355" J4_offset="0.0" J6_offset="1.57" gazebo_ros_control="${gazebo_ros_control}"/>
+    </xacro:macro>
+    <!-- Inertial of Cylinder -->
+    <xacro:macro name="inertia_cylinder" params="mass height radius axis:=0">
+        <xacro:property name="Ir" value="${0.0833*mass*(3.0*radius*radius + height*height)}" />
+        <xacro:property name="Ih" value="${0.5*mass*(radius*radius)}" />
+        <!-- z Axis -->
+        <xacro:unless value="${axis}">
+            <inertia ixx="${Ir}" ixy="0" ixz="0" iyy="${Ir}" iyz="0" izz="${Ih}" />
+        </xacro:unless>
+        <!-- y Axis -->
+        <xacro:unless value="${axis-1}">
+            <inertia ixx="${Ir}" ixy="0" ixz="0" iyy="${Ih}" izz="${Ir}" iyz="0" />
+        </xacro:unless>
+        <!-- x Axis -->
+        <xacro:unless value="${axis-2}">
+            <inertia ixx="${Ih}" iyy="${Ir}" iyz="0" izz="${Ir}" ixy="0" ixz="0" />
+        </xacro:unless>
+    </xacro:macro>
+    <!-- Inertial of Box -->
+    <xacro:macro name="inertia_box" params="mass height:=0.05 width:=0.0 depth:=0.0">
+        <xacro:if value="${width == 0.0}">
+            <xacro:property name="width" value="${height}"/>
+        </xacro:if>
+        <xacro:if value="${depth == 0.0}">
+            <xacro:property name="depth" value="${height}"/>
+        </xacro:if>
+        <xacro:property name="Iw" value="${(1.0/12.0)*mass*(height*height + depth*depth)}" />
+        <xacro:property name="Ih" value="${(1.0/12.0)*mass*(width*width + depth*depth)}" />
+        <xacro:property name="Id" value="${(1.0/12.0)*mass*(width*width + height*height)}" />
+        <inertia ixx="${Iw}" ixy="0" ixz="0" iyy="${Ih}" iyz="0" izz="${Id}" />
     </xacro:macro>
 </robot>
