Commit message: minor updates

File: mico_description/urdf/kinova_common.xacro (robot description, xacro)
@@ -18,12 +18,12 @@
     <link name="${link_name}">
       <xacro:unless value="${link_mesh == 'None'}">
-        <visual>
-          <geometry>
-            <mesh filename="package://kinova_description/meshes/${link_mesh}.dae"/>
-          </geometry>
-          <material name="carbon_fiber">
-            <color rgba="0.792156862745098 0.819607843137255 0.933333333333333 1" />
-          </material>
-        </visual>
+          <visual>
+            <geometry>
+              <mesh filename="package://kinova_description/meshes/${link_mesh}.dae"/>
+            </geometry>
+            <material name="carbon_fiber">
+              <color rgba="0.792156862745098 0.819607843137255 0.933333333333333 1" />
+            </material>
+          </visual>
         <!-- Adding ring to the model -->
         <xacro:if value="${use_ring_mesh}">
@@ -32,4 +32,7 @@
               <mesh filename="package://kinova_description/meshes/${ring_mesh}.dae"/>
             </geometry>
+            <material name="carbon_fiber">
+              <color rgba="0.792156862745098 0.819607843137255 0.933333333333333 1" />
+            </material>
           </visual>
         </xacro:if>
@@ -43,7 +46,8 @@
       <xacro:if value="${link_mesh == 'None'}">
         <inertial>
-          <mass value="1" />
-          <origin xyz="0 0 0" />
-          <xacro:inertia_cylinder2 height="0.14"  radius = "0.04" mass="0.7477"/>
+          <mass value="0.1" />
+          <inertia  ixx="0.1"
+          iyy="0.1" iyz="0"
+          izz="0.1" ixy="0" ixz="0" />
         </inertial>
       </xacro:if>
@@ -57,5 +61,5 @@
       <limit effort="${joint_torque_limit}" velocity="${joint_velocity_limit}" lower="${joint_lower_limit}" upper="${joint_upper_limit}"/>
       <origin xyz="${joint_origin_xyz}" rpy="${joint_origin_rpy}"/>
-      <dynamics damping="0.5" friction="0.5"/>
+      <dynamics damping="1.5" friction="0.5"/>
     </joint>
     <xacro:unless value="${fixed}">
@@ -99,4 +103,9 @@
   <xacro:macro name="kinova_virtual_link" params="link_name">
     <link name="${link_name}"/>
+    <inertial>
+      <origin xyz="0 0 0" />
+      <mass value="1.0" />
+      <xacro:inertia_cylinder2 height="0.14"  radius = "0.04" mass="0.7477"/>
+    </inertial>
   </xacro:macro>
   <xacro:macro name="kinova_virtual_joint" params="joint_name type parent child joint_axis_xyz joint_origin_xyz joint_origin_rpy joint_lower_limit joint_upper_limit">
@@ -105,6 +114,7 @@
       <child link="${child}"/>
       <axis xyz="${joint_axis_xyz}"/>
-      <limit effort="20000" velocity="2" lower="${joint_lower_limit}" upper="${joint_upper_limit}"/>
+      <limit effort="20000" velocity="3" lower="${joint_lower_limit}" upper="${joint_upper_limit}"/>
       <origin xyz="${joint_origin_xyz}" rpy="${joint_origin_rpy}"/>
+      <dynamics damping="1.5" friction="0.5"/>
     </joint>
   </xacro:macro>
@@ -123,5 +133,5 @@
       <origin xyz="${finger_origin_xyz}" rpy="${finger_origin_rpy}"/>
       <limit lower="0" upper="1.51" effort="2" velocity="1"/>
-      <dynamics damping="0.5" friction="0.5"/>
+      <dynamics damping="1.5" friction="0.5"/>
     </joint>
     <xacro:kinova_armlink link_name="${prefix}link_finger_tip_${finger_number}" link_mesh="finger_distal" mesh_no="58"/>
@@ -132,5 +142,5 @@
       <origin xyz="0.044 -0.003 0" rpy="0 0 0"/>
       <limit lower="0" upper="2" effort="2" velocity="1"/>
-      <dynamics damping="0.5" friction="0.5"/>
+      <dynamics damping="1.5" friction="0.5"/>
     </joint>
     <xacro:unless value="${fixed}">

File: mico_description/urdf/kinova_inertial.xacro (robot description, xacro)
@@ -40,13 +40,13 @@
   <!-- y Axis -->
   <xacro:unless value="${axis-1}">
-   <inertia  ixx="1" ixy="0" ixz="0"
-             iyy="1"
-             izz="1" iyz="0" />
+   <inertia  ixx="0.4" ixy="0" ixz="0"
+             iyy="0.4"
+             izz="0.4" iyz="0" />
   </xacro:unless>
   <!-- x Axis -->
   <xacro:unless value="${axis-2}">
-   <inertia  ixx="1"
-             iyy="1" iyz="0"
-             izz="1" ixy="0" ixz="0" />
+   <inertia  ixx="0.1"
+             iyy="0.1" iyz="0"
+             izz="0.1" ixy="0" ixz="0" />
   </xacro:unless>
 </xacro:macro>
@@ -76,5 +76,5 @@
         <!-- <origin xyz="0 -0.2065 -0.01" /> -->
         <origin xyz="0 0 0" rpy="0 0 0"/>
-        <xacro:inertia_cylinder2 height="0.35"  radius = "0.04" mass="0.99" axis="1"/>
+        <xacro:inertia_cylinder2 height="0.35"  radius = "0.04" mass="0.99" axis="0"/>
     </inertial>
   </xacro:unless>
@@ -85,5 +85,5 @@
         <!-- <origin xyz="0 0.081 -0.0086" /> -->
         <origin xyz="0 0 0" rpy="0 0 0"/>
-        <xacro:inertia_cylinder2 height="0.15"  radius = "0.03" mass="0.6763" axis="1"/>
+        <xacro:inertia_cylinder2 height="0.15"  radius = "0.03" mass="0.6763" axis="0"/>
     </inertial>
   </xacro:unless>
@@ -94,5 +94,5 @@
         <!-- <origin xyz="0 -0.037 -0.0642" /> -->
         <origin xyz="0 0 0" rpy="0 0 0"/>
-        <xacro:inertia_cylinder2 height="0.02"  radius = "0.04" mass="0.1785"/>
+        <xacro:inertia_cylinder2 height="0.02"  radius = "0.04" mass="0.1785" axis="2"/>
     </inertial>
   </xacro:unless>
@@ -103,5 +103,5 @@
         <!-- <origin xyz="0 -0.145  -0.0076"/> -->
         <origin xyz="0 0 0" rpy="0 0 0"/>
-        <xacro:inertia_cylinder2 height="0.25"  radius = "0.03" mass="0.85968" axis="1"/>
+        <xacro:inertia_cylinder2 height="0.25"  radius = "0.03" mass="0.85968" axis="0"/>
     </inertial>
   </xacro:unless>
@@ -112,5 +112,5 @@
         <!-- <origin xyz="0 -0.103563213 0" /> -->
         <origin xyz="0 0 0" rpy="0 0 0"/>
-        <xacro:inertia_cylinder2 height="0.18"  radius = "0.03" mass="0.8447" axis="1"/>
+        <xacro:inertia_cylinder2 height="0.18"  radius = "0.03" mass="0.8447" axis="0"/>
     </inertial>
   </xacro:unless>
@@ -139,5 +139,5 @@
         <!-- <origin xyz="0 0.0497208855 -0.0028562765" /> -->
         <origin xyz="0 0 0" rpy="0 0 0"/>
-        <xacro:inertia_cylinder2 height="0.1"  radius = "0.02" mass="0.463" axis="1"/>
+        <xacro:inertia_cylinder2 height="0.1"  radius = "0.02" mass="0.463" axis="0"/>
     </inertial>
   </xacro:unless>
@@ -148,5 +148,5 @@
         <!-- <origin xyz="0 0.0463 -0.0065" /> -->
         <origin xyz="0 0 0" rpy="0 0 0"/>
-        <xacro:inertia_cylinder2 height="0.08"  radius = "0.02" mass="0.606" axis="1"/>
+        <xacro:inertia_cylinder2 height="0.08"  radius = "0.02" mass="0.606" axis="0"/>
     </inertial>
   </xacro:unless>
@@ -161,10 +161,10 @@
   </xacro:unless>
   <!-- hand 2 finger = 56 -->
-  <xacro:unless value="${global_mass}">
+  <xacro:unless value="${mesh_no - 56}">
    <inertial>
-        <mass value="0.78" />
+        <mass value="0.1" />
         <!-- <origin xyz="0 0 -0.06" /> -->
         <origin xyz="0 0 0" rpy="0 0 0"/>
-        <xacro:inertia_cylinder2 height="0.03"  radius = "0.04" mass="0.78"/>
+        <xacro:inertia_cylinder2 height="0.03"  radius = "0.04" mass="0.78" axis="2"/>
     </inertial>
   </xacro:unless>

File: mico_description/urdf/mico2fingers_root.xacro (robot description, xacro)
@@ -24,7 +24,8 @@
         <xacro:kinova_armlink link_name="${prefix}_link_6" link_mesh="${link_6_mesh}" use_ring_mesh="true" ring_mesh="ring_small" mesh_no="${link_6_mesh_no}"/>
         <xacro:kinova_armjoint joint_name="${prefix}_joint_6" type="${joint_6_type}" parent="${prefix}_link_5" child="${prefix}_link_6" joint_axis_xyz="${joint_6_axis_xyz}" joint_origin_xyz="${joint_6_origin_xyz}" joint_origin_rpy="${joint_6_origin_rpy}" joint_lower_limit="${joint_6_lower_limit}" joint_upper_limit="${joint_6_upper_limit}" joint_velocity_limit="${joint_6_velocity_limit}" joint_torque_limit="${joint_6_torque_limit}" interface="${interface}"/>
+<!--
         <xacro:kinova_virtual_link link_name="${prefix}_end_effector"/>
         <xacro:kinova_virtual_joint joint_name="${prefix}_joint_end_effector" type="${joint_end_effector_type}" parent="${prefix}_link_6" child="${prefix}_end_effector" joint_axis_xyz="${joint_end_effector_axis_xyz}" joint_origin_xyz="${joint_end_effector_origin_xyz}" joint_origin_rpy="${joint_end_effector_origin_rpy}" joint_lower_limit="0" joint_upper_limit="0"/>
-        <xacro:kinova_2fingers link_hand="${prefix}_link_6" prefix="${prefix}_"/>
+        <xacro:kinova_2fingers link_hand="${prefix}_link_6" prefix="${prefix}_"/> -->
     </xacro:macro>
 </robot>

File: mico_description/urdf/micoproperties.xacro (robot description, xacro)
@@ -26,5 +26,5 @@
     <xacro:property name="joint_base_origin_rpy" value="0 0 0" />
     <xacro:property name="joint_1" value="joint_1" />
-    <xacro:property name="joint_1_type" value="continuous" />
+    <xacro:property name="joint_1_type" value="revolute" />
     <xacro:property name="joint_1_axis_xyz" value="0 0 1" />
     <xacro:property name="joint_1_origin_xyz" value="0 0 0.15675" />
@@ -33,6 +33,6 @@
     <xacro:property name="joint_1_upper_limit" value="${2*J_PI}" />
     <!-- <xacro:property name="joint_1_velocity_limit" value="${36*J_PI/180}" /> -->
-    <xacro:property name="joint_1_velocity_limit" value="2.0" />
-    <xacro:property name="joint_1_torque_limit" value="140" />
+    <xacro:property name="joint_1_velocity_limit" value="6.0" />
+    <xacro:property name="joint_1_torque_limit" value="500" />
     <xacro:property name="joint_2" value="joint_2" />
     <xacro:property name="joint_2_type" value="revolute" />
@@ -43,6 +43,6 @@
     <xacro:property name="joint_2_upper_limit" value="${310/180*J_PI}" />
     <!-- <xacro:property name="joint_2_velocity_limit" value="${36*J_PI/180}" /> -->
-    <xacro:property name="joint_2_velocity_limit" value="2.0" />
-    <xacro:property name="joint_2_torque_limit" value="180" />
+    <xacro:property name="joint_2_velocity_limit" value="6.0" />
+    <xacro:property name="joint_2_torque_limit" value="500" />
     <xacro:property name="joint_3" value="joint_3" />
     <xacro:property name="joint_3_type" value="revolute" />
@@ -53,8 +53,8 @@
     <xacro:property name="joint_3_upper_limit" value="${325/180*J_PI}" />
     <!-- <xacro:property name="joint_3_velocity_limit" value="${36*J_PI/180}" /> -->
-    <xacro:property name="joint_3_velocity_limit" value="2.0" />
-    <xacro:property name="joint_3_torque_limit" value="140" />
+    <xacro:property name="joint_3_velocity_limit" value="6.0" />
+    <xacro:property name="joint_3_torque_limit" value="500" />
     <xacro:property name="joint_4" value="joint_4" />
-    <xacro:property name="joint_4_type" value="continuous" />
+    <xacro:property name="joint_4_type" value="revolute" />
     <xacro:property name="joint_4_axis_xyz" value="0 0 1" />
     <xacro:property name="joint_4_origin_xyz" value="0 0.1231 -0.0086" />
@@ -63,8 +63,8 @@
     <xacro:property name="joint_4_upper_limit" value="${2*J_PI}" />
     <!-- <xacro:property name="joint_4_velocity_limit" value="${48*J_PI/180}" /> -->
-    <xacro:property name="joint_4_velocity_limit" value="2.0" />
-    <xacro:property name="joint_4_torque_limit" value="120" />
+    <xacro:property name="joint_4_velocity_limit" value="6.0" />
+    <xacro:property name="joint_4_torque_limit" value="500" />
     <xacro:property name="joint_5" value="joint_5" />
-    <xacro:property name="joint_5_type" value="continuous" />
+    <xacro:property name="joint_5_type" value="revolute" />
     <xacro:property name="joint_5_axis_xyz" value="0 0 1" />
     <xacro:property name="joint_5_origin_xyz" value="0 -0.03703 -0.06414" />
@@ -73,6 +73,6 @@
     <xacro:property name="joint_5_upper_limit" value="${2*J_PI}" />
     <!-- <xacro:property name="joint_5_velocity_limit" value="${48*J_PI/180}" /> -->
-    <xacro:property name="joint_5_velocity_limit" value="2.0" />
-    <xacro:property name="joint_5_torque_limit" value="120" />
+    <xacro:property name="joint_5_velocity_limit" value="6.0" />
+    <xacro:property name="joint_5_torque_limit" value="500" />
     <xacro:property name="joint_6" value="joint_6" />
     <xacro:property name="joint_6_type" value="continuous" />
@@ -83,6 +83,6 @@
     <xacro:property name="joint_6_upper_limit" value="${2*J_PI}" />
     <!-- <xacro:property name="joint_6_velocity_limit" value="${48*J_PI/180}" /> -->
-    <xacro:property name="joint_6_velocity_limit" value="2.0" />
-    <xacro:property name="joint_6_torque_limit" value="120" />
+    <xacro:property name="joint_6_velocity_limit" value="6.0" />
+    <xacro:property name="joint_6_torque_limit" value="500" />
     <xacro:property name="joint_end_effector" value="end_effector_offset" />
     <xacro:property name="joint_end_effector_type" value="fixed" />

File: summit_description/robots/summit_xl_hl_root.urdf.xacro (robot description, xacro)
@@ -14,5 +14,5 @@
     <!-- Import all available sensors -->
     <xacro:include filename="$(find robotnik_sensors)/urdf/all_sensors.urdf.xacro" />
-    <xacro:macro name="summit_xl_robot" params="prefix *origin kinematic_model:='omni' kinect:=true mini_pc:=true enable_ros_control:=true publish_tf:=false virtual_platform_joints:=false">
+    <xacro:macro name="summit_xl_robot" params="prefix *origin kinematic_model:='omni' kinect:=true mini_pc:=true enable_ros_control:=true publish_tf:=false virtual_platform_joints:=false interface:='velocity'">
         <!-- ***************** -->
         <!-- Global parameters -->
@@ -51,5 +51,5 @@
             <xacro:property name="wheel_radius" value="0.11" />
         </xacro:unless>
-        <xacro:summit_xl_hl_base prefix="${prefix}" publish_bf="true" hq="${hq}" virtual_platform_joints="${virtual_platform_joints}">
+        <xacro:summit_xl_hl_base prefix="${prefix}" publish_bf="true" hq="${hq}" virtual_platform_joints="${virtual_platform_joints}" interface="${interface}">
             <xacro:insert_block name="origin" />
         </xacro:summit_xl_hl_base>

File: summit_description/urdf/bases/summit_xl_hl_base.urdf.xacro (robot description, xacro)
@@ -3,5 +3,5 @@
   xmlns:xacro="http://www.ros.org/wiki/xacro">
   <xacro:include filename="$(find summit_description)/urdf/bases/summit_xl_base.gazebo.xacro" />
-  <xacro:macro name="summit_xl_hl_base" params="prefix publish_bf hq virtual_platform_joints:=false *origin">
+  <xacro:macro name="summit_xl_hl_base" params="prefix publish_bf hq virtual_platform_joints:=false interface:='velocity' *origin">
     <!-- Robot mechanical and motor parameters -->
     <xacro:property name="PI" value="3.1415926535897931"/>
@@ -17,7 +17,7 @@
         </visual>
         <inertial>
-          <mass value="155.0" />
+          <mass value="15.0" />
           <origin xyz="0 0 0" />
-          <inertia ixx="230.391" ixy="0.004" ixz="0.0" iyy="236.853" iyz="0.0" izz="36.125" />
+          <inertia ixx="30.391" ixy="0.004" ixz="0.0" iyy="36.853" iyz="0.0" izz="36.125" />
         </inertial>
       </link>
@@ -32,7 +32,7 @@
     <link name="${prefix}base_link">
       <inertial>
-        <mass value="155.0" />
+        <mass value="15.0" />
         <origin xyz="0 0 0" />
-        <inertia ixx="230.391" ixy="0.004" ixz="0.0" iyy="236.853" iyz="0.0" izz="36.125" />
+        <inertia ixx="23.391" ixy="0.004" ixz="0.0" iyy="23.853" iyz="0.0" izz="36.125" />
       </inertial>
       <visual>
@@ -63,7 +63,7 @@
       <link name="${prefix}world">
         <inertial>
-          <mass value="1.0" />
+          <mass value="5.0" />
           <origin xyz="0 0 0" />
-          <inertia ixx="1.0" ixy="0.004" ixz="0.0" iyy="1.0" iyz="0.0" izz="1.0" />
+          <inertia ixx="5.0" ixy="0.00" ixz="0.0" iyy="5.0" iyz="0.0" izz="5.0" />
         </inertial>
       </link>
@@ -71,7 +71,7 @@
       <link name="${prefix}platform_linear_1">
         <inertial>
-          <mass value="1.0" />
+          <mass value="5.0" />
           <origin xyz="0 0 0" />
-          <inertia ixx="1.0" ixy="0.004" ixz="0.0" iyy="1.0" iyz="0.0" izz="1.0" />
+          <inertia ixx="5.0" ixy="0.00" ixz="0.0" iyy="5.0" iyz="0.0" izz="5.0" />
         </inertial>
       </link>
@@ -79,7 +79,7 @@
       <link name="${prefix}platform_linear_2">
         <inertial>
-          <mass value="1.0" />
+          <mass value="5.0" />
           <origin xyz="0 0 0" />
-          <inertia ixx="1.0" ixy="0.004" ixz="0.0" iyy="1.0" iyz="0.0" izz="1.0" />
+          <inertia ixx="5.0" ixy="0.00" ixz="0.0" iyy="5.0" iyz="0.0" izz="5.0" />
         </inertial>
       </link>
@@ -89,6 +89,6 @@
         <child link="${prefix}platform_linear_1" />
         <axis xyz="1 0 0"/>
-        <limit lower="-500" upper="500" effort="1000" velocity="4"/>
-        <joint_properties damping="0.1" friction="0.0"/>
+        <limit lower="-500" upper="500" effort="1000" velocity="6"/>
+        <joint_properties damping="1.5" friction="0.4"/>
       </joint>
       <joint name="${prefix}platform_prismatic_y" type="prismatic">
@@ -97,6 +97,6 @@
         <child link="${prefix}platform_linear_2" />
         <axis xyz="0 1 0"/>
-        <limit lower="-500" upper="500" effort="1000" velocity="4"/>
-        <joint_properties damping="0.1" friction="0.0"/>
+        <limit lower="-500" upper="500" effort="1000" velocity="6"/>
+        <joint_properties damping="1.5" friction="0.4"/>
       </joint>
       <joint name="${prefix}platform_continuous_z" type="continuous">
@@ -105,14 +105,23 @@
         <child link="${prefix}base_footprint" />
         <axis xyz="0 0 1"/>
-        <limit lower="-500" upper="500" effort="1000" velocity="4"/>
-        <joint_properties damping="0.1" friction="0.0"/>
+        <limit lower="-500" upper="500" effort="1000" velocity="6"/>
+        <joint_properties damping="1.5" friction="0.4"/>
       </joint>
+      <xacro:if value="${interface == 'position'}">
+        <xacro:property name="hwInterface" value="hardware_interface/PositionJointInterface"/>
+      </xacro:if>
+      <xacro:if value="${interface == 'effort'}">
+        <xacro:property name="hwInterface" value="hardware_interface/EffortJointInterface"/>
+      </xacro:if>
+      <xacro:unless value="${interface in ['position','effort']}">
+        <xacro:property name="hwInterface" value="hardware_interface/VelocityJointInterface"/>
+      </xacro:unless>
       <transmission name="${prefix}platform_prismatic_x_trans">
         <type>transmission_interface/SimpleTransmission</type>
         <joint name="${prefix}platform_prismatic_x">
-          <hardwareInterface>hardware_interface/VelocityJointInterface</hardwareInterface>
+          <hardwareInterface>${hwInterface}</hardwareInterface>
         </joint>
         <actuator name="${prefix}platform_prismatic_x_actuator">
-          <hardwareInterface>hardware_interface/VelocityJointInterface</hardwareInterface>
+          <hardwareInterface>${hwInterface}</hardwareInterface>
           <mechanicalReduction>1</mechanicalReduction>
         </actuator>
@@ -121,8 +130,8 @@
         <type>transmission_interface/SimpleTransmission</type>
         <joint name="${prefix}platform_prismatic_y">
-          <hardwareInterface>hardware_interface/VelocityJointInterface</hardwareInterface>
+          <hardwareInterface>${hwInterface}</hardwareInterface>
         </joint>
         <actuator name="${prefix}platform_prismatic_y_actuator">
-          <hardwareInterface>hardware_interface/VelocityJointInterface</hardwareInterface>
+          <hardwareInterface>${hwInterface}</hardwareInterface>
           <mechanicalReduction>1</mechanicalReduction>
         </actuator>
@@ -131,8 +140,8 @@
         <type>transmission_interface/SimpleTransmission</type>
         <joint name="${prefix}platform_continuous_z">
-          <hardwareInterface>hardware_interface/VelocityJointInterface</hardwareInterface>
+          <hardwareInterface>${hwInterface}</hardwareInterface>
         </joint>
         <actuator name="${prefix}platform_continuous_z_actuator">
-          <hardwareInterface>hardware_interface/VelocityJointInterface</hardwareInterface>
+          <hardwareInterface>${hwInterface}</hardwareInterface>
           <mechanicalReduction>1</mechanicalReduction>
         </actuator>

File: summit_description/urdf/wheels/omni_wheel.urdf.xacro (robot description, xacro)
@@ -87,5 +87,5 @@
         <mu2 value="1.0"/>
         <kp value="10000000.0" />
-        <kd value="1.0" />
+        <kd value="10000.0" />
         <fdir1 value="1 0 0"/>
         <turnGravityOff>false</turnGravityOff>
