Commit message: minor updates

File: summit_mico_description/robots/summit_mico_cooperative_root.urdf.xacro (robot description, xacro)
@@ -58,5 +58,5 @@
         </xacro:if>
     </xacro:if>
-    <!-- Robot 3 Properties Dictionary if set agents > 2 -->
+    <!-- Robot 3 Properties Dictionary if set agents 2 -->
     <xacro:property name="theta_3" value="${robot_props['theta_3']}"/>
     <xacro:if value="${$(arg agents)-2}">
@@ -139,5 +139,5 @@
     <link name="world"/>
     <!-- First Robot -->
-    <xacro:summit_mico prefix="${robot_1['prefix']}" platform_mode="${robot_1['platform_mode']}" arm_interface="${robot_1['arm_interface']}" color="${robot_1['color']}" camera="${robot_1['camera']}">
+    <xacro:summit_mico prefix="${robot_1['prefix']}" platform_mode="${robot_1['platform_mode']}" arm_interface="${robot_1['arm_interface']}" color="${robot_1['color']}" camera="${robot_1['camera']}" platform_interface="effort">
         <origin xyz="0 0 0" rpy="0 0 0"/>
     </xacro:summit_mico>
@@ -149,14 +149,23 @@
     </joint>
     <xacro:ft_sensor_plugin name="${robot_1['prefix']}mico_joint_6" joint_name="${robot_1['prefix']}mico_joint_6" />
-    <xacro:if value="true">
+    <xacro:property name="use_object" value="true"/>
+    <xacro:if value="${object['mass'] == 0 and $(arg agents) == 1}">
+        <xacro:property name="use_object" value="false"/>
+    </xacro:if>
+    <xacro:if value="${use_object}">
         <!-- Object Link -->
         <link name="object">
             <visual>
+                <!-- <origin xyz="0.22 0 0.05" rpy="3.14 0 0" /> -->
                 <geometry>
                     <xacro:if value="${object['type'] == 'cylinder'}">
                         <cylinder length="${object_width}" radius="${object_length/2}"/>
                     </xacro:if>
+                    <!-- <xacro:if value="${object['type'] == 'box'}">
+                        <box size="${object_height} ${object_length} ${object_width}"/>
+                    </xacro:if> -->
                     <xacro:if value="${object['type'] == 'box'}">
                         <box size="${object_height} ${object_length} ${object_width}"/>
+                        <!-- <mesh filename="package://summit_mico_description/meshes/objects/plate.stl" scale=".013 0.015 0.015"/> -->
                     </xacro:if>
                 </geometry>
@@ -182,8 +191,10 @@
                 </xacro:if>
             </inertial>
-            <gazebo reference="object">
-                <material>Gazebo/Orange</material>
-            </gazebo>
         </link>
+        <gazebo reference="object">
+            <material>Gazebo/Orange</material>
+            <kp value="10.0" />
+            <kd value="100000.0" />
+        </gazebo>
         <!-- Attach Object to Robot 1 End effector -->
         <joint name="${robot_1['prefix']}to_object" type="fixed">

File: summit_mico_description/robots/summit_mico_root.xacro (robot description, xacro)
@@ -6,5 +6,5 @@
     <!--  -->
     <xacro:include filename="$(find mico_description)/urdf/mico2fingers.xacro" />
-    <xacro:macro name="summit_mico" params="prefix *origin platform_mode:='omni' arm_interface:='velocity' color:='None' camera:=true gazebo_ros_control:=true">
+    <xacro:macro name="summit_mico" params="prefix *origin platform_mode:='omni' arm_interface:='velocity' color:='None' camera:=true gazebo_ros_control:=true platform_interface:='velocity'">
         <xacro:if value="${platform_mode in ['omni', 'force_omni', 'force', 'Omni']}">
             <xacro:property name="kin_mode" value="force_omni"/>
@@ -13,5 +13,5 @@
             <xacro:property name="kin_mode" value="force_diff"/>
         </xacro:unless>
-        <xacro:summit_xl_robot prefix="${prefix}" kinematic_model="${kin_mode}" kinect="${camera}" mini_pc="true" enable_ros_control="false" publish_tf="false" virtual_platform_joints="true">
+        <xacro:summit_xl_robot prefix="${prefix}" kinematic_model="${kin_mode}" kinect="${camera}" mini_pc="true" enable_ros_control="false" publish_tf="false" virtual_platform_joints="true" interface="${platform_interface}">
             <xacro:insert_block name="origin" />
         </xacro:summit_xl_robot>
@@ -25,5 +25,5 @@
             <inertial>
                 <mass value="1"/>
-                <inertia ixx="0.1" ixy="0.0" ixz="0.0" iyy="0.1" iyz="0.0" izz="0.1"/>
+                <inertia ixx="1" ixy="0.0" ixz="0.0" iyy="1" iyz="0.0" izz="1"/>
             </inertial>
         </link>
